File: main.sch (EAGLE design)
At the start: 212 parts, among them CN1 5X2HEADER, CN2 MUSB-05-S-B-SM-A, CN3 1X2_HEADER, CN4 1X4_HEADER, CN5 NEB-21-R, U1 93LC56B-I/SN, U10 SN74LVC1G17D, U11 SN74LVC1G17D, U12 FT232H, U13 TPS62160, U14 LMH6639MF, U15 TCD1209DG, U16 TPS61165, U17 LMH6639MF, U18 LMH6639MF, U19 TPS62160, U2 EP4CE6E22C8N, U20 100MHz, U21 LMH6639MF, U22 TPS54233D, U23 ADS7946, U24 TPS62160, U25 DRV8825, U3 M25P16, U4 MCP1416, U5 TPS562209, U6 MCP1416, U7 USBLC6-2SC6, U8 DAC8552, U9 SN74LVC1G17D

Commit message: main board architectre
Parts:
- removed C101, C103, C104, C41, C47, C48, C49, C50, C60, C61, C66, C69, C71, C75, C76, C82, C83, C87, C88, C89: 10uF 16V, CAPACITORS:MC1206B106K160CT
- removed C113, C40, C68: 10pF 100V, CAPACITORS:06031A100FAT2A
- removed C114, C18, C19, C20, C21, C22, C23, C24, C25, C3, C34, C38, C4, C42, C43, C44, C45, C46, C5, C51, C52, C53, C54, C55, C56, C57, C6, C65, C67, C7, C70, C72, C73, C74, C77, C81, C84, C92, C94, C95, C96, C97, C98: 100nF 50V, CAPACITORS:VJ0603Y104KXACW1BC
- removed C58, C59: 18pF 50V, CAPACITORS:MC0603N180J500CT
- removed C62, C63: 1uF 50V, CAPACITORS:GRM31MR71H105KA88L
- removed C64: 220nF 50V, CAPACITORS:C1608X7R1H224K080AB
- removed C78: 8.2nF 50V, CAPACITORS:MC0603B822K500CT
- removed C79: 1.5nF 50V, CAPACITORS:MC0603B152K500CT
- removed C80: 33pF 50V, CAPACITORS:MC0603N330J500CT
- removed C85, C86: 1uF 25V, CAPACITORS:MC0603X105K250CT
- removed C90, C99: 470uF 16V, CAPACITORS:16ML470MEFC10X9
- removed C91: 470nF 25V, CAPACITORS:GRM188R71E474KA12D
- removed C93: 10nF 50V, CAPACITORS:MC0603B103K500CT
- removed CN4: 1X4_HEADER, CONNECTORs:1X4_HEADER
- removed CN5: NEB-21-R, CONNECTORs:NEB-21-R
- removed D1, D2, D3, D5: SML-311UTT86K, OPTO:SML-311UTT86K
- removed D12: B0540W, DIODES:B0540W
- removed D4: B230A, DIODES:B230A-13-F
- removed FB2, FB3, FB7: 600R, INDUCTORS:742792651
- removed L1: 3.3uH 3.3A, INDUCTORS:SRN5040-3R3M
- removed L2, L6: 2.2uH 3.5A, INDUCTORS:SRN5040-2R2Y
- removed L4: NRS6045T 100MMGK, PASSIVES:L_SMD6045T
- removed L5: 22uH, INDUCTORS:MSS1038-223MLC
- removed L7: 180uH, INDUCTORS:SRN6045TA-181M
- removed R1, R13, R2, R26, R27, R28, R29, R37, R38, R5, R50, R6: 10K, RESISTORS:CRCW060310K0FKEA
- removed R10: 33k, RESISTORS:CRCW060333K0FKEA
- removed R11: 100k, RESISTORS:CRCW0603100KFKEA
- removed R12, R39, R40, R41, R42: 51k, RESISTORS:CRCW060351K0FKEA
- removed R14: 82k, RESISTORS:CRCW060382K0FKEA
- removed R15, R36: 180k, RESISTORS:CRCW0603180KFKEA
- removed R16, R31: 12k, RESISTORS:CRCW060312K0FKEA
- removed R17: 820R, RESISTORS:CRCW0603820RFKEA
- removed R18: 330R, RESISTORS:CRCW0603330RFKEA
- removed R19: 680R, RESISTORS:CRCW0603680RFKEA
- removed R20, R21, R7, R8, R9: 1k, RESISTORS:CRCW06031K00FKEA
- removed R22: 220R, RESISTORS:CRCW0603220RFKEA
- removed R23, R24, R25, R32: 4R7, RESISTORS:CRCW06034R70FKEA
- removed R30: 2k, RESISTORS:CRCW06032K00FKEA
- removed R33, R44, R45: 0.33R, RESISTORS:CRL0603-FW-R330ELF
- removed R35, R43: 1M, RESISTORS:CRCW06031M00FKEA
- removed R4: 16R, RESISTORS:CRCW060316R0FKEA
- removed R46, R47, R48, R49: 470R, RESISTORS:CRCW0603470RFKEA
- removed TP1, TP2, TP3, TP4, TP5, TP6, TP7, TP8: 2MM_TEST_POINT, MISC:2MM_TEST_POINT
- removed U10, U11, U9: SN74LVC1G17D, ICs:SN74LVC1G17DBVR
- removed U12: FT232H, ICs:FT232HL
- removed U13, U19, U24: TPS62160, ICs:TPS62160DGKT
- removed U14, U17, U21: LMH6639MF, ICs:LMH6639MF
- removed U15: TCD1209DG, ICs:TCD1209DG
- removed U16: TPS61165, ICs:TPS61165DBVT
- removed U20: 100MHz, CRYSTALS:510BBA100M000BAG
- removed U22: TPS54233D, ICs:TPS54233D
- removed U23: ADS7946, ICs:ADS7946RTET
- removed U25: DRV8825, ICs:DRV8825PWP
- removed U3: M25P16, ICs:M25P16-VMN6P
- removed U6: MCP1416, ICs:MCP1416T
- removed U7: USBLC6-2SC6, ICs:USBLC6-2SC6
- removed U8: DAC8552, ICs:DAC8552
- removed XTAL1: ABM8-12.000MHZ-B2-T, CRYSTALS:ABM8-12.000MHZ-B2-T
- added FB1: 150R 100MHz, INDUCTORS:ILB1206ER151V
- added OSC1: 33MHz, CRYSTALS:KC2016Z33.0000C15XXK
- added R126, R130, R137, R138, R139, R140, R141, R142, R143, R144, R145, R146, R147: 10k, r_0603:ERJ3EKF1002V
- added R148, R149: 180k, r_0603:CRCW0603180KFKEA
- C1, C10, C11, C12, C13, C14, C15, C16, C17, C8, C9: value 100nF 50V -> 100nF 16V; device CAPACITORS:VJ0603Y104KXACW1BC -> CAPACITORS:CL10B104KO8WPNC; FARNELL 2407338 -> (none); PRICE_PER 0.0085 -> (none); VALUE 100nF 50V -> (none)
- C2: value 100nF 50V -> 10uF 25V; device CAPACITORS:VJ0603Y104KXACW1BC -> c_1206:C1206C106K3RACAUTO; FARNELL 2407338 -> (none); PRICE_PER 0.0085 -> (none); VALUE 100nF 50V -> (none)
- C26, C27, C28: value 10uF 16V -> 100nF 16V; device CAPACITORS:MC1206B106K160CT -> CAPACITORS:CL10B104KO8WPNC
- C29: value 100nF 50V -> 100nF 16V; device CAPACITORS:VJ0603Y104KXACW1BC -> CAPACITORS:CL10B104KO8WPNC
- C30: value 470pF 25V -> 100nF 16V; device CAPACITORS:06035A471KAT2A -> CAPACITORS:CL10B104KO8WPNC
- C31, C33, C35: value 100nF 50V -> 100nF 16V; device CAPACITORS:VJ0603Y104KXACW1BC -> CAPACITORS:CL10B104KO8WPNC; VALUE 100nF 50V -> (none)
- C32: value 10pF 100V -> 100nF 16V; device CAPACITORS:06031A100FAT2A -> CAPACITORS:CL10B104KO8WPNC
- C36: value 10uF 16V -> 10uF 6.3V; device CAPACITORS:MC1206B106K160CT -> c_0603:CL10A106KQ8NNWC
- C37: value 100nF 50V -> 10uF 6.3V; device CAPACITORS:VJ0603Y104KXACW1BC -> c_0603:CL10A106KQ8NNWC; FARNELL 2407338 -> (none); PRICE_PER 0.0085 -> (none); VALUE 100nF 50V -> (none)
- C39: value 100nF 50V -> 33pF 10V; device CAPACITORS:VJ0603Y104KXACW1BC -> c_0603:C0603C330J8GAC7867
- CN1: value 5X2HEADER -> 2.1mm DC Jack; device CONNECTORs:5X2HEADER -> CONNECTORs:PJ-202AH
- CN2: value MUSB-05-S-B-SM-A -> USB C CON; device CONNECTORs:MUSB-05-S-B-SM-A -> CONNECTORs:12401832E402A
- CN3: value 1X2_HEADER -> 2X6; device CONNECTORs:1X2_HEADER -> CONNECTORs:TSM-103-03-T-DV
- L3: value 2.2uH 3.5A -> 1uH; device INDUCTORS:SRN5040-2R2Y -> INDUCTORS:CIGT252010EH1R0MNE
- R3: value 10K -> 10k; device RESISTORS:CRCW060310K0FKEA -> r_0603:ERJ3EKF1002V; FARNELL 1469748 -> (none); PRICE_PER 0.0095 -> (none); VALUE 10K -> (none)
- U1: value 93LC56B-I/SN -> TCD2565BFG; device ICs:93LC56B-I/SN -> ICs:TCD2565BFG
- U18: value LMH6639MF -> T8Q144C4; device ICs:LMH6639MF -> ICs:T8Q144C4
- U2: value EP4CE6E22C8N -> FT232H; device ICs:EP4CE6E22C8N -> ICs:FT232HQ
- U4: value MCP1416 -> W25Q128JV; device ICs:MCP1416T -> ICs:W25Q128JVSIQ
- U5: value TPS562209 -> TPS62065; device ICs:TPS562209DDCT -> ICs:TPS62065DSGR
Connections:
- removed net 12V: C101.2, C28.2, C43.2, C44.2, C45.2, C46.2, C47.2, C50.2, C60.2, C61.2, C65.2, C81.2, C82.2, C83.2, C87.2, C99.2, FB7.1, L4.1, L5.2, L7.1, R16.2, U13.EN, U13.VIN, U14.SF, U14.V+, U16.VIN, U17.SF, U17.V+, U18.SF, U18.V+, U19.EN, U19.VIN, U21.SF, U21.V+, U24.EN, U24.VIN, U5.EN, U5.VIN
- removed net 12VMTR: C90.2, C95.1, C97.2, C98.2, L7.2, R43.1, U25.VMA, U25.VMB
- removed net 1V2: C1.2, C10.2, C2.2, C26.2, C27.2, C3.2, C4.2, C5.2, C6.2, C7.2, C8.2, C9.2, L3.2, R12.2, U19.VOS, U2A.VCCD_PLL, U2A.VCCINT
- removed net 2V5: C11.2, C12.2, C48.2, C49.2, L2.2, R15.2, U13.VOS, U2A.VCCA
- removed net 5V: C31.2, C33.2, C34.2, C35.2, C71.2, C72.2, C86.2, C88.2, C89.2, C94.2, C96.2, L6.2, R22.1, R35.2, U10.VCC, U11.VCC, U23.AVDD, U24.VOS, U4.VCC, U6.VCC, U8.VDD, U9.VCC
- removed net 5VUSB: C113.2, C114.2, CN2.5V, U7.VBUS
- removed net 794984: R4.1, U3.DATA
- removed net ADC0_CS: U23.!CS, U2C.IO15
- removed net ADC0_SCLK: U23.SCLK, U2C.IO14
- removed net ADC0_SDO: U23.SDO, U2C.IO13
- removed net ADC_IN: R18.2, R32.1, TP4.P$1, U21.OUT
- removed net ADC_VREF: C84.2, C85.2, TP5.P$1, U14.-, U14.OUT, U23.REF
- removed net ASDO: U2B.ASDO, U3.ASDI
- removed net CCD_CP: U10.A, U2D.IO17
- removed net CCD_P1: U2D.IO25, U4.IN
- removed net CCD_P2: U2D.IO26, U6.IN
- removed net CCD_RS: U11.A, U2D.IO18
- removed net CCD_SH: U2D.IO16, U9.A
- removed net CLK_100M: U20.OUT, U2B.CLK1
- removed net CONF_DN: R3.2, U2G.CNFIG_DN
- removed net DAC0_SCLK: U2C.IO11, U8.SCLK
- removed net DAC0_SDIN: U2C.IO10, U8.DIN
- removed net DAC0_SYNC: U2C.IO12, U8.!SYNC
- removed net DATA0: R4.2, U2B.DATA0
- removed net DCLK: U2B.DCLK, U3.DCLK
- removed net FT_AC_8: U12.ACBUS8, U2E.IO34
- removed net FT_AC_9: U12.ACBUS9, U2E.IO33
- removed net FT_CLK: U12.ACBUS5, U2F.CLK7
- removed net FT_D0: U12.D0, U2F.IO49
- removed net FT_D1: U12.D1, U2F.IO48
- removed net FT_D2: U12.D2, U2F.IO47
- removed net FT_D3: U12.D3, U2F.IO46
- removed net FT_D4: U12.D4, U2F.IO45
- removed net FT_D5: U12.D5, U2F.IO44
- removed net FT_D6: U12.D6, U2F.IO43
- removed net FT_D7: U12.D7, U2F.IO42
- removed net FT_EE_CLK: R27.1, U1.CLK, U12.EECLK
- removed net FT_EE_CS: R28.1, U1.CS, U12.EECS
- removed net FT_EE_DI: R30.2, U1.DI, U12.EEDATA
- removed net FT_NRST: R29.1, U12.!RESET, U2E.IO32
- removed net FT_OE: U12.ACBUS6, U2E.IO36
- removed net FT_PWRSAV: R50.1, U12.PWRSAV#, U2E.IO35
- removed net FT_RD: U12.RD#, U2E.IO39
- removed net FT_RXF: U12.RXF#, U2F.IO41
- removed net FT_SIWU: R37.1, U12.SIWU#, U2E.IO37
- removed net FT_TXE: U12.TXE#, U2E.IO40
- removed net FT_WR: U12.WR#, U2E.IO38
- removed net INIT_DONE: R6.2, U2G.IO52
- removed net LED0: R46.2, U2I.IO81
- removed net LED0_PWM: U16.CTRL, U2B.IO8
- removed net LED1: R47.2, U2I.IO82
- removed net LED2: R48.2, U2I.IO83
- removed net LED3: R49.2, U2I.IO84
- removed net LED_IN: CN3.2, R33.2, U16.FB
- removed net LED_OUT: C62.2, C63.2, CN3.1, D12.K
- removed net MTR_A1: CN4.4, U25.AOUT1
- removed net MTR_A2: CN4.3, U25.AOUT2
- removed net MTR_B1: CN4.1, U25.BOUT1
- removed net MTR_B2: CN4.2, U25.BOUT2
- removed net MTR_DECAY: U25.DECAY, U2E.IO28
- removed net MTR_DIR: U25.DIR, U2E.IO27
- removed net MTR_M0: U25.M0, U2D.IO22
- removed net MTR_M1: U25.M1, U2D.IO21
- removed net MTR_M2: U25.M2, U2D.IO20
- removed net MTR_NEN: U25.!ENABLE, U2D.IO24
- removed net MTR_NFLT: U25.!FAULT, U2E.IO29
- removed net MTR_NHOME: U25.!HOME, U2D.IO19
- removed net MTR_NRST: U25.!RESET, U2E.IO31
- removed net MTR_NSLP: U25.!SLEEP, U2E.IO30
- removed net MTR_STEP: U25.STEP, U2D.IO23
- removed net N$10: R21.1, U8.VOUT_A
- removed net N$11: C32.2, C36.2, C39.2, R20.2, TP2.P$1, U17.+
- removed net N$12: R20.1, U8.VOUT_B
- removed net N$13: U11.Q, U15.RS
- removed net N$14: C29.1, U5.VBST
- removed net N$15: L2.1, U13.SW
- removed net N$16: R14.2, R15.1, U13.FB
- removed net N$17: C40.2, C41.2, C42.2, R21.2, TP7.P$1, U14.+
- removed net N$18: L3.1, U19.SW
- removed net N$19: U15.SH, U9.Q
- removed net N$20: R11.2, R12.1, U19.FB
- removed net N$21: C29.2, L1.1, U5.SW
- removed net N$22: R10.1, R13.1, U5.VFB
- removed net N$23: TP1.P$1, U15.OS, U18.+
- removed net N$24: U15.1, U4.OUT
- removed net N$25: U15.2, U15.2B, U6.OUT
- removed net N$26: C66.2, C67.2, FB7.2, U15.OD
- removed net N$27: C68.2, C69.2, C70.2, R22.2, U8.VREF
- removed net N$28: R25.2, U23.AIN1P
- removed net N$29: R23.2, U23.AIN1GND
- removed net N$30: C38.2, U12.VCCA
- removed net N$31: C73.1, U22.BOOT
- removed net N$32: C37.2, U12.VCCCORE
- removed net N$33: C73.2, D4.K, L5.1, U22.PH
- removed net N$34: C30.2, R32.2, U23.AIN0P
- removed net N$35: R38.2, R39.1, U22.EN
- removed net N$36: R31.2, U12.REF
- removed net N$37: R26.1, R30.1, U1.DO
- removed net N$38: C78.2, U22.SS
- removed net N$39: C30.1, R24.2, U23.AIN0GND
- removed net N$40: L6.1, U24.SW
- removed net N$41: C59.2, U12.XCSO, XTAL1.P$1
- removed net N$42: C58.2, U12.XCSI, XTAL1.P$2
- removed net N$43: R35.1, R36.2, U24.FB
- removed net N$45: C91.2, R41.2, U25.V3P3OUT
- removed net N$46: R41.1, R42.2, U25.AVREF, U25.BVREF
- removed net N$47: C95.2, R43.2, U25.VCP
- removed net N$48: C80.2, R40.2, U22.COMP
- removed net N$49: C79.2, R40.1
- removed net N$50: R16.1, R17.2, U22.VSNS
- removed net N$51: C93.2, U25.CP1
- removed net N$52: C93.1, U25.CP2
- removed net N$53: D1.A, R46.1
- removed net N$54: R45.2, U25.ISENA
- removed net N$55: D2.A, R47.1
- removed net N$56: D3.A, R48.1
- removed net N$57: D5.A, R49.1
- removed net N$58: R44.2, U25.ISENB
- removed net N$59: C64.2, U16.COMP
- removed net N$6: R18.1, R19.2, U21.-
- removed net N$64: D12.A, L4.2, U16.SW
- removed net N$7: TP3.P$1, U17.-, U17.OUT, U21.+
- removed net N$9: R19.1, TP6.P$1, U18.-, U18.OUT
- removed net NCE: R5.2, U2B.NCE
- removed net NCONFIG: R2.2, U2B.NCONFIG
- removed net NCSO: U2B.NCSO, U3.NCS
- removed net NSTATUS: R1.2, U2B.NSTATUS
- removed net TCLK: CN1.1, R9.2, U2B.TCLK
- removed net TDI: CN1.5, R7.1, U2B.TDI
- removed net TDO: CN1.2, U2B.TDO
- removed net TMS: CN1.3, R8.1, U2B.TMS
- removed net USB_IN_N: CN2.D-, U7.D+_IN
- removed net USB_IN_P: CN2.D+, U7.D-_IN
- removed net USB_N: U12.D-, U7.D+_OUT
- removed net USB_P: U12.D+, U7.D-OUT
- removed net VDDD: C75.2, C76.2, C77.2, CN5.V+, R39.2, U22.VIN
- removed net VPHY: C56.2, FB3.2, U12.VPHY
- removed net VPLL: C55.2, FB2.2, U12.VPLL
- new net FLS_NHOLD: R138.1, U4.!HOLD!/IO3
- new net FLS_SPI_CLK: R144.1, U18.GPIOL_01_CCK, U4.SCK
- new net FLS_SPI_MISO: U18.GPIOL_09_CDI1, U4.SO/IO1
- new net FLS_SPI_MOSI: U18.GPIOL_08_CDI0, U4.SI/IO0
- new net FLS_SPI_NCS: R142.1, U18.GPIOL_00_SS_N, U4.!CE
- new net FPGA_CBUS_0: R141.1, U18.GPIOR_151_CBUS0
- new net FPGA_CBUS_1: R140.1, U18.GPIOR_150_CBUS1
- new net FPGA_CBUS_2: R139.1, U18.GPIOR_149_CBUS2
- new net FPGA_CDONE: R147.1, U18.CDONE
- new net FPGA_CLK_33M: OSC1.OUT, U18.GPIOR_157_PLLIN
- new net FPGA_CSI: R145.1, U18.GPIOL_04_CSI
- new net FPGA_JTAG_TCK: CN3.2, R3.1, U18.TCK
- new net FPGA_JTAG_TDI: CN3.4, U18.TDI
- new net FPGA_JTAG_TDO: CN3.6, R130.1, U18.TDO
- new net FPGA_JTAG_TMS: CN3.5, U18.TMS
- new net FPGA_NCRST: R146.1, U18.CRESET_N
- new net FPGA_NTEST: R143.1, U18.GPIOR_158_TEST_N
- new net FPGA_SPI_CLK: U18.GPIOR_86
- new net FPGA_SPI_DATA: U18.GPIOR_85
- new net FPGA_SPI_NCS: U18.GPIOR_87_CDI29
- new net GPIOB_CN0: U18.GPIOB_CLKN0
- new net GPIOB_CP0: U18.GPIOB_CLKP0
- new net GPIOB_N0: U18.GPIOB_RXN00
- new net GPIOB_N10: U18.GPIOB_RXN10
- new net GPIOB_N12: U18.GPIOB_RXN12_EXTFB0
- new net GPIOB_N2: U18.GPIOB_RXN02
- new net GPIOB_N3: U18.GPIOB_RXN03
- new net GPIOB_N7: U18.GPIOB_RXN07
- new net GPIOB_P0: U18.GPIOB_RXP00
- new net GPIOB_P10: U18.GPIOB_RXP10
- new net GPIOB_P12: U18.GPIOB_RXP12_EXTFB0
- new net GPIOB_P2: U18.GPIOB_RXP02
- new net GPIOB_P3: U18.GPIOB_RXP03
- new net GPIOB_P7: U18.GPIOB_RXP07
- new net GPIOB_TN0: U18.GPIOB_TXN00
- new net GPIOB_TN11: U18.GPIOB_TXN11
- new net GPIOB_TN2: U18.GPIOB_TXN02
- new net GPIOB_TN4: U18.GPIOB_TXN04
- new net GPIOB_TN6: U18.GPIOB_TXN06
- new net GPIOB_TN9: U18.GPIOB_TXN09
- new net GPIOB_TP0: U18.GPIOB_TXP00
- new net GPIOB_TP11: U18.GPIOB_TXP11
- new net GPIOB_TP2: U18.GPIOB_TXP02
- new net GPIOB_TP4: U18.GPIOB_TXP04
- new net GPIOB_TP6: U18.GPIOB_TXP06
- new net GPIOB_TP9: U18.GPIOB_TXP09
- new net GPIOL_12: U18.GPIOL_12_CDI2
- new net GPIOL_13: U18.GPIOL_13_CDI3
- new net GPIOL_20: U18.GPIOL_20_CTRL0_CDI4
- new net GPIOL_21: U18.GPIOL_21_CTRL1_CDI5
- new net GPIOL_22: U18.GPIOL_22_CTRL2
- new net GPIOL_24: U18.GPIOL_24_CLK0
- new net GPIOL_25: U18.GPIOL_25_CLK1
- new net GPIOL_31: U18.GPIOL_31_CLK7_CDI6
- new net GPIOL_32: U18.GPIOL_32_CTRL4_CDI7
- new net GPIOL_40: U18.GPIOL_40_CDI8
- new net GPIOL_41: U18.GPIOL_41_CDI9
- new net GPIOL_46: U18.GPIOL_46
- new net GPIOL_53: U18.GPIOL_53_CDI10
- new net GPIOL_54: U18.GPIOL_54_CDI11
- new net GPIOL_64: U18.GPIOL_64
- new net GPIOL_65: U18.GPIOL_65
- new net GPIOL_66: U18.GPIOL_66_CDI12
- new net GPIOL_67: U18.GPIOL_67_CDI13
- new net GPIOL_68: U18.GPIOL_68
- new net GPIOL_69: U18.GPIOL_69_CBSEL1
- new net GPIOL_70: U18.GPIOL_70_CBSEL0
- new net GPIOL_71: U18.GPIOL_71_NSTATUS
- new net GPIOL_72: U18.GPIOL_72_EXTFB0_CDI14
- new net GPIOL_73: U18.GPIOL_73_EXTFB1_CDI15
- new net GPIOL_74: U18.GPIOL_74_PLLIN0
- new net GPIOL_75: U18.GPIOL_75_PLLIN1
- new net GPIOR_104: U18.GPIOR_104_CDI25
- new net GPIOR_105: U18.GPIOR_105_CDI24
- new net GPIOR_112: U18.GPIOR_112_CDI23
- new net GPIOR_113: U18.GPIOR_113_CDI22
- new net GPIOR_116: U18.GPIOR_116_CTRL15
- new net GPIOR_117: U18.GPIOR_117_CTRL14
- new net GPIOR_122: U18.GPIOR_122_CLK13_CDI21
- new net GPIOR_123: U18.GPIOR_123_CLK12_CDI20
- new net GPIOR_125: U18.GPIOR_125_CLK10
- new net GPIOR_128: U18.GPIOR_128_CTRL11
- new net GPIOR_129: U18.GPIOR_129_CTRL10
- new net GPIOR_132: U18.GPIOR_132_CDI19
- new net GPIOR_133: U18.GPIOR_133_CDI18
- new net GPIOR_135: U18.GPIOR_135_CDI17
- new net GPIOR_136: U18.GPIOR_136_CDI16
- new net GPIOR_138: U18.GPIOR_138
- new net GPIOR_139: U18.GPIOR_139
- new net GPIOR_154: U18.GPIOR_154
- new net GPIOR_155: U18.GPIOR_155
- new net GPIOR_76: U18.GPIOR_76_PLLIN0
- new net GPIOR_77: U18.GPIOR_77_PLLIN1
- new net GPIOR_78: U18.GPIOR_78_EXTFB0_CDI31
- new net GPIOR_79: U18.GPIOR_79_EXTFB1_CDI30
- new net GPIOR_80: U18.GPIOR_80
- new net GPIOR_81: U18.GPIOR_81_MREFCLK
- new net GPIOR_82: U18.GPIOR_82
- new net GPIOR_83: U18.GPIOR_83
- new net GPIOR_84: U18.GPIOR_84
- new net GPIOR_88: U18.GPIOR_88_CDI28
- new net GPIOR_94: U18.GPIOR_94_CDI27
- new net GPIOR_95: U18.GPIOR_95_CDI26
- new net N$1: C1.2, C2.2, FB1.2, U1.OD
- new net N$145: R126.2, U18.REF_RES
- new net N$2: FB1.1
- new net N$3: L3.1, U5.SW
- new net N$4: C39.1, R148.1, R149.2, U5.FB
- new net PWR_FPGA_1V2: C10.2, C11.2, C12.2, C13.2, C14.2, C15.2, C16.2, C17.2, C26.2, C37.2, C39.2, C8.2, C9.2, L3.2, R148.2, U18.VCC, U18.VCCA_BR, U18.VCCA_TL, U18.VCCA_TR
- net 3V3: now also C27.2, C28.1, C29.2, C30.2, C31.2, C32.2, C33.2, C35.2, C36.2, CN3.1, OSC1.!ST, OSC1.VCC, R130.2, R137.2, R138.2, R139.2, R140.2, R141.2, R142.2, R143.2, R144.2, R145.2, R146.2, R147.2, R3.2, U18.VCCIO1A, U18.VCCIO1B, U18.VCCIO1C_1D, U18.VCCIO1E, U18.VCCIO3A, U18.VCCIO3B_3C, U18.VCCIO3D, U18.VCCIO3E, U18.VCCIO4A, U18.VCCIO4B, U4.VCC, U5.EN, U5.VIN; no longer C103.2, C104.2, C13.2, C14.2, C15.2, C16.2, C17.2, C18.2, C19.2, C20.2, C21.2, C22.2, C23.2, C24.2, C25.2, C51.2, C52.2, C53.2, C54.2, C57.2, C74.2, C92.2, CN1.8, CN1.9, FB2.1, FB3.1, L1.2, R1.1, R10.2, R2.1, R26.2, R27.2, R28.2, R29.2, R3.1, R37.2, R50.2, R6.1, R7.2, R8.2, U1.ORG, U1.V+, U12.VCCD, U12.VCCIO, U12.VREGIN, U20.!ST, U20.VCC, U23.DVDD, U2A.VCCIO1, U2A.VCCIO2, U2A.VCCIO3, U2A.VCCIO4, U2A.VCCIO5, U2A.VCCIO6, U2A.VCCIO7, U2A.VCCIO8, U2G.MSEL0, U2G.MSEL2, U3.VCC
- net GND: now also C28.2, C29.1, C30.1, CN3.3, OSC1.GND, R126.1, R149.1, U1.SS, U18.GND, U5.MODE; no longer C101.1, C103.1, C104.1, C113.1, C114.1, C18.1, C19.1, C20.1, C21.1, C22.1, C23.1, C24.1, C25.1, C28.1, C3.1, C34.1, C38.1, C39.1, C4.1, C40.1, C41.1, C42.1, C43.1, C44.1, C45.1, C46.1, C47.1, C48.1, C49.1, C5.1, C50.1, C51.1, C52.1, C53.1, C54.1, C55.1, C56.1, C57.1, C58.1, C59.1, C6.1, C60.1, C61.1, C62.1, C63.1, C64.1, C65.1, C66.1, C67.1, C68.1, C69.1, C7.1, C70.1, C71.1, C72.1, C74.1, C75.1, C76.1, C77.1, C78.1, C79.1, C80.1, C81.1, C82.1, C83.1, C84.1, C85.1, C86.1, C87.1, C88.1, C89.1, C90.1, C91.1, C92.1, C94.1, C96.1, C97.1, C98.1, C99.1, CN1.10, CN1.6, CN2.GND, CN2.SHIELD, CN5.GND, D1.K, D2.K, D3.K, D4.A, D5.K, R11.1, R13.2, R14.1, R17.1, R23.1, R24.1, R25.1, R31.1, R33.1, R36.1, R38.1, R42.1, R44.1, R45.1, R5.1, R9.1, TP8.P$1, U1.GND, U10.GND, U11.GND, U12.GND, U12.TEST, U13.AGND, U13.PGND, U14.V-, U15.SS, U16.GND, U17.V-, U18.V-, U19.AGND, U19.PGND, U20.GND, U21.V-, U22.GND, U23.CHSEL, U23.GND, U23.PDEN, U23.REFGND, U24.AGND, U24.PGND, U25.GND, U2A.GND, U2G.MSEL1, U3.GND, U6.GND, U7.GND, U8.GND, U9.GND, XTAL1.GND
- net N$8: now also R137.1, U4.!WP!/IO2; no longer U10.Q, U15.CP
Other:
- note added: "2023.06.28 - GSWDH LTD. MOON CONTROLLER REVISION 1.0.0 DESIGN BY GEORGE WALLER AT GSWDH LTD. GEORGEWALLER@GSWDH.CO.UK CONFIDENTIAL. FOR THE INTENDED READER ONLY."
- note added: "UNCONTROLLED WHEN PRINTED"

Commit message: Progress
Parts:
- removed CN3: 2X6, CONNECTORs:TSM-103-03-T-DV
- added C18, C19, C21, C23, C24, C3, C34, C4, C6: 0.1uF 16V, c_0402:0402YC104KAT2A
- added C20, C25, C5: 220pF 25V, c_0402:04023A221FAT2A
- added C22, C38, C7: NO FIT, c_0402:C0402C100J3GACAUTO
- added CN4: 8 PIN FFC, CONNECTORs:SFV8R-1STBE1HLF
- added R1, R5, R8: 100R, r_0402:RC0402FR-10100RL
- added R10, R4, R7: 680R, r_0402:RC0402FR-07680RL
- added R2, R6, R9: 330R, r_0402:RC0402FR-07330RL
- added U10, U6, U8: LT1806, ICs:LT1806CS6#TRMPBF
- added U11, U12, U13, U14, U15: SN74LVC2G17, ICs:SN74LVC2G17DBVR
- added U3, U7, U9: ADS7056, ICs:ADS7056IRUGR
Connections:
- net FPGA_CBUS_0 renamed FPGA_CONF_CBUS_0
- net FPGA_CBUS_1 renamed FPGA_CONF_CBUS_1
- net FPGA_CBUS_2 renamed FPGA_CONF_CBUS_2
- net FPGA_CDONE renamed FPGA_CONF_CDONE
- net FPGA_NTEST renamed FPGA_CONF_NTEST
- removed net 3V3: C27.2, C28.1, C29.2, C30.2, C31.2, C32.2, C33.2, C35.2, C36.2, CN3.1, OSC1.!ST, OSC1.VCC, R130.2, R137.2, R138.2, R139.2, R140.2, R141.2, R142.2, R143.2, R144.2, R145.2, R146.2, R147.2, R3.2, U18.VCCIO1A, U18.VCCIO1B, U18.VCCIO1C_1D, U18.VCCIO1E, U18.VCCIO3A, U18.VCCIO3B_3C, U18.VCCIO3D, U18.VCCIO3E, U18.VCCIO4A, U18.VCCIO4B, U4.VCC, U5.EN, U5.VIN
- removed net FPGA_CSI: R145.1, U18.GPIOL_04_CSI
- removed net FPGA_NCRST: R146.1, U18.CRESET_N
- new net ADC_OS1_SPI_MISO: U9.MISO
- new net ADC_OS1_SPI_NCS: U9.!CS
- new net ADC_OS1_SPI_SCLK: U9.SCLK
- new net ADC_OS2_SPI_MISO: U7.MISO
- new net ADC_OS2_SPI_NCS: U7.!CS
- new net ADC_OS2_SPI_SCLK: U7.SCLK
- new net ADC_OS3_SPI_MISO: U3.MISO
- new net ADC_OS3_SPI_NCS: U3.!CS
- new net ADC_OS3_SPI_SCLK: U3.SCLK
- new net FPGA_CONF_CSI: CN4.6, R145.1, U18.GPIOL_04_CSI
- new net FPGA_CONF_NCRST: CN4.7, R146.1, U18.CRESET_N
- new net N$10: U1.2B
- new net N$11: U1.SH1
- new net N$12: U1.SH2A
- new net N$13: U1.SH2B
- new net N$14: U1.SH3
- new net N$15: U1.CP
- new net N$16: U1.RS
- new net N$17: U1.TG
- new net N$18: U1.SW
- new net N$19: C20.2, R5.2, U7.AINP
- new net N$20: C22.2, R5.1, R7.2, U8.OUT
- new net N$21: C22.1, R6.2, R7.1, U8.-
- new net N$22: C25.2, R8.2, U9.AINP
- new net N$23: C38.2, R10.2, R8.1, U10.OUT
- new net N$24: C38.1, R10.1, R9.2, U10.-
- new net N$5: C7.2, R1.1, R4.2, U6.OUT
- new net N$6: C7.1, R2.2, R4.1, U6.-
- new net N$7: U1.1A
- new net N$9: U1.2A
- new net PWR_ANA_10V: C21.2, C34.2, C6.2, FB1.1, U10.V+, U6.V+, U8.V+
- new net PWR_ANA_3V3: C18.2, C23.2, C3.2, U3.AVDD, U7.AVDD, U9.AVDD
- new net PWR_SYS_3V3: C19.2, C24.2, C27.2, C28.1, C29.2, C30.2, C31.2, C32.2, C33.2, C35.2, C36.2, C4.2, CN4.1, OSC1.!ST, OSC1.VCC, R130.2, R137.2, R138.2, R139.2, R140.2, R141.2, R142.2, R143.2, R144.2, R145.2, R146.2, R147.2, R3.2, U18.VCCIO1A, U18.VCCIO1B, U18.VCCIO1C_1D, U18.VCCIO1E, U18.VCCIO3A, U18.VCCIO3B_3C, U18.VCCIO3D, U18.VCCIO3E, U18.VCCIO4A, U18.VCCIO4B, U3.DVDD, U4.VCC, U5.EN, U5.VIN, U7.DVDD, U9.DVDD
- new net SEN_OFFSET_OS1: U10.+
- new net SEN_OFFSET_OS2: U8.+
- new net SEN_OFFSET_OS3: U6.+
- new net SEN_SIG_OS1: R9.1, U1.OS1
- new net SEN_SIG_OS2: R6.1, U1.OS2
- new net SEN_SIG_OS3: R2.1, U1.OS3
- net FPGA_JTAG_TCK: now also CN4.3; no longer CN3.2
- net FPGA_JTAG_TDI: now also CN4.2; no longer CN3.4
- net FPGA_JTAG_TDO: now also CN4.5; no longer CN3.6
- net FPGA_JTAG_TMS: now also CN4.4; no longer CN3.5
- net GND: now also C18.1, C19.1, C20.1, C21.1, C23.1, C24.1, C25.1, C3.1, C34.1, C4.1, C5.1, C6.1, CN4.8, U10.V-, U3.AINM, U3.GND, U6.V-, U7.AINM, U7.GND, U8.V-, U9.AINM, U9.GND; no longer CN3.3
- net N$2: now also C5.2, R1.2, U3.AINP; no longer FB1.1
Other:
- moved on the sheet: C1, C2, FB1, R130, R3, U1

Commit message: Smaller form factor
Parts:
- removed CN1: 2.1mm DC Jack, CONNECTORs:PJ-202AH
- added C40, C41, C44, C45, C46, C47, C48, C49, C50, C51: 0.1uF 16V, c_0603:0603YC104JAZ2A
- added C42, C43: 10pF 100V, c_0603:06031A100B4T2A
- added FB2: 150R 100MHz, INDUCTORS:ILB1206ER151V
- added R11: 12k, RESISTORS:CRCW060312K0FKEA
- added R12, R13, R14: 10k, r_0603:ERJ3EKF1002V
- added R15: 2.2k, r_0603:CRCW06032K20FKEA
- added U16: USBLC6-2SC6, ICs:USBLC6-2SC6
- added U17: 93LC56B-I/SN, ICs:93LC56B-I/SN
- added U19: DRV8825, ICs:DRV8825PWP
- added XTAL1: 12MHz, CRYSTALS:ABM8-12.000MHZ-B2-T
- CN2: value USB C CON -> USB B; device CONNECTORs:12401832E402A -> CONNECTORs:M701-330442
Connections:
- new net FT_AC5: U2.ACBUS5
- new net FT_AC6: U2.ACBUS6
- new net FT_AC8: U2.ACBUS8
- new net FT_AC9: U2.ACBUS9
- new net FT_D0: U2.D0
- new net FT_D1: U2.D1
- new net FT_D2: U2.D2
- new net FT_D3: U2.D3
- new net FT_D4: U2.D4
- new net FT_D5: U2.D5
- new net FT_D6: U2.D6
- new net FT_D7: U2.D7
- new net FT_NPWRSAV: U2.PWRSAV#
- new net FT_NRD: U2.RD#
- new net FT_NRST: U2.!RESET
- new net FT_NRXF: U2.RXF#
- new net FT_NSIWU: U2.SIWU#
- new net FT_NTXE: U2.TXE#
- new net FT_NWR: U2.WR#
- new net N$25: CN2.D-, U16.D-_IN
- new net N$26: CN2.D+, U16.D+_IN
- new net N$27: CN2.5V, FB2.1
- new net N$28: R11.2, U2.REF
- new net N$29: R12.1, U17.CS, U2.EECS
- new net N$30: R13.1, U17.CLK, U2.EECLK
- new net N$31: R15.2, U17.DI, U2.EEDATA
- new net N$32: R14.1, R15.1, U17.DO
- new net N$33: C42.2, U2.XCSO, XTAL1.P$2
- new net N$34: C43.2, U2.XCSI, XTAL1.P$1
- new net N$35: C51.2, U2.VCCCORE
- new net N$36: C50.2, U2.VCCA
- new net PWR_USB_VBUS: C40.2, FB2.2, U16.VBUS
- new net USB_D_N: U16.D-OUT, U2.D-
- new net USB_D_P: U16.D+_OUT, U2.D+
- net GND: now also C40.1, C41.1, C42.1, C43.1, C44.1, C45.1, C46.1, C47.1, C48.1, C49.1, C50.1, C51.1, CN2.GND, CN2.SHIELD, R11.1, U16.GND, U17.GND, U2.GND, U2.TEST, XTAL1.GND
- net PWR_SYS_3V3: now also C41.2, C44.2, C45.2, C46.2, C47.2, C48.2, C49.2, R12.2, R13.2, R14.2, U17.V+, U2.VCCD, U2.VCCIO, U2.VPHY, U2.VPLL, U2.VREGIN

Commit message: gain through digiport implemented
Parts:
- added C52, C53: 0.1uF 16V, c_0402:0402YC104KAT2A
- added U20: SN74LVC2G17, ICs:SN74LVC2G17DBVR
- added U21: AD5258BRMZ1-R7, ICs:AD5258BRMZ1-R7
Connections:
- net N$11 renamed CCD_SH1
- net N$12 renamed CCD_SH2A
- net N$13 renamed CCD_SH2B
- net N$14 renamed CCD_SH3
- net N$15 renamed CCD_CP
- net N$16 renamed CCD_RS
- net N$17 renamed CCD_TG
- net N$18 renamed CCD_SW
- net N$7 renamed CCD_1A
- new net CCD_2A: U1.2A, U1.2B
- new net N$7: U11B.A, U11C.A
- new net PWR_ANA_5V: C21.2, C34.2, C53.2, C6.2, U10.V+, U21.VDD, U6.V+, U8.V+
- net GND: now also C52.1, C53.1, U21.GND
- net N$10: now also R4.1, U21.W; no longer U1.2B
- net N$6: now also U21.B; no longer R4.1
- net N$9: now also U11B.Q, U11C.Q; no longer U1.2A
- net PWR_ANA_10V: no longer C21.2, C34.2, C6.2, U10.V+, U6.V+, U8.V+
- net PWR_SYS_3V3: now also C52.2, U21.VIO
Other:
- moved on the sheet: C18, C19, C20, C21, C22, C23, C24, C25, C3, C34, C38, C4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
