File: main.sch (EAGLE design)
At the start: 287 parts, among them CN1 DC-012A-D010, CN2 JST GH 10 Pin, CN3 5.8ZSPT, CN4 8 PIN FFC, CN5 MC-118LS-H100, CN7 8 PIN FFC, Q1 GSFP0449, Q2 2SCR586D, Q3 MMBT3904, U1 TPS54302, U10 SN74LVC2G17, U11 SN74LVC2G17, U12 SN74LVC2G17, U13 SN74LVC2G17, U14 SN74LVC2G17, U15 SN74LVC2G17, U16 SN74LVC2G17, U17 SN74LVC2G17, U18 T8Q144C4, U19 SN74LVC2G17, U2 USBLC6-2SC6, U20 R2A20169SA#W5, U21 LM317MDT, U22 LM317MDT, U27 ADS7056, U28 AD5258BRMZ1-R7, U29 COS8092SR, U3 93LC56B-I/SN, U30 ADS7056, U31 AD5258BRMZ1-R7, U32 COS8092SR, U33 LM317MDT, U34 LM317MDT, U35 ADS7056, U36 AD5258BRMZ1-R7, U37 COS8092SR, U4 W25Q128JV, U41 ADS7056, U42 AD5258BRMZ1-R7, U43 COS8092SR, U44 ADS7056, U45 AD5258BRMZ1-R7, U46 COS8092SR, U5 TPS62065, U50 ADS7056, U51 AD5258BRMZ1-R7, U52 COS8092SR, U6 FT2232H, U7 TPS563201, U8 TCD2720BFG, U9 SN74LVC2G17

Commit message: Progress, motor controller remaining
Parts:
- added C64, C65: 0.1uF 16V, c_0402:0402YC104KAT2A
- added C66: 100nF 16V, CAPACITORS:CL10B104KO8WPNC
- added D11, D12, D9: RED LED, OPTO:150060RS75000
- added Q4, Q5: MMBT3906, TRANSISTORs:MMBT3906-7-F
- added R16: 0R, RESISTORS:CRCW06030000Z0EA
- added R17: 12k, r_0402:RC0402FR-0712KL
- added R57: 10k, r_0603:CRCW060310K0FKTA
- added R58, R66: 20k, r_0402:RC0402FR-0720KL
- added R67: 1k, r_0402:RC0402FR-071KL
- added U23: ADC101C027, ICs:ADC101C027CIMKX/NOPB
Connections:
- net FT_CONT_NRXLED renamed LED_FT_CONT_NRXLED
- net FT_CONT_NTXLED renamed LED_FT_CONT_NTXLED
- removed net FPGA_STATUS: D6.K
- removed net N$105: U18.GPIOR_123_CLK12_CDI20
- removed net N$19: C2.A, C7.1, D1.K, D2.K, D4.K, Q1.S, R1.1
- removed net N$92: U18.GPIOR_79_EXTFB1_CDI30
- removed net N$93: U18.GPIOR_80
- removed net N$94: U18.GPIOR_81_MREFCLK
- removed net PROC_SCANNING: D10.K
- new net LED_FPGA_STATUS: D6.K, U18.GPIOR_79_EXTFB1_CDI30
- new net LED_PROC_SCANNING: D10.K, U18.GPIOR_81_MREFCLK
- new net LED_PROC_STATUS: D5.K
- new net LED_USB_ACT: D12.K
- new net N$18: Q4.B, Q5.B, Q5.C, R17.2
- new net N$24: D9.A, R58.1
- new net N$37: D11.A, R66.1
- new net N$38: R57.1, U23.!ALERT
- new net N$47: D12.A, R67.1
- new net PWR_SYS_VIN: C2.A, C7.1, D1.K, D2.K, D4.K, Q1.S, R1.1, R66.2
- net FPGA_CONF_NCRST: now also C66.2
- net GND: now also C64.1, C65.1, C66.1, D11.K, D9.K, R16.1, R17.1, U23.GND
- net LED_PWM_CONT: now also U18.GPIOR_123_CLK12_CDI20
- net POT_I2C1_SCL: now also U23.SCL
- net POT_I2C1_SDA: now also U23.SDA
- net PROC_STATUS: now also U18.GPIOR_80; no longer D5.K
- net PWR_BUS_24V_UNREG: now also R58.2
- net PWR_SYS_3V3: now also C64.2, Q4.E, Q5.E, R57.2, R67.2, U23.VDD
- net TEMP_SEN_A: now also C65.2, Q4.C, U23.AIN
- net TEMP_SEN_B: now also R16.2

Commit message: Bits and pieces
Connections:
- removed net PROC_STATUS: U18.GPIOR_80
- net LED_PROC_STATUS: now also U18.GPIOR_80
Changed lines of the file:
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@@
-</segment>
-</net>
-<net name="PROC_STATUS" class="0">
-<segment>
-<pinref part="U18" gate="G$1" pin="GPIOR_80"/>
-<wire x1="-66.04" y1="-17.78" x2="-33.02" y2="-17.78" width="0.1524" layer="91"/>
-<label x="-63.5" y="-17.78" size="1.778" layer="95"/>
 </segment>
 </net>
@@
 <label x="-114.3" y="-182.88" size="1.778" layer="95"/>
 </segment>
-</net>
+<segment>
+<pinref part="U18" gate="G$1" pin="GPIOR_80"/>
+<wire x1="-66.04" y1="-17.78" x2="-33.02" y2="-17.78" width="0.1524" layer="91"/>
+<label x="-63.5" y="-17.78" size="1.778" layer="95"/>
+</segment>
+</net>

Commit message: New LED PCB formfactor. UART debug added to FPGA for softcore.
Parts:
- added C67: 470uF 25V, CAPACITORS:ECA-1EM471
- added C68: 0.1uF 50V, c_0603:06035C104JAT2A
- added C69, C70: 0.1uF 16V, c_0402:0402YC104KAT2A
- added CN6: JST GH 10 Pin, CONNECTORs:1.25-10PWT
- added D13: B360A-13-F, DIODES:B360A-13-F
- added Q6: IRLML6244, TRANSISTORs:IRLML6244TRPBF
- added R68, R72, R73: 10k, r_0603:CRCW060310K0FKTA
- added R74, R75: 10k, r_0603:ERJ3EKF1002V
- added U24, U25: SCHMITT, ICs:SN74LVC1G17DBVR
Connections:
- removed net N$76: U18.GPIOL_73_EXTFB1_CDI15
- removed net N$77: U18.GPIOL_74_PLLIN0
- removed net N$78: U18.GPIOL_75_PLLIN1
- removed net N$79: U18.GPIOR_76_PLLIN0
- removed net N$80: U18.GPIOR_77_PLLIN1
- new net MTR_PWM: Q6.G, R68.2, U18.GPIOL_73_EXTFB1_CDI15
- new net MTR_SENSE_A: U18.GPIOL_75_PLLIN1, U24.Q
- new net MTR_SENSE_B: U18.GPIOL_74_PLLIN0, U25.Q
- new net MTR_SENSE_IN_A: CN6.3, R72.2, U24.A
- new net MTR_SENSE_IN_B: CN6.2, R73.2, U25.A
- new net N$57: C68.1, CN6.5, CN6.6, CN6.7, D13.A, Q6.D
- new net PROC_UART_RX: CN7.2, R75.1, U18.GPIOR_77_PLLIN1
- new net PROC_UART_TX: CN7.3, R74.1, U18.GPIOR_76_PLLIN0
- net GND: now also C67.K, C69.1, C70.1, CN6.1, Q6.S, R68.1, R72.1, R73.1, U24.GND, U25.GND
- net PWR_SYS_12V: now also C67.A, C68.2, CN6.10, CN6.8, CN6.9, D13.K
- net PWR_SYS_3V3: now also C69.2, C70.2, CN6.4, R74.2, R75.2, U24.VCC, U25.VCC
Other:
- moved on the sheet: C6

Commit message: New formactor
Parts:
- removed C106, C107, C109, C111, C112, C113, C114, C115, C117, C119, C120, C121, C122, C123, C125, C127, C128, C129, C138, C139, C141, C143, C144, C145, C146, C147, C149, C151, C152, C153, C162, C163, C165, C167, C168, C169, C76, C78: 0.1uF 16V, c_0402:0402YC104KAT2A
- removed C108, C116, C124, C140, C148, C164: 220pF 25V, c_0402:04023A221FAT2A
- removed C110, C118, C126, C142, C150, C166: NO FIT, c_0402:C0402C100J3GACAUTO
- removed C61, C62, C63, C71, C72, C73, C74, C75: 100nF 16V, CAPACITORS:CL10B104KO8WPNC
- removed C67: 470uF 25V, CAPACITORS:ECA-1EM471
- removed C77, C79: 10uF 10V, c_0603:0603ZD106KAT2A
- removed C80, C84: 100uF 50V, CAPACITORS:107CKR050M
- removed C81, C83, C85, C87, C89, C91: 0.1uF 50V, c_0603:06035C104JAT2A
- removed C82: 100pF 50V, c_0603:06035A101J4T4A
- removed C86, C88, C92: 1uF 10V, c_0603:C0603C105K8PAC7411
- removed C90: 1uF 16V, c_1206:1206YC105JAT2A
- removed C93, C96, C97: 10uF 10V, c_1206:1206ZC106KAT2A
- removed FB1, FB3: 150R 100MHz, INDUCTORS:ILB1206ER151V
- removed FB2: 600R, INDUCTORS:742792651
- removed Q2: 2SCR586D, TRANSISTORs:2SCR586DGTL
- removed Q3: MMBT3904, TRANSISTORs:MMBT3904-7-F
- removed R126, R139, R140, R141: 10k, r_0603:ERJ3EKF1002V
- removed R25, R29, R31, R33: 430R, r_0402:RC0402FR-07430RL
- removed R28, R30, R32, R34: 110k, r_0402:RC0402FR-07110KL
- removed R35: 20k, r_0603:CRCW060320K0FKEA
- removed R36, R38, R40, R42: 240R, r_0402:RC0402FR-07240RL
- removed R37, R39: 715R, r_0402:RC0402FR-07715RL
- removed R41: 1.69k, r_0402:RC0402FR-071K69L
- removed R43: 390R, r_0402:RC0402FR-07390RL
- removed R44, R45, R46, R56: 2.2k, r_0402:RC0402FR-072K2L
- removed R47, R50, R53, R60, R63, R69: 100R, r_0402:RC0402FR-10100RL
- removed R48, R51, R54, R61, R64, R70: 330R, r_0402:RC0402FR-07330RL
- removed R49, R52, R55, R62, R65, R71: 680R, r_0402:RC0402FR-07680RL
- removed U13, U14, U15, U16, U17, U19: SN74LVC2G17, ICs:SN74LVC2G17DBVR
- removed U18: T8Q144C4, ICs:T8Q144C4
- removed U20: R2A20169SA#W5, ICs:R2A20169SA#W5
- removed U21, U22, U33, U34: LM317MDT, ICs:LM317MDT-TR
- removed U27, U30, U35, U41, U44, U50: ADS7056, ICs:ADS7056IRUGR
- removed U28, U31, U36, U42, U45, U51: AD5258BRMZ1-R7, ICs:AD5258BRMZ1-R7
- removed U29, U32, U37, U43, U46, U52: COS8092SR, ICs:COS8092SRD
- C1, C51: value 100nF 16V -> 1uF 10V; device CAPACITORS:CL10B104KO8WPNC -> c_0402:0402ZD105KAT2A
- C10, C14, C17, C29, C31: value 100nF 16V -> 10uF 6.3V; device CAPACITORS:CL10B104KO8WPNC -> c_0402:GRM155R60J106ME15D
- C11, C12, C13, C15, C16, C26, C27, C28, C30, C32, C60, C66, C8, C9: value 100nF 16V -> 0.1uF 16V; device CAPACITORS:CL10B104KO8WPNC -> c_0402:0402YD104JAT2A
- C18, C19, C20: value 10uF 50V -> 0.1uF 16V; device CAPACITORS:CL21A106KAYNNNE -> c_0402:0402YD104JAT2A
- C2, C6: value 100uF 50V -> 470uF 25V; device CAPACITORS:107CKR050M -> CAPACITORS:ECA-1EM471
- C21: device c_0603:0603YC104JAZ2A -> c_0402:0402YD104JAT2A
- C3: value 100pF 50V -> 10uF 6.3V; device c_0603:06035A101J4T4A -> c_0402:GRM155R60J106ME15D
- C33, C35: value 100nF 16V -> 10uF 6.3V; device CAPACITORS:CL10B104KO8WPNC -> c_0603:CL10A106KQ8NNWC
- C39: value 33pF 10V -> 150pF 25V; device c_0603:C0603C330J8GAC7867 -> c_0402:04023A151JAT2A
- C4: value 10uF 50V -> 0.1uF 16V; device CAPACITORS:C3225X7S1H106M250AB -> c_0402:0402YD104JAT2A
- C40: value 10uF 50V -> 150pF 25V; device CAPACITORS:CL21A106KAYNNNE -> c_0402:04023A151JAT2A
- C41: value 10uF 50V -> 1uF 10V; device CAPACITORS:CL21A106KAYNNNE -> c_0402:0402ZD105KAT2A
- C49: value 100nF 16V -> 2.2uF 6.3V; device CAPACITORS:CL10B104KO8WPNC -> c_0402:C0402C225K9PAC7867
- C5: value 0.1uF 50V -> 0.1uF 16V; device c_0603:06035C104JAT2A -> c_0402:0402YD104JAT2A
- C50: value 10uF 25V -> 1uF 10V; device c_1206:C1206C106K3RACAUTO -> c_0402:0402ZD105KAT2A
- L1: value 15uH 6.5A -> 1uH; device INDUCTORS:MWSA1004S-150MT -> INDUCTORS:CIGT252010EH1R0MNE
- R130, R137, R138, R142, R143, R144, R145, R146, R147, R20, R21, R3, R74, R75: device r_0603:ERJ3EKF1002V -> r_0402:RC0402FR-0710KL
- R148: value 180k -> 36k; device r_0603:CRCW0603180KFKEA -> r_0402:RC0402FR-0736KL
- R149: value 180k -> 62k; device r_0603:CRCW0603180KFKEA -> r_0402:RC0402FR-0762KL
- R15: value 5.23k -> 36k; device r_0603:CRCW06035K23FKEA -> r_0402:RC0402FR-0736KL
- R2: value 51k -> 1.5k; device RESISTORS:CRCW060351K0FKEA -> r_0402:RC0402FR-071K5L
- R22: value 430R -> 62k; device r_0402:RC0402FR-07430RL -> r_0402:RC0402FR-0762KL
- R23: value 10k -> 30k; device r_0603:CRCW060310K0FKTA -> r_0402:RC0402FR-0730KL
- R24: value 110k -> 12k; device r_0402:RC0402FR-07110KL -> r_0402:RC0402FR-0712KL
- R26: value 110k -> 10k; device r_0402:RC0402FR-07110KL -> r_0402:RC0402FR-0710KL
- R27: value 430R -> 10k; device r_0402:RC0402FR-07430RL -> r_0402:RC0402FR-0710KL
- R4: value 100k -> 1.5k; device r_0603:CRCW0603100KFKEB -> r_0402:RC0402FR-071K5L
- U1: value TPS54302 -> Ti60F225C4; device ICs:TPS54302 -> ICs:TI60F225C4
- U10: value SN74LVC2G17 -> W958D8NBYA5I; device ICs:SN74LVC2G17DBVR -> ICs:W958D8NBYA5I
- U11: value SN74LVC2G17 -> TPS70918; device ICs:SN74LVC2G17DBVR -> ICs:TPS70918DBVT
- U12: value SN74LVC2G17 -> AP7335; device ICs:SN74LVC2G17DBVR -> ICs:AP7335-SNG-7
- U8: value TCD2720BFG -> AR0822; device ICs:TCD2720BFG -> ICs:AR0822NPSC10SMTA0
- U9: value SN74LVC2G17 -> TPS62065; device ICs:SN74LVC2G17DBVR -> ICs:TPS62065DSGR
Connections:
- removed net ADC_SPI_MISO_1: U18.GPIOR_84, U27.MISO
- removed net ADC_SPI_MISO_2: U18.GPIOR_87_CDI29, U35.MISO
- removed net ADC_SPI_MISO_3: U18.GPIOR_95_CDI26, U41.MISO
- removed net ADC_SPI_MISO_4: U18.GPIOR_128_CTRL11, U30.MISO
- removed net ADC_SPI_MISO_5: U18.GPIOR_138, U44.MISO
- removed net ADC_SPI_MISO_6: U18.GPIOR_133_CDI18, U50.MISO
- removed net ADC_SPI_NCS_1: U18.GPIOR_83, U27.!CS
- removed net ADC_SPI_NCS_2: U18.GPIOR_85, U35.!CS
- removed net ADC_SPI_NCS_3: U18.GPIOR_94_CDI27, U41.!CS
- removed net ADC_SPI_NCS_4: U18.GPIOR_125_CLK10, U30.!CS
- removed net ADC_SPI_NCS_5: U18.GPIOR_136_CDI16, U44.!CS
- removed net ADC_SPI_NCS_6: U18.GPIOR_132_CDI19, U50.!CS
- removed net ADC_SPI_SCLK_1: U18.GPIOR_86, U27.SCLK
- removed net ADC_SPI_SCLK_2: U18.GPIOR_88_CDI28, U35.SCLK
- removed net ADC_SPI_SCLK_3: U18.GPIOR_104_CDI25, U41.SCLK
- removed net ADC_SPI_SCLK_4: U18.GPIOR_129_CTRL10, U30.SCLK
- removed net ADC_SPI_SCLK_5: U18.GPIOR_139, U44.SCLK
- removed net ADC_SPI_SCLK_6: U18.GPIOR_135_CDI17, U50.SCLK
- removed net CCD_1A1: U8.1A1, U9B.Q
- removed net CCD_1A2: U8.1A2
- removed net CCD_1A3: U11B.Q, U8.1A3
- removed net CCD_1A4: U12B.Q, U8.1A4
- removed net CCD_1A5: U17C.Q, U8.1A5
- removed net CCD_2A1: U8.2A1, U9C.Q
- removed net CCD_2A2: U10C.Q, U8.2A2
- removed net CCD_2A3: U11C.Q, U8.2A3
- removed net CCD_2A4: U19B.Q, U8.2A4
- removed net CCD_2A5: U19C.Q, U8.2A5
- removed net CCD_2B: U10B.Q, U8.2B
- removed net CCD_CP: U13B.Q, U8.CP
- removed net CCD_RS: U13C.Q, U8.RS
- removed net CCD_SH_M1: U15C.Q, U8.SH_M1
- removed net CCD_SH_M2: U15B.Q, U8.SH_M2
- removed net CCD_SH_S1: U14C.Q, U8.SH_S1
- removed net CCD_SH_S2: U16B.Q, U8.SH_S2
- removed net CCD_SH_S3: U14B.Q, U8.SH_S3
- removed net CCD_SH_S4: U16C.Q, U8.SH_S4
- removed net CCD_SIG_1A: U11B.A, U12B.A, U17C.A, U18.GPIOB_RXP03, U9B.A
- removed net CCD_SIG_2A: U10B.A, U10C.A, U11C.A, U18.GPIOB_RXN07, U19B.A, U19C.A, U9C.A
- removed net CCD_SIG_CP: U13B.A, U18.GPIOB_CLKN0
- removed net CCD_SIG_RS: U13C.A, U18.GPIOB_RXP12_EXTFB0
- removed net CCD_SIG_SH_M1: U15C.A, U18.GPIOB_RXP07
- removed net CCD_SIG_SH_M2: U15B.A, U18.GPIOB_TXP06
- removed net CCD_SIG_SH_S1: U14C.A, U18.GPIOB_RXP10
- removed net CCD_SIG_SH_S2: U16B.A, U18.GPIOB_RXP02
- removed net CCD_SIG_SH_S3: U14B.A, U18.GPIOB_RXN10
- removed net CCD_SIG_SH_S4: U16C.A, U18.GPIOB_RXN02
- removed net CCD_SIG_SW: U17B.A, U18.GPIOB_RXN03
- removed net CCD_SIG_TG: U12C.A, U18.GPIOB_RXN12_EXTFB0
- removed net CCD_SW: U17B.Q, U8.SW
- removed net CCD_TG: U12C.Q, U8.TG
- removed net DAC_SPI_MOSI: U18.GPIOL_72_EXTFB0_CDI14, U20.DI
- removed net DAC_SPI_NCS: U18.GPIOL_70_CBSEL0, U20.LD
- removed net DAC_SPI_SCLK: U18.GPIOL_71_NSTATUS, U20.CLK
- removed net FPGA_CONF_CBUS_0: R141.1, U18.GPIOR_151_CBUS0
- removed net FPGA_CONF_CBUS_1: R140.1, U18.GPIOR_150_CBUS1
- removed net FPGA_CONF_CBUS_2: R139.1, U18.GPIOR_149_CBUS2
- removed net FT_CONT_NCTS: U18.GPIOL_32_CTRL4_CDI7, U6.BDBUS3
- removed net FT_CONT_NDCD: U18.GPIOL_31_CLK7_CDI6, U6.BDBUS6
- removed net FT_CONT_NDSR: U18.GPIOL_22_CTRL2, U6.BDBUS5
- removed net FT_CONT_NDTR: U18.GPIOL_40_CDI8, U6.BDBUS4
- removed net FT_CONT_NRI: U18.GPIOL_24_CLK0, U6.BDBUS7
- removed net FT_CONT_NRTS: U18.GPIOL_41_CDI9, U6.BDBUS2
- removed net FT_CONT_PWRSAV: U18.GPIOL_53_CDI10, U6.BCBUS7
- removed net FT_CONT_TXDEN: U18.GPIOL_25_CLK1, U6.BCBUS0
- removed net FT_NPWREN: U18.GPIOL_54_CDI11, U6.!PWREN
- removed net FT_NSUSPEND: U18.GPIOL_20_CTRL0_CDI4, U6.!SUSPEND
- removed net MTR_PWM: Q6.G, R68.2, U18.GPIOL_73_EXTFB1_CDI15
- removed net N$100: R70.1, U52B.-, U52B.OUT
- removed net N$101: U18.GPIOR_113_CDI22
- removed net N$102: U18.GPIOR_116_CTRL15
- removed net N$103: U18.GPIOR_117_CTRL14
- removed net N$104: U18.GPIOR_122_CLK13_CDI21
- removed net N$145: R126.2, U18.REF_RES
- removed net N$21: C49.2, C50.2, FB1.2, U8.OD
- removed net N$22: R22.1, U20.AO1
- removed net N$23: R24.1, U20.AO2
- removed net N$26: R25.1, U20.AO3
- removed net N$27: R26.1, U20.AO4
- removed net N$28: R27.1, U20.AO5
- removed net N$29: R28.1, U20.AO6
- removed net N$30: R29.1, U20.AO7
- removed net N$31: R30.1, U20.AO8
- removed net N$32: R31.1, U20.AO9
- removed net N$33: R32.1, U20.AO10
- removed net N$34: R33.1, U20.AO11
- removed net N$35: R34.1, U20.AO12
- removed net N$36: C81.2, C82.2, FB2.2, Q2.C, Q3.C, R23.2
- removed net N$39: C80.A, C83.2, Q3.B, R23.1, R35.2
- removed net N$40: Q2.B, Q3.E
- removed net N$41: CN5.VBUS, FB3.1
- removed net N$52: R36.1, R37.2, U21.ADJ
- removed net N$53: R38.1, R39.2, U22.ADJ
- removed net N$54: C96.2, R40.1, R41.2, U33.ADJ
- removed net N$55: R42.1, R43.2, U34.ADJ
- removed net N$59: U18.GPIOR_105_CDI24
- removed net N$60: U18.GPIOR_112_CDI23
- removed net N$61: C108.2, R47.2, U27.AINP
- removed net N$62: C110.2, R47.1, R49.2, U29A.OUT
- removed net N$63: C110.1, R48.2, U28.B, U29A.-
- removed net N$64: R49.1, U28.W
- removed net N$65: R48.1, U29B.-, U29B.OUT
- removed net N$66: C116.2, R50.2, U30.AINP
- removed net N$67: C118.2, R50.1, R52.2, U32A.OUT
- removed net N$68: C118.1, R51.2, U31.B, U32A.-
- removed net N$69: R52.1, U31.W
- removed net N$70: R51.1, U32B.-, U32B.OUT
- removed net N$71: C124.2, R53.2, U35.AINP
- removed net N$72: C126.2, R53.1, R55.2, U37A.OUT
- removed net N$73: C126.1, R54.2, U36.B, U37A.-
- removed net N$74: R55.1, U36.W
- removed net N$75: R54.1, U37B.-, U37B.OUT
- removed net N$81: C140.2, R60.2, U41.AINP
- removed net N$82: C142.2, R60.1, R62.2, U43A.OUT
- removed net N$83: C142.1, R61.2, U42.B, U43A.-
- removed net N$84: R62.1, U42.W
- removed net N$85: R61.1, U43B.-, U43B.OUT
- removed net N$86: C148.2, R63.2, U44.AINP
- removed net N$87: C150.2, R63.1, R65.2, U46A.OUT
- removed net N$88: C150.1, R64.2, U45.B, U46A.-
- removed net N$89: R65.1, U45.W
- removed net N$9: C3.1, R15.2, R4.1, U1.FB
- removed net N$90: R64.1, U46B.-, U46B.OUT
- removed net N$91: U18.GPIOR_78_EXTFB0_CDI31
- removed net N$95: U18.GPIOR_82
- removed net N$96: C164.2, R69.2, U50.AINP
- removed net N$97: C166.2, R69.1, R71.2, U52A.OUT
- removed net N$98: C166.1, R70.2, U51.B, U52A.-
- removed net N$99: R71.1, U51.W
- removed net POT_I2C0_SCL: R44.1, U18.GPIOL_65, U28.SCL, U36.SCL, U42.SCL
- removed net POT_I2C0_SDA: R45.1, U18.GPIOL_66_CDI12, U28.SDA, U36.SDA, U42.SDA
- removed net PWR_ANA_10V: C90.2, FB1.1, R40.2, U33.VOUT
- removed net PWR_ANA_3V3: C106.2, C114.2, C122.2, C138.2, C146.2, C162.2, C76.2, C77.2, C78.2, C79.2, C92.2, R42.2, U20.VCC, U20.VREFH, U27.AVDD, U30.AVDD, U34.VOUT, U35.AVDD, U41.AVDD, U44.AVDD, U50.AVDD
- removed net PWR_ANA_5V: C109.2, C112.2, C117.2, C120.2, C125.2, C128.2, C141.2, C144.2, C149.2, C152.2, C165.2, C168.2, C86.2, R36.2, U21.VOUT, U28.VDD, U29A.V+, U31.VDD, U32A.V+, U36.VDD, U37A.V+, U42.VDD, U43A.V+, U45.VDD, U46A.V+, U51.VDD, U52A.V+
- removed net PWR_ANA_UNREG: C84.A, C85.2, C89.2, C91.2, Q2.E, U21.VIN, U33.VIN, U34.VIN
- removed net PWR_BUS_24V_UNREG: C4.2, C5.2, C6.A, CN2.10, CN2.8, CN2.9, FB2.1, Q1.D, R58.2, U1.VIN
- removed net PWR_CLK_5V: C51.2, C60.2, C61.2, C62.2, C63.2, C71.2, C72.2, C73.2, C74.2, C75.2, C88.2, C93.2, C97.2, R38.2, U10A.V+, U11A.V+, U12A.V+, U13A.V+, U14A.V+, U15A.V+, U16A.V+, U17A.V+, U19A.V+, U22.VOUT, U9A.V+
- removed net PWR_FPGA_1V2: C10.2, C11.2, C12.2, C13.2, C14.2, C15.2, C16.2, C17.2, C26.2, C37.2, C39.2, C8.2, C9.2, L3.2, R148.2, U18.VCC, U18.VCCA_BR, U18.VCCA_TL, U18.VCCA_TR
- removed net PWR_SYS_12V: C18.2, C19.2, C20.2, C40.2, C41.2, C42.2, C47.2, C67.A, C68.2, C87.2, CN6.10, CN6.8, CN6.9, D13.K, L1.2, R2.2, U22.VIN, U7.EN, U7.VIN
- removed net PWR_USB_VBUS: C21.2, FB3.2, U2.VBUS
- removed net SEN_OFFSET_OS1: C113.2, R22.2, R24.2, U29A.+
- removed net SEN_OFFSET_OS2: C129.2, R25.2, R26.2, U37A.+
- removed net SEN_OFFSET_OS3: C145.2, R27.2, R28.2, U43A.+
- removed net SEN_OFFSET_OS4: C121.2, R29.2, R30.2, U32A.+
- removed net SEN_OFFSET_OS5: C153.2, R33.2, R34.2, U46A.+
- removed net SEN_OFFSET_OS6: C169.2, R31.2, R32.2, U52A.+
- removed net SEN_SIG_OS1: U29B.+, U8.OS1
- removed net SEN_SIG_OS2: U37B.+, U8.OS2
- removed net SEN_SIG_OS3: U43B.+, U8.OS3
- removed net SEN_SIG_OS4: U32B.+, U8.OS4
- removed net SEN_SIG_OS5: U46B.+, U8.OS5
- removed net SEN_SIG_OS6: U52B.+, U8.OS6
- new net AR_CLK: U1.GPIOB_N_01, U8.EXTCLK
- new net AR_GPIO0: U1.GPIOB_N_02_CDI5, U8.GPIO_0
- new net AR_GPIO1: U1.GPIOB_P_01_EXTFB, U8.GPIO_1
- new net AR_GPIO2: U1.GPIOB_N_07_CLK15_N, U8.GPIO_2
- new net AR_GPIO3: U1.GPIOB_P_02_CDI4, U8.GPIO_3
- new net AR_I2C_SCL: R4.1, U1.GPIOB_P_07_CLK15_P, U8.SCL
- new net AR_I2C_SDA: R2.1, U1.GPIOB_P_08_CLK14_P, U8.SDA
- new net AR_MIPI_CLK_N: U1.GPIOL_N_09_CLK2_N, U8.CLKN
- new net AR_MIPI_CLK_P: U1.GPIOL_P_09_CLK2_P, U8.CLKP
- new net AR_MIPI_D0_N: U1.GPIOL_N_11, U8.DATA0N
- new net AR_MIPI_D0_P: U1.GPIOL_P_11, U8.DATA0P
- new net AR_MIPI_D1_N: U1.GPIOL_N_14, U8.DATA1N
- new net AR_MIPI_D1_P: U1.GPIOL_P_14, U8.DATA1P
- new net AR_MIPI_D2_N: U1.GPIOL_N_16, U8.DATA2N
- new net AR_MIPI_D2_P: U1.GPIOL_P_16, U8.DATA2P
- new net AR_MIPI_D3_N: U1.GPIOL_N_18, U8.DATA3N
- new net AR_MIPI_D3_P: U1.GPIOL_P_18_PLLIN0, U8.DATA3P
- new net AR_NRESET: U1.GPIOB_P_00_PLLIN1, U8.!RESET
- new net AR_XSHUTDOWN: U1.GPIOB_N_00, U8.XSHUTDOWN
- new net MTR_CONT_PWM: Q6.G, R68.2
- new net N$19: R23.1, R24.2, U12.FB
- new net PWR_BUS_UNREG: C42.2, C47.2, C6.A, C68.2, CN2.10, CN2.8, CN2.9, CN6.1, CN6.2, CN6.3, D13.K, Q1.D, R58.2, U7.EN, U7.VIN
- new net PWR_FPGA_0V95: C37.2, C39.2, L3.2, R148.2, U1.VCC, U1.VCCA_BL, U1.VCCA_BR, U1.VCCA_TL, U1.VCCA_TR
- new net PWR_FPGA_1V8: U1.VCCAUX
- new net PWR_MIPI_1V2: R143.2, U1.VCCIO1B
- new net PWR_SEN_1V05D: C17.2, C18.2, C19.2, C20.2, C21.2, C26.2, C29.2, C30.2, C31.2, C32.2, C35.2, C40.2, L1.2, R15.2, U8.DVDD, U8.DVDDCORE, U8.DVDDPHY
- new net PWR_SEN_2V8A: C10.2, C11.2, C12.2, C13.2, C14.2, C15.2, C16.2, C51.2, C60.2, R23.2, U12.VOUT, U8.VAA2V8_ANA, U8.VAA2V8_PIX
- new net PWR_SYS_1V8: C3.2, C4.2, C49.2, C5.2, C8.2, C9.2, R2.2, R4.2, U1.VCCIO4B, U11.VOUT, U8.VDDIO
- net FLS_SPI_CLK: now also U1.GPIOL_N_01_CCK; no longer U18.GPIOL_01_CCK
- net FLS_SPI_MISO: now also R27.1, U1.GPIOL_N_03_CDI1; no longer U18.GPIOL_09_CDI1
- net FLS_SPI_MOSI: now also R26.1, U1.GPIOL_P_03_CDI0; no longer U18.GPIOL_08_CDI0
- net FLS_SPI_NCS: now also U1.GPIOL_P_01_SSL_N; no longer U18.GPIOL_00_SS_N
- net FPGA_CLK_33M: now also U1.GPIOL_P_00_PLLIN0; no longer U18.GPIOR_157_PLLIN
- net FPGA_CONF_CDONE: now also U1.CDONE; no longer U18.CDONE
- net FPGA_CONF_CSI: now also U1.GPIOL_P_02_CSI; no longer U18.GPIOL_04_CSI
- net FPGA_CONF_NCRST: now also U1.CRESET_N; no longer U18.CRESET_N
- net FPGA_CONF_NTEST: now also U1.GPIOL_N_15_TEST_N; no longer U18.GPIOR_158_TEST_N
- net FPGA_JTAG_TCK: now also U1.TCK; no longer U18.TCK
- net FPGA_JTAG_TDI: now also U1.TDI; no longer U18.TDI
- net FPGA_JTAG_TDO: now also U1.TDO; no longer U18.TDO
- net FPGA_JTAG_TMS: now also U1.TMS; no longer U18.TMS
- net FT_CLKOUT: now also U1.GPIOR_N_11_CLK8_N; no longer U18.GPIOB_CLKP0
- net FT_CONT_RX: now also U1.GPIOR_P_11_CLK8_P; no longer U18.GPIOL_21_CTRL1_CDI5
- net FT_CONT_TX: now also U1.GPIOR_P_13; no longer U18.GPIOL_46
- net FT_D0: now also U1.GPIOR_P_17; no longer U18.GPIOB_RXN00
- net FT_D1: now also U1.GPIOR_P_19_PLLIN0; no longer U18.GPIOB_RXP00
- net FT_D2: now also U1.GPIOR_P_12; no longer U18.GPIOB_TXN11
- net FT_D3: now also U1.GPIOR_N_12; no longer U18.GPIOB_TXP02
- net FT_D4: now also U1.GPIOR_P_15; no longer U18.GPIOB_TXN00
- net FT_D5: now also U1.GPIOR_N_15; no longer U18.GPIOB_TXN09
- net FT_D6: now also U1.GPIOR_N_17; no longer U18.GPIOB_TXP09
- net FT_D7: now also U1.GPIOR_N_19; no longer U18.GPIOB_TXN06
- net FT_NOE: now also U1.GPIOR_P_10_CLK9_P; no longer U18.GPIOB_TXP00
- net FT_NRD: now also U1.GPIOR_N_16; no longer U18.GPIOB_TXP04
- net FT_NRST: now also U1.GPIOR_N_10_CLK9_N; no longer U18.GPIOB_TXP11
- net FT_NRXF: now also U1.GPIOR_N_18; no longer U18.GPIOB_TXN04
- net FT_NSIWU: now also U1.GPIOR_N_13; no longer U18.GPIOL_12_CDI2
- net FT_NTXE: now also U1.GPIOR_P_18; no longer U18.GPIOL_13_CDI3
- net FT_NWR: now also U1.GPIOR_P_16; no longer U18.GPIOB_TXN02
- net GND: now also C1.1, C3.1, CN6.10, R22.1, R24.1, U10.VSS, U10.VSSQ, U11.GND, U12.GND, U6.BDBUS3, U6.BDBUS4, U6.BDBUS5, U6.BDBUS6, U8.AGND, U8.GND, U8.SADDR0, U8.SADDR1, U8.SADDR2, U9.GND, U9.MODE; no longer C106.1, C107.1, C108.1, C109.1, C111.1, C112.1, C113.1, C114.1, C115.1, C116.1, C117.1, C119.1, C120.1, C121.1, C122.1, C123.1, C124.1, C125.1, C127.1, C128.1, C129.1, C138.1, C139.1, C140.1, C141.1, C143.1, C144.1, C145.1, C146.1, C147.1, C148.1, C149.1, C151.1, C152.1, C153.1, C162.1, C163.1, C164.1, C165.1, C167.1, C168.1, C169.1, C40.1, C61.1, C62.1, C63.1, C67.K, C71.1, C72.1, C73.1, C74.1, C75.1, C76.1, C77.1, C78.1, C79.1, C80.K, C81.1, C82.1, C83.1, C84.K, C85.1, C86.1, C87.1, C88.1, C89.1, C90.1, C91.1, C92.1, C93.1, C96.1, C97.1, CN6.1, R126.1, R15.1, R35.1, R37.1, R39.1, R41.1, R43.1, U10A.GND, U11A.GND, U12A.GND, U13A.GND, U14A.GND, U15A.GND, U16A.GND, U17A.GND, U18.GND, U19A.GND, U20.GND, U20.VREFL, U27.AINM, U27.GND, U28.A0, U28.A1, U28.GND, U29A.V-, U30.AINM, U30.GND, U31.A0, U31.A1, U31.GND, U32A.V-, U35.AINM, U35.GND, U36.A1, U36.GND, U37A.V-, U41.AINM, U41.GND, U42.A0, U42.GND, U43A.V-, U44.AINM, U44.GND, U45.A1, U45.GND, U46A.V-, U50.AINM, U50.GND, U51.A0, U51.GND, U52A.V-, U8.SS, U9A.GND
- net LED_FPGA_STATUS: no longer U18.GPIOR_79_EXTFB1_CDI30
- net LED_PROC_SCANNING: no longer U18.GPIOR_81_MREFCLK
- net LED_PROC_STATUS: no longer U18.GPIOR_80
- net LED_PWM_CONT: no longer U18.GPIOR_123_CLK12_CDI20
- net MTR_SENSE_A: no longer U18.GPIOL_75_PLLIN1
- net MTR_SENSE_B: no longer U18.GPIOL_74_PLLIN0
- net MTR_SENSE_IN_A: now also CN6.8; no longer CN6.3
- net MTR_SENSE_IN_B: now also CN6.9; no longer CN6.2
- net N$2: now also L1.1, U9.SW; no longer C1.1, U1.BOOT
- net N$57: now also CN6.4; no longer CN6.7
- net N$6: now also U8.VAA2V8_FILT; no longer L1.1, U1.SW
- net N$7: now also C40.1, R15.1, R22.2, U9.FB; no longer C3.2, R2.1, R4.2
- net POT_I2C1_SCL: no longer R46.1, U18.GPIOR_154, U31.SCL, U45.SCL, U51.SCL
- net POT_I2C1_SDA: no longer R56.1, U18.GPIOR_155, U31.SDA, U45.SDA, U51.SDA
- net PROC_JTAG_TCK: no longer U18.GPIOL_67_CDI13
- net PROC_JTAG_TDI: no longer U18.GPIOL_64
- net PROC_JTAG_TDO: no longer U18.GPIOL_69_CBSEL1
- net PROC_JTAG_TMS: no longer U18.GPIOL_68
- net PROC_UART_RX: no longer U18.GPIOR_77_PLLIN1
- net PROC_UART_TX: no longer U18.GPIOR_76_PLLIN0
- net PWR_SYS_3V3: now also C41.2, C50.2, CN6.7, R26.2, R27.2, U1.VCCIO1A, U1.VCCIO33_BL, U1.VCCIO3A, U11.EN, U11.VIN, U12.ON, U12.VIN, U6.BCBUS7, U9.EN, U9.VIN; no longer C107.2, C111.2, C115.2, C119.2, C123.2, C127.2, C139.2, C143.2, C147.2, C151.2, C163.2, C167.2, C29.2, C30.2, C31.2, C32.2, C35.2, CN6.4, R139.2, R140.2, R141.2, R143.2, R44.2, R45.2, R46.2, R56.2, U18.VCCIO1A, U18.VCCIO1B, U18.VCCIO1C_1D, U18.VCCIO1E, U18.VCCIO3A, U18.VCCIO3B_3C, U18.VCCIO3D, U18.VCCIO3E, U18.VCCIO4A, U18.VCCIO4B, U27.DVDD, U28.VIO, U30.DVDD, U31.VIO, U35.DVDD, U36.A0, U36.VIO, U41.DVDD, U42.A1, U42.VIO, U44.DVDD, U45.A0, U45.VIO, U50.DVDD, U51.A1, U51.VIO

Commit message: Progression
Parts:
- removed Q4, Q5: MMBT3906, TRANSISTORs:MMBT3906-7-F
- removed R16: 0R, RESISTORS:CRCW06030000Z0EA
- removed R17: 12k, r_0402:RC0402FR-0712KL
- removed R57: 10k, r_0603:CRCW060310K0FKTA
- removed U23: ADC101C027, ICs:ADC101C027CIMKX/NOPB
- added C61, C62, C63, C67, C71, C72, C73, C74, C75, C77, C78, C79, C80, C81, C82: 0.1uF 16V, c_0402:0402YD104JAT2A
- added C76, C83: 10uF 6.3V, c_0402:GRM155R60J106ME15D
- C64: device c_0402:0402YC104KAT2A -> c_0402:0402YD104JAT2A
- C65: value 0.1uF 16V -> 10uF 6.3V; device c_0402:0402YC104KAT2A -> c_0402:GRM155R60J106ME15D
Connections:
- removed net N$18: Q4.B, Q5.B, Q5.C, R17.2
- removed net N$38: R57.1, U23.!ALERT
- removed net POT_I2C1_SCL: U23.SCL
- removed net POT_I2C1_SDA: U23.SDA
- new net RAM_CLKN: U1.GPIOR_N_02_CDI25, U10.!CLK
- new net RAM_CLKP: U1.GPIOR_P_02_CDI24, U10.CLK
- new net RAM_D0: U1.GPIOR_P_06_CDI20, U10.D0
- new net RAM_D1: U1.GPIOR_N_06_CDI21, U10.D1
- new net RAM_D2: U1.GPIOR_P_01_EXTFB, U10.D2
- new net RAM_D3: U1.GPIOR_N_01_CDI23, U10.D3
- new net RAM_D4: U1.GPIOR_N_05_CDI31, U10.D4
- new net RAM_D5: U1.GPIOR_P_07, U10.D5
- new net RAM_D6: U1.GPIOR_P_09_CLK10_P, U10.D6
- new net RAM_D7: U1.GPIOR_N_07, U10.D7
- new net RAM_NCS: U1.GPIOR_N_04_CDI29, U10.!CS
- new net RAM_NRESET: U1.GPIOR_P_05_CDI30, U10.!RESET
- new net RAM_RWDS: U1.GPIOR_P_04_CDI28, U10.RWDS
- net GND: now also C61.1, C62.1, C63.1, C67.1, C71.1, C72.1, C73.1, C74.1, C75.1, C76.1, C77.1, C78.1, C79.1, C80.1, C81.1, C82.1, C83.1; no longer R16.1, R17.1, U23.GND
- net LED_FPGA_STATUS: now also U1.GPIOL_09
- net LED_PROC_SCANNING: now also U1.GPIOL_03
- net LED_PROC_STATUS: now also U1.GPIOL_04
- net PROC_JTAG_TCK: now also U1.GPIOR_16
- net PROC_JTAG_TDI: now also U1.GPIOR_12
- net PROC_JTAG_TDO: now also U1.GPIOR_18
- net PROC_JTAG_TMS: now also U1.GPIOR_19
- net PROC_UART_RX: now also U1.GPIOR_13
- net PROC_UART_TX: now also U1.GPIOR_15
- net PWR_FPGA_0V95: now also C61.2, C62.2, C63.2, C64.2, C65.2, C67.2, C71.2, C72.2, C73.2
- net PWR_FPGA_1V8: now also C74.2, C77.2, C78.2, C79.2
- net PWR_MIPI_1V2: now also C75.2, C76.2
- net PWR_SYS_1V8: now also C80.2, C81.2, C82.2, C83.2, U1.VCCIO3B, U10.VCC, U10.VCCQ
- net PWR_SYS_3V3: now also U1.VCCIO33_TL, U1.VCCIO33_TR; no longer C64.2, Q4.E, Q5.E, R57.2, U23.VDD
- net TEMP_SEN_A: no longer C65.2, Q4.C, U23.AIN
- net TEMP_SEN_B: no longer R16.2
