File: main.sch (EAGLE design)
At the start: 172 parts, among them CN1 DC-012A-D010, CN2 JST GH 10 Pin, CN3 5.8ZSPT, CN4 8 PIN FFC, CN5 MC-118LS-H100, CN6 JST GH 10 Pin, CN7 8 PIN FFC, Q1 GSFP0449, Q6 IRLML6244, U1 Ti60F225C4, U10 W958D8NBYA5I, U11 TPS70918, U12 AP7335, U2 USBLC6-2SC6, U24 SCHMITT, U25 SCHMITT, U3 93LC56B-I/SN, U4 W25Q128JV, U5 TPS62065, U6 FT2232H, U7 TPS563201, U8 AR0822, U9 TPS62065

Commit message: Initial layout done
Parts:
- CN2, CN6: value JST GH 10 Pin -> JST GH 6P V-TH; device CONNECTORs:1.25-10PWT -> CONNECTORs:2.0MM-6PZZ
Connections:
- removed net PWR_FPGA_1V8: C74.2, C77.2, C78.2, C79.2, U1.VCCAUX
- removed net TEMP_SEN_A: CN2.2
- removed net TEMP_SEN_B: CN2.1
- net GND: now also CN2.3, CN6.6; no longer CN2.5, CN2.7, CN6.10
- net LED_PWM_CONT: now also CN2.5, U1.GPIOL_11_PLLIN2; no longer CN2.3
- net MTR_CONT_PWM: now also U1.GPIOL_10
- net MTR_SENSE_A: now also U1.GPIOL_06
- net MTR_SENSE_B: now also U1.GPIOL_07
- net MTR_SENSE_IN_A: now also CN6.4; no longer CN6.8
- net MTR_SENSE_IN_B: now also CN6.5; no longer CN6.9
- net N$57: now also CN6.2; no longer CN6.4, CN6.5, CN6.6
- net PWR_BUS_UNREG: now also CN2.1, CN2.2; no longer CN2.10, CN2.8, CN2.9, CN6.2, CN6.3
- net PWR_SYS_1V8: now also C74.2, C77.2, C78.2, C79.2, U1.VCCAUX
- net PWR_SYS_3V3: now also CN6.3; no longer CN6.7

Commit message: New LED driver PCB
Changed lines of the file:
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@@
 <pinref part="U1" gate="G$1" pin="GPIOB_P_00_PLLIN1"/>
 <wire x1="71.12" y1="20.32" x2="33.02" y2="20.32" width="0.1524" layer="91"/>
-<label x="35.56" y="20.32" size="1.778" layer="95"/>
+<label x="38.1" y="20.32" size="1.778" layer="95"/>
 </segment>
 </net>
@@
 <pinref part="U1" gate="G$1" pin="GPIOB_N_00"/>
 <wire x1="71.12" y1="17.78" x2="33.02" y2="17.78" width="0.1524" layer="91"/>
-<label x="35.56" y="17.78" size="1.778" layer="95"/>
+<label x="38.1" y="17.78" size="1.778" layer="95"/>
 </segment>
 </net>
@@
 <pinref part="U1" gate="G$1" pin="GPIOB_P_01_EXTFB"/>
 <wire x1="71.12" y1="15.24" x2="33.02" y2="15.24" width="0.1524" layer="91"/>
-<label x="35.56" y="15.24" size="1.778" layer="95"/>
+<label x="38.1" y="15.24" size="1.778" layer="95"/>
 </segment>
 </net>
@@
 <pinref part="U1" gate="G$1" pin="GPIOB_N_01"/>
 <wire x1="71.12" y1="12.7" x2="33.02" y2="12.7" width="0.1524" layer="91"/>
-<label x="35.56" y="12.7" size="1.778" layer="95"/>
+<label x="38.1" y="12.7" size="1.778" layer="95"/>
 </segment>
 </net>
@@
 <pinref part="U1" gate="G$1" pin="GPIOB_P_02_CDI4"/>
 <wire x1="71.12" y1="10.16" x2="33.02" y2="10.16" width="0.1524" layer="91"/>
-<label x="35.56" y="10.16" size="1.778" layer="95"/>
+<label x="38.1" y="10.16" size="1.778" layer="95"/>
 </segment>
 </net>
@@
 <pinref part="U1" gate="G$1" pin="GPIOB_N_02_CDI5"/>
 <wire x1="71.12" y1="7.62" x2="33.02" y2="7.62" width="0.1524" layer="91"/>
-<label x="35.56" y="7.62" size="1.778" layer="95"/>
+<label x="38.1" y="7.62" size="1.778" layer="95"/>
 </segment>
 </net>
@@
 <pinref part="U1" gate="G$1" pin="GPIOB_P_07_CLK15_P"/>
 <wire x1="71.12" y1="-10.16" x2="33.02" y2="-10.16" width="0.1524" layer="91"/>
-<label x="35.56" y="-10.16" size="1.778" layer="95"/>
+<label x="38.1" y="-10.16" size="1.778" layer="95"/>
 </segment>
 </net>
@@
 <pinref part="U1" gate="G$1" pin="GPIOB_N_07_CLK15_N"/>
 <wire x1="71.12" y1="-12.7" x2="33.02" y2="-12.7" width="0.1524" layer="91"/>
-<label x="35.56" y="-12.7" size="1.778" layer="95"/>
+<label x="38.1" y="-12.7" size="1.778" layer="95"/>
 </segment>
 </net>
@@
 <pinref part="U1" gate="G$1" pin="GPIOB_P_08_CLK14_P"/>
 <wire x1="33.02" y1="-15.24" x2="71.12" y2="-15.24" width="0.1524" layer="91"/>
-<label x="35.56" y="-15.24" size="1.778" layer="95"/>
+<label x="38.1" y="-15.24" size="1.778" layer="95"/>
 </segment>
 </net>

Commit message: Moving back to Trion
Parts:
- removed C22, C34, C38, C52, C53, C54, C55, C56, C57, C59: 0.1uF 16V, c_0603:0603YC104JAZ2A
- removed C23, C24: 10pF 100V, c_0603:06031A100B4T2A
- removed C28, C61, C62, C63, C64, C66, C67, C71, C72, C73, C74, C75, C77, C78, C79, C80, C81, C82: 0.1uF 16V, c_0402:0402YD104JAT2A
- removed C58: 4.7uF 6.3V, c_0603:06036D475KAT4A
- removed C65, C76, C83: 10uF 6.3V, c_0402:GRM155R60J106ME15D
- removed CN4, CN7: 8 PIN FFC, CONNECTORs:SFV8R-1STBE1HLF
- removed D10, D12, D5, D6, D7, D8: RED LED, OPTO:150060RS75000
- removed R10, R11, R12, R13, R14, R59: 2.2k, r_0603:CRCW06032K20FKEA
- removed R130, R137, R138, R142, R143, R144, R145, R146, R147, R20, R21, R26, R27, R74, R75: 10k, r_0402:RC0402FR-0710KL
- removed R6: 12k, RESISTORS:CRCW060312K0FKEA
- removed R67: 1k, r_0402:RC0402FR-071KL
- removed R7, R8, R9: 10k, r_0603:ERJ3EKF1002V
- removed U10: W958D8NBYA5I, ICs:W958D8NBYA5I
- removed U3: 93LC56B-I/SN, ICs:93LC56B-I/SN
- removed U4: W25Q128JV, ICs:W25Q128JVSIQ
- removed U6: FT2232H, ICs:FT2232H
- removed XTAL2: 12MHz, CRYSTALS:ABM8-12.000MHZ-B2-T
- added U37: W25Q128JV, ICs:W25Q128JVSIQ
- C25: value 0.1uF 16V -> 0.1uF 10V; device c_0603:0603YC104JAZ2A -> c_0402:0402ZC104KAT2A
- C27: value 0.1uF 16V -> 0.1uF 10V; device c_0402:0402YD104JAT2A -> c_0402:0402ZC104KAT2A
- OSC1: device CRYSTALS:KC2016Z33.0000C15XXK -> CRYSTALS:KC2016Z33.0000C1KX00
- R3: value 10k -> 10R; device r_0402:RC0402FR-0710KL -> r_0402:RC0402FR-0710RL
- U1: value Ti60F225C4 -> T20F169; device ICs:TI60F225C4 -> ICs:T20F169I4
Connections:
- removed net FLS_NHOLD: R138.1, U4.!HOLD!/IO3
- removed net FLS_SPI_CLK: R144.1, U1.GPIOL_N_01_CCK, U4.SCK
- removed net FLS_SPI_MISO: R27.1, U1.GPIOL_N_03_CDI1, U4.SO/IO1
- removed net FLS_SPI_MOSI: R26.1, U1.GPIOL_P_03_CDI0, U4.SI/IO0
- removed net FLS_SPI_NCS: R142.1, U1.GPIOL_P_01_SSL_N, U4.!CE
- removed net FPGA_CLK_33M: OSC1.OUT, U1.GPIOL_P_00_PLLIN0
- removed net FPGA_CONF_CDONE: R147.1, U1.CDONE
- removed net FPGA_CONF_CSI: CN4.3, R145.1, U1.GPIOL_P_02_CSI
- removed net FPGA_CONF_NCRST: C66.2, CN4.2, R146.1, U1.CRESET_N
- removed net FPGA_CONF_NTEST: R143.1, U1.GPIOL_N_15_TEST_N
- removed net FPGA_JTAG_TCK: CN4.5, R3.1, U1.TCK
- removed net FPGA_JTAG_TDI: CN4.4, U1.TDI
- removed net FPGA_JTAG_TDO: CN4.7, R130.1, U1.TDO
- removed net FPGA_JTAG_TMS: CN4.6, U1.TMS
- removed net FT_CLKOUT: U1.GPIOR_N_11_CLK8_N, U6.ACBUS5
- removed net FT_CONT_RX: U1.GPIOR_P_11_CLK8_P, U6.BDBUS1
- removed net FT_CONT_TX: U1.GPIOR_P_13, U6.BDBUS0
- removed net FT_D0: U1.GPIOR_P_17, U6.ADBUS0
- removed net FT_D1: U1.GPIOR_P_19_PLLIN0, U6.ADBUS1
- removed net FT_D2: U1.GPIOR_P_12, U6.ADBUS2
- removed net FT_D3: U1.GPIOR_N_12, U6.ADBUS3
- removed net FT_D4: U1.GPIOR_P_15, U6.ADBUS4
- removed net FT_D5: U1.GPIOR_N_15, U6.ADBUS5
- removed net FT_D6: U1.GPIOR_N_17, U6.ADBUS6
- removed net FT_D7: U1.GPIOR_N_19, U6.ADBUS7
- removed net FT_NOE: U1.GPIOR_P_10_CLK9_P, U6.ACBUS6
- removed net FT_NRD: U1.GPIOR_N_16, U6.ACBUS2
- removed net FT_NRST: U1.GPIOR_N_10_CLK9_N, U6.!RESET
- removed net FT_NRXF: U1.GPIOR_N_18, U6.ACBUS0
- removed net FT_NSIWU: U1.GPIOR_N_13, U6.ACBUS4
- removed net FT_NTXE: U1.GPIOR_P_18, U6.ACBUS1
- removed net FT_NWR: U1.GPIOR_P_16, U6.ACBUS3
- removed net LED_FPGA_STATUS: D6.K, U1.GPIOL_09
- removed net LED_FT_CONT_NRXLED: D8.K, U6.BCBUS3
- removed net LED_FT_CONT_NTXLED: D7.K, U6.BCBUS4
- removed net LED_PROC_SCANNING: D10.K, U1.GPIOL_03
- removed net LED_PROC_STATUS: D5.K, U1.GPIOL_04
- removed net LED_USB_ACT: D12.K
- removed net N$113: D10.A, R59.1
- removed net N$14: D5.A, R11.1
- removed net N$15: D6.A, R12.1
- removed net N$16: D7.A, R13.1
- removed net N$17: D8.A, R14.1
- removed net N$42: R6.2, U6.REF
- removed net N$43: R7.1, U3.CS, U6.EECS
- removed net N$44: R8.1, U3.CLK, U6.EECLK
- removed net N$45: R10.2, U3.DI, U6.EEDATA
- removed net N$46: R10.1, R9.1, U3.DO
- removed net N$47: D12.A, R67.1
- removed net N$49: C23.2, U6.XCSO, XTAL2.P$2
- removed net N$50: C24.2, U6.XCSI, XTAL2.P$1
- removed net N$51: C55.2, C56.2, C57.2, C58.2, U6.VCORE, U6.VREGOUT
- removed net N$8: R137.1, U4.!WP!/IO2
- removed net PROC_JTAG_TCK: CN7.5, R21.1, U1.GPIOR_16
- removed net PROC_JTAG_TDI: CN7.4, U1.GPIOR_12
- removed net PROC_JTAG_TDO: CN7.7, R20.1, U1.GPIOR_18
- removed net PROC_JTAG_TMS: CN7.6, U1.GPIOR_19
- removed net PROC_UART_RX: CN7.2, R75.1, U1.GPIOR_13
- removed net PROC_UART_TX: CN7.3, R74.1, U1.GPIOR_15
- removed net PWR_MIPI_1V2: C75.2, C76.2, R143.2, U1.VCCIO1B
- removed net RAM_CLKN: U1.GPIOR_N_02_CDI25, U10.!CLK
- removed net RAM_CLKP: U1.GPIOR_P_02_CDI24, U10.CLK
- removed net RAM_D0: U1.GPIOR_P_06_CDI20, U10.D0
- removed net RAM_D1: U1.GPIOR_N_06_CDI21, U10.D1
- removed net RAM_D2: U1.GPIOR_P_01_EXTFB, U10.D2
- removed net RAM_D3: U1.GPIOR_N_01_CDI23, U10.D3
- removed net RAM_D4: U1.GPIOR_N_05_CDI31, U10.D4
- removed net RAM_D5: U1.GPIOR_P_07, U10.D5
- removed net RAM_D6: U1.GPIOR_P_09_CLK10_P, U10.D6
- removed net RAM_D7: U1.GPIOR_N_07, U10.D7
- removed net RAM_NCS: U1.GPIOR_N_04_CDI29, U10.!CS
- removed net RAM_NRESET: U1.GPIOR_P_05_CDI30, U10.!RESET
- removed net RAM_RWDS: U1.GPIOR_P_04_CDI28, U10.RWDS
- new net N$9: OSC1.OUT, R3.1
- new net PSS_CLK_33M: R3.2
- new net PSS_FLASH_D0: U37.SI/IO0
- new net PSS_FLASH_D1: U37.SO/IO1
- new net PSS_FLASH_D2: U37.!WP!/IO2
- new net PSS_FLASH_D3: U37.!HOLD!/IO3
- new net PSS_FLASH_NCS: U37.!CE
- new net PSS_FLASH_SCLK: U37.SCK
- new net USB_VBUS: CN5.VBUS, U2.VBUS
- net AR_CLK: no longer U1.GPIOB_N_01
- net AR_GPIO0: no longer U1.GPIOB_N_02_CDI5
- net AR_GPIO1: no longer U1.GPIOB_P_01_EXTFB
- net AR_GPIO2: no longer U1.GPIOB_N_07_CLK15_N
- net AR_GPIO3: no longer U1.GPIOB_P_02_CDI4
- net AR_I2C_SCL: no longer U1.GPIOB_P_07_CLK15_P
- net AR_I2C_SDA: no longer U1.GPIOB_P_08_CLK14_P
- net AR_MIPI_CLK_N: no longer U1.GPIOL_N_09_CLK2_N
- net AR_MIPI_CLK_P: no longer U1.GPIOL_P_09_CLK2_P
- net AR_MIPI_D0_N: no longer U1.GPIOL_N_11
- net AR_MIPI_D0_P: no longer U1.GPIOL_P_11
- net AR_MIPI_D1_N: no longer U1.GPIOL_N_14
- net AR_MIPI_D1_P: no longer U1.GPIOL_P_14
- net AR_MIPI_D2_N: no longer U1.GPIOL_N_16
- net AR_MIPI_D2_P: no longer U1.GPIOL_P_16
- net AR_MIPI_D3_N: no longer U1.GPIOL_N_18
- net AR_MIPI_D3_P: no longer U1.GPIOL_P_18_PLLIN0
- net AR_NRESET: no longer U1.GPIOB_P_00_PLLIN1
- net AR_XSHUTDOWN: no longer U1.GPIOB_N_00
- net GND: now also U37.GND; no longer C22.1, C23.1, C24.1, C28.2, C34.1, C38.1, C52.1, C53.1, C54.1, C55.1, C56.1, C57.1, C58.1, C59.1, C61.1, C62.1, C63.1, C64.1, C65.1, C66.1, C67.1, C71.1, C72.1, C73.1, C74.1, C75.1, C76.1, C77.1, C78.1, C79.1, C80.1, C81.1, C82.1, C83.1, CN4.8, CN7.8, R6.1, U1.GND, U10.VSS, U10.VSSQ, U3.GND, U4.GND, U6.BDBUS3, U6.BDBUS4, U6.BDBUS5, U6.BDBUS6, U6.GND, U6.TEST, XTAL2.GND
- net LED_PWM_CONT: no longer U1.GPIOL_11_PLLIN2
- net MTR_CONT_PWM: no longer U1.GPIOL_10
- net MTR_SENSE_A: no longer U1.GPIOL_06
- net MTR_SENSE_B: no longer U1.GPIOL_07
- net PWR_FPGA_0V95: no longer C61.2, C62.2, C63.2, C64.2, C65.2, C67.2, C71.2, C72.2, C73.2, U1.VCC, U1.VCCA_BL, U1.VCCA_BR, U1.VCCA_TL, U1.VCCA_TR
- net PWR_SYS_1V8: now also C25.2, OSC1.!ST, OSC1.VCC; no longer C74.2, C77.2, C78.2, C79.2, C80.2, C81.2, C82.2, C83.2, U1.VCCAUX, U1.VCCIO3B, U1.VCCIO4B, U10.VCC, U10.VCCQ
- net PWR_SYS_3V3: now also U37.VCC; no longer C22.2, C25.2, C28.1, C34.2, C38.2, C52.2, C53.2, C54.2, C59.2, CN4.1, CN7.1, OSC1.!ST, OSC1.VCC, R11.2, R12.2, R13.2, R130.2, R137.2, R138.2, R14.2, R142.2, R144.2, R145.2, R146.2, R147.2, R20.2, R21.2, R26.2, R27.2, R3.2, R59.2, R67.2, R7.2, R74.2, R75.2, R8.2, R9.2, U1.VCCIO1A, U1.VCCIO33_BL, U1.VCCIO33_TL, U1.VCCIO33_TR, U1.VCCIO3A, U3.V+, U4.VCC, U6.BCBUS7, U6.VCCIO, U6.VPHY, U6.VPLL, U6.VREGIN
- net USB_D_N: no longer U6.D-
- net USB_D_P: no longer U6.D+
Other:
- note added: "2024.03.19 - GSWDH LTD. FILM SCANNER MAIN REVISION 3.0.0 DESIGN BY GEORGE WALLER AT GSWDH LTD. GEORGEWALLER@GSWDH.CO.UK CONFIDENTIAL. FOR THE INTENDED READER ONLY."
- note removed: "2023.06.28 - GSWDH LTD. MOON CONTROLLER REVISION 1.0.0 DESIGN BY GEORGE WALLER AT GSWDH LTD. GEORGEWALLER@GSWDH.CO.UK CONFIDENTIAL. FOR THE INTENDED READER ONLY."
- moved on the sheet: C27, C36, C37, C39, CN5, L3, OSC1, R148, R149, R3, U2, U5

Commit message: Initial layout done
Parts:
- removed U37: W25Q128JV, ICs:W25Q128JVSIQ
- added C22, C28, C34, C38, C52, C53, C54, C55, C56, C57, C59, C61, C64, C65, C66, C67, C72, C73, C74, C75, C76, C78, C79, C82: 0.1uF 16V, c_0402:0402YD104JAT2A
- added C23, C24: 10pF 10V, c_0402:C0402C100C8GACTU
- added C58, C62, C63, C71, C77, C80: 10uF 6.3V, c_0402:GRM155R60J106ME15D
- added CN4, CN8: FFC 8P 0.5mm, CONNECTORs:HC-FPC-05-09-8RLTAG
- added R10: 2.2k, r_0402:RC0402FR-072K2L
- added R11, R12, R13, R137, R138, R14, R140, R141, R142, R143, R144, R146, R147, R16, R26, R7, R76, R77, R8, R9: 10k, r_0402:RC0402FR-0710KL
- added R17: 20k, r_0402:RC0402FR-0720KL
- added R20: 16k, r_0402:RC0402FR-1316KL
- added R21: 51k, r_0402:RC0402FR-0751KL
- added R25: 24k, r_0402:RC0402FR-0724KL
- added R6: 12k, r_0402:RC0402FR-0712KL
- added U10: AP7335, ICs:AP7335-SNG-7
- added U13: W958D8NBYA5I, ICs:W958D8NBYA5I
- added U3: 93LC56B-I/SN, ICs:93LC56B-I/SN
- added U4: W25Q128JV, ICs:W25Q128JVSIQ
- added U6: FT2232H, ICs:FT2232H
- added XTAL2: 12MHz, CRYSTALS:ABM8-12.000MHZ-B2-T
- C25: value 0.1uF 10V -> 0.1uF 16V; device c_0402:0402ZC104KAT2A -> c_0402:0402YD104JAT2A
- C27: value 0.1uF 10V -> 1uF 10V; device c_0402:0402ZC104KAT2A -> c_0402:0402ZD105KAT2A
- C43: value 100nF 16V -> 0.1uF 16V; device CAPACITORS:CL10B104KO8WPNC -> c_0402:0402YD104JAT2A
- C48: device c_0603:06035A101J4T4A -> c_0402:C0402C100C8GACTU
- C49: value 2.2uF 6.3V -> 1uF 10V; device c_0402:C0402C225K9PAC7867 -> c_0402:0402ZD105KAT2A
- C69, C70: device c_0402:0402YC104KAT2A -> c_0402:0402YD104JAT2A
- C7: value 100pF 50V -> 100pF 25V; device c_0603:06035A101J4T4A -> c_0402:04023A101KAT2A
- R1, R19, R5, R68, R72, R73: device r_0603:CRCW060310K0FKTA -> r_0402:RC0402FR-0710KL
- R18: device r_0603:CRCW060334K0FKEA -> r_0402:RC0402FR-0734KL
- R58, R66: value 20k -> 10k; device r_0402:RC0402FR-0720KL -> r_0402:RC0402FR-0710KL
- U11: value TPS70918 -> AP7335; device ICs:TPS70918DBVT -> ICs:AP7335-SNG-7
Connections:
- removed net PSS_CLK_33M: R3.2
- removed net PSS_FLASH_D0: U37.SI/IO0
- removed net PSS_FLASH_D1: U37.SO/IO1
- removed net PSS_FLASH_D2: U37.!WP!/IO2
- removed net PSS_FLASH_D3: U37.!HOLD!/IO3
- removed net PSS_FLASH_NCS: U37.!CE
- removed net PSS_FLASH_SCLK: U37.SCK
- removed net PWR_FPGA_0V95: C37.2, C39.2, L3.2, R148.2
- new net FLS_NHOLD: R138.1, U4.!HOLD!/IO3
- new net FLS_SPI_CLK: R144.1, U1.GPIOL_01_CCK, U4.SCK
- new net FLS_SPI_MISO: R12.1, U1.GPIOL_09_CDI1, U4.SO/IO1
- new net FLS_SPI_MOSI: R11.1, U1.GPIOL_08_CDI0, U4.SI/IO0
- new net FLS_SPI_NCS: R142.1, U1.GPIOL_00_SS_N, U4.!CE
- new net FPGA_CLK33M: R3.2, U1.GPIOR_157_PLLIN
- new net FPGA_CONF_CBUS_0: R141.1, U1.GPIOR_151_CBUS0
- new net FPGA_CONF_CBUS_1: R140.1, U1.GPIOR_150_CBUS1
- new net FPGA_CONF_CDONE: R147.1, U1.CDONE
- new net FPGA_CONF_NCRST: C66.2, CN8.7, R146.1, U1.CRESET_N
- new net FPGA_CONF_NTEST: R143.1, U1.GPIOR_158_TEST_N
- new net FPGA_JTAG_TCK: CN8.4, R76.1, U1.TCK
- new net FPGA_JTAG_TDI: CN8.5, U1.TDI
- new net FPGA_JTAG_TDO: CN8.2, R77.1, U1.TDO
- new net FPGA_JTAG_TMS: CN8.3, U1.TMS
- new net FT_CLKOUT: U1.GPIOB_CLKP0, U6.ACBUS5
- new net FT_CONT_RX: U1.GPIOB_RXN06, U6.BDBUS1
- new net FT_CONT_TX: U1.GPIOB_RXN04, U6.BDBUS0
- new net FT_D0: U1.GPIOB_RXN09, U6.ADBUS0
- new net FT_D1: U1.GPIOB_RXN10, U6.ADBUS1
- new net FT_D2: U1.GPIOB_RXP09, U6.ADBUS2
- new net FT_D3: U1.GPIOB_RXP10, U6.ADBUS3
- new net FT_D4: U1.GPIOB_RXN07, U6.ADBUS4
- new net FT_D5: U1.GPIOB_RXP07, U6.ADBUS5
- new net FT_D6: U1.GPIOB_RXP05, U6.ADBUS6
- new net FT_D7: U1.GPIOB_RXN05, U6.ADBUS7
- new net FT_NOE: U1.GPIOB_RXP00, U6.ACBUS6
- new net FT_NRD: U1.GPIOB_RXN03, U6.ACBUS2
- new net FT_NRST: U1.GPIOB_RXN08, U6.!RESET
- new net FT_NRXF: U1.GPIOB_RXP02, U6.ACBUS0
- new net FT_NSIWU: U1.GPIOB_RXP01, U6.ACBUS4
- new net FT_NTXE: U1.GPIOB_RXP03, U6.ACBUS1
- new net FT_NWR: U1.GPIOB_RXN01, U6.ACBUS3
- new net LED_FT_CONT_NRXLED: U6.BCBUS3
- new net LED_FT_CONT_NTXLED: U6.BCBUS4
- new net N$17: R21.1, R25.2, U11.FB
- new net N$23: R26.1, U1.REF_RES
- new net N$38: R137.1, U4.!WP!/IO2
- new net N$42: R6.2, U6.REF
- new net N$43: R7.1, U3.CS, U6.EECS
- new net N$44: R8.1, U3.CLK, U6.EECLK
- new net N$45: R10.2, U3.DI, U6.EEDATA
- new net N$46: R10.1, R9.1, U3.DO
- new net N$49: C23.2, U6.XCSO, XTAL2.P$2
- new net N$50: C24.2, U6.XCSI, XTAL2.P$1
- new net N$51: C55.2, C56.2, C57.2, C58.2, U6.VCORE, U6.VREGOUT
- new net N$8: R17.1, R20.2, U10.FB
- new net PROC_JTAG_TCK: CN4.4, R13.1, U1.GPIOB_TXP00
- new net PROC_JTAG_TDI: CN4.5, U1.GPIOB_TXN05
- new net PROC_JTAG_TDO: CN4.2, R14.1, U1.GPIOB_TXN00
- new net PROC_JTAG_TMS: CN4.3, U1.GPIOL_21_CTRL1_CDI5
- new net PROC_NRST: CN4.7, R16.1, U1.GPIOL_25_CLK1
- new net PWR_FPGA_1V2: C37.2, C39.2, C71.2, C72.2, C73.2, C74.2, C75.2, C76.2, L3.2, R148.2, U1.VCC, U1.VCC12A_MIPI0_RX, U1.VCC12A_MIPI0_TX, U1.VCC12A_MIPI1_RX, U1.VCC12A_MIPI1_TX, U1.VCCA_BR, U1.VCCA_TL, U1.VCCA_TR
- new net PWR_FPGA_2V5: C62.2, C82.2, R21.2, U1.VCC25A_MIPI0, U1.VCC25A_MIPI1, U11.VOUT
- new net RAM_CLK_N: U1.GPIOB_TXN01, U13.!CLK
- new net RAM_CLK_P: U1.GPIOB_TXP01, U13.CLK
- new net RAM_D0: U1.GPIOB_TXP08, U13.D0
- new net RAM_D1: U1.GPIOB_TXP06, U13.D1
- new net RAM_D2: U1.GPIOB_TXN08, U13.D2
- new net RAM_D3: U1.GPIOB_TXN09, U13.D3
- new net RAM_D4: U1.GPIOB_TXP09, U13.D4
- new net RAM_D5: U1.GPIOB_TXP05, U13.D5
- new net RAM_D6: U1.GPIOB_TXP02, U13.D6
- new net RAM_D7: U1.GPIOB_TXN03, U13.D7
- new net RAM_NCS: U1.GPIOB_TXN02, U13.!CS
- new net RAM_NRST: U1.GPIOB_TXP03, U13.!RESET
- new net RAM_RWDS: U1.GPIOB_TXN06, U13.RWDS
- net AR_CLK: now also U1.GPIOL_72_EXTFB0_CDI14
- net AR_GPIO0: now also U1.GPIOL_73_EXTFB1_CDI15
- net AR_GPIO1: now also U1.GPIOL_71_NSTATUS
- net AR_GPIO2: now also U1.GPIOL_69_CBSEL1
- net AR_GPIO3: now also U1.GPIOL_70_CBSEL0
- net AR_I2C_SCL: now also U1.GPIOL_20_CTRL0_CDI4
- net AR_I2C_SDA: now also U1.GPIOL_12_CDI2
- net AR_MIPI_CLK_N: now also U1.MIPI1_RXDP2
- net AR_MIPI_CLK_P: now also U1.MIPI1_RXDN2
- net AR_MIPI_D0_N: now also U1.MIPI1_RXDP1
- net AR_MIPI_D0_P: now also U1.MIPI1_RXDN1
- net AR_MIPI_D1_N: now also U1.MIPI1_RXDN0
- net AR_MIPI_D1_P: now also U1.MIPI1_RXDP0
- net AR_MIPI_D2_N: now also U1.MIPI1_RXDP4
- net AR_MIPI_D2_P: now also U1.MIPI1_RXDN4
- net AR_MIPI_D3_N: now also U1.MIPI1_RXDN3
- net AR_MIPI_D3_P: now also U1.MIPI1_RXDP3
- net AR_NRESET: now also U1.GPIOL_74_PLLIN0
- net AR_XSHUTDOWN: now also U1.GPIOL_75_PLLIN1
- net GND: now also C22.1, C23.1, C24.1, C28.1, C34.1, C38.1, C52.1, C53.1, C54.1, C55.1, C56.1, C57.1, C58.1, C59.1, C61.1, C62.1, C63.1, C64.1, C65.1, C66.1, C67.1, C71.1, C72.1, C73.1, C74.1, C75.1, C76.1, C77.1, C78.1, C79.1, C80.1, C82.1, CN4.1, CN8.1, R20.1, R25.1, R26.2, R6.1, U1.GND, U1.GNDA_MIPI, U10.GND, U13.VSS, U13.VSSQ, U3.GND, U4.GND, U6.BDBUS3, U6.BDBUS5, U6.BDBUS6, U6.GND, U6.TEST, XTAL2.GND; no longer U37.GND
- net LED_PWM_CONT: now also U1.GPIOR_77_PLLIN1
- net MTR_SENSE_A: now also U1.GPIOR_78_EXTFB0_CDI31
- net MTR_SENSE_B: now also U1.GPIOR_119_CTRL12
- net PWR_SYS_1V8: now also C41.2, C63.2, C64.2, C65.2, C67.2, R17.2, U1.VCCIO1B_1C_1D, U1.VCCIO1E, U1.VCCIO4B, U10.VOUT, U13.VCC, U13.VCCQ; no longer C25.2, C49.2, OSC1.!ST, OSC1.VCC, U11.VOUT
- net PWR_SYS_3V3: now also C22.2, C25.2, C28.2, C34.2, C38.2, C49.2, C52.2, C53.2, C54.2, C59.2, C61.2, C77.2, C78.2, C79.2, C80.2, CN4.8, CN8.8, OSC1.!ST, OSC1.VCC, R11.2, R12.2, R13.2, R137.2, R138.2, R14.2, R140.2, R141.2, R142.2, R143.2, R144.2, R146.2, R147.2, R16.2, R7.2, R76.2, R77.2, R8.2, R9.2, U1.VCCIO1A, U1.VCCIO3A_3B, U1.VCCIO3C_3D_3E, U1.VCCIO4A, U10.ON, U10.VIN, U11.ON, U3.V+, U4.VCC, U6.BCBUS7, U6.BDBUS7, U6.VCCIO, U6.VPHY, U6.VPLL, U6.VREGIN; no longer C41.2, U11.EN, U37.VCC
- net USB_D_N: now also U6.D-
- net USB_D_P: now also U6.D+
Other:
- moved on the sheet: C25, C41, C50, C51, OSC1, R23, R24, R3, U12
