File: main.sch (EAGLE design)
At the start: 192 parts, among them CN1 DC-012A-D010, CN2 JST GH 6P V-TH, CN3 5.8ZSPT, CN5 MC-118LS-H100, CN6 JST GH 6P V-TH, CN8 FFC 8P 0.5mm, Q1 GSFP0449, Q2 MMBT3904, Q3 MMBT3904, U1 T20F169, U10 AP7335, U11 AP7335, U12 AP7335, U13 W958D8NBYA5I, U14 AS4950, U15 ESP32, U16 PI4ULS3V204ZBEX, U2 USBLC6-2SC6, U24 SCHMITT, U3 93LC56B-I/SN, U4 SCHMITT, U5 TPS62065, U6 FT2232H, U7 TPS563201, U8 AR0822, U9 TPS62065

Commit message: LEDs routed. Text added. Pushed to Fusion
Connections:
- removed net FPGA_LED_1: R79.2
- removed net FPGA_LED_2: R59.2
- new net ESP_LED_0: R79.2, U15.IO22
- new net ESP_LED_1: R59.2, U15.IO23
- net FPGA_LED_0: now also U1.GPIOR_119_CTRL12
Other:
- moved on the sheet: D5, D6, D7, R59, R79, R80
Changed lines of the file:
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@@
 <attribute name="VALUE" x="63.5" y="-157.48" size="1.27" layer="96" rot="R90" align="center"/>
 </instance>
-<instance part="D6" gate="G$1" x="121.92" y="-68.58" smashed="yes" rot="R270">
-<attribute name="NAME" x="119.38" y="-68.58" size="1.27" layer="95" rot="R270" align="center"/>
-<attribute name="VALUE" x="116.84" y="-68.58" size="1.27" layer="96" rot="R270" align="center"/>
+<instance part="D6" gate="G$1" x="134.62" y="-127" smashed="yes" rot="R270">
+<attribute name="NAME" x="132.08" y="-127" size="1.27" layer="95" rot="R270" align="center"/>
+<attribute name="VALUE" x="129.54" y="-127" size="1.27" layer="96" rot="R270" align="center"/>
 </instance>
-<instance part="D7" gate="G$1" x="132.08" y="-68.58" smashed="yes" rot="R270">
-<attribute name="NAME" x="129.54" y="-68.58" size="1.27" layer="95" rot="R270" align="center"/>
-<attribute name="VALUE" x="127" y="-68.58" size="1.27" layer="96" rot="R270" align="center"/>
+<instance part="D7" gate="G$1" x="144.78" y="-127" smashed="yes" rot="R270">
+<attribute name="NAME" x="142.24" y="-127" size="1.27" layer="95" rot="R270" align="center"/>
+<attribute name="VALUE" x="139.7" y="-127" size="1.27" layer="96" rot="R270" align="center"/>
 </instance>
-<instance part="D5" gate="G$1" x="142.24" y="-68.58" smashed="yes" rot="R270">
-<attribute name="NAME" x="139.7" y="-68.58" size="1.27" layer="95" rot="R270" align="center"/>
-<attribute name="VALUE" x="137.16" y="-68.58" size="1.27" layer="96" rot="R270" align="center"/>
+<instance part="D5" gate="G$1" x="-142.24" y="86.36" smashed="yes" rot="R270">
+<attribute name="NAME" x="-144.78" y="86.36" size="1.27" layer="95" rot="R270" align="center"/>
+<attribute name="VALUE" x="-147.32" y="86.36" size="1.27" layer="96" rot="R270" align="center"/>
 </instance>
-<instance part="R59" gate="G$1" x="121.92" y="-55.88" smashed="yes" rot="R90">
-<attribute name="NAME" x="119.38" y="-55.88" size="1.27" layer="95" rot="R90" align="center"/>
-<attribute name="VALUE" x="124.46" y="-55.88" size="1.27" layer="96" rot="R90" align="center"/>
+<instance part="R59" gate="G$1" x="134.62" y="-114.3" smashed="yes" rot="R90">
+<attribute name="NAME" x="132.08" y="-114.3" size="1.27" layer="95" rot="R90" align="center"/>
+<attribute name="VALUE" x="137.16" y="-114.3" size="1.27" layer="96" rot="R90" align="center"/>
 </instance>
-<instance part="R79" gate="G$1" x="132.08" y="-55.88" smashed="yes" rot="R90">
-<attribute name="NAME" x="129.54" y="-55.88" size="1.27" layer="95" rot="R90" align="center"/>
-<attribute name="VALUE" x="134.62" y="-55.88" size="1.27" layer="96" rot="R90" align="center"/>
+<instance part="R79" gate="G$1" x="144.78" y="-114.3" smashed="yes" rot="R90">
+<attribute name="NAME" x="142.24" y="-114.3" size="1.27" layer="95" rot="R90" align="center"/>
+<attribute name="VALUE" x="147.32" y="-114.3" size="1.27" layer="96" rot="R90" align="center"/>
 </instance>
-<instance part="R80" gate="G$1" x="142.24" y="-55.88" smashed="yes" rot="R90">
-<attribute name="NAME" x="139.7" y="-55.88" size="1.27" layer="95" rot="R90" align="center"/>
-<attribute name="VALUE" x="144.78" y="-55.88" size="1.27" layer="96" rot="R90" align="center"/>
+<instance part="R80" gate="G$1" x="-142.24" y="99.06" smashed="yes" rot="R90">
+<attribute name="NAME" x="-144.78" y="99.06" size="1.27" layer="95" rot="R90" align="center"/>
+<attribute name="VALUE" x="-139.7" y="99.06" size="1.27" layer="96" rot="R90" align="center"/>
 </instance>
-<instance part="GND170" gate="G$1" x="121.92" y="-78.74" smashed="yes">
-<attribute name="VALUE" x="121.92" y="-81.28" size="1.778" layer="96" align="center"/>
+<instance part="GND170" gate="G$1" x="134.62" y="-137.16" smashed="yes">
+<attribute name="VALUE" x="134.62" y="-139.7" size="1.778" layer="96" align="center"/>
 </instance>
-<instance part="GND171" gate="G$1" x="132.08" y="-78.74" smashed="yes">
-<attribute name="VALUE" x="132.08" y="-81.28" size="1.778" layer="96" align="center"/>
+<instance part="GND171" gate="G$1" x="144.78" y="-137.16" smashed="yes">
+<attribute name="VALUE" x="144.78" y="-139.7" size="1.778" layer="96" align="center"/>
 </instance>
-<instance part="GND172" gate="G$1" x="142.24" y="-78.74" smashed="yes">
-<attribute name="VALUE" x="142.24" y="-81.28" size="1.778" layer="96" align="center"/>
+<instance part="GND172" gate="G$1" x="-142.24" y="76.2" smashed="yes">
+<attribute name="VALUE" x="-142.24" y="73.66" size="1.778" layer="96" align="center"/>
 </instance>
 <instance part="R29" gate="G$1" x="162.56" y="-165.1" smashed="yes">
@@
 <pinref part="D6" gate="G$1" pin="K"/>
 <pinref part="GND170" gate="G$1" pin="GND"/>
-<wire x1="121.92" y1="-76.2" x2="121.92" y2="-73.66" width="0.1524" layer="91"/>
+<wire x1="134.62" y1="-134.62" x2="134.62" y2="-132.08" width="0.1524" layer="91"/>
 </segment>
 <segment>
 <pinref part="D7" gate="G$1" pin="K"/>
 <pinref part="GND171" gate="G$1" pin="GND"/>
-<wire x1="132.08" y1="-76.2" x2="132.08" y2="-73.66" width="0.1524" layer="91"/>
+<wire x1="144.78" y1="-134.62" x2="144.78" y2="-132.08" width="0.1524" layer="91"/>
 </segment>
 <segment>
 <pinref part="D5" gate="G$1" pin="K"/>
 <pinref part="GND172" gate="G$1" pin="GND"/>
-<wire x1="142.24" y1="-76.2" x2="142.24" y2="-73.66" width="0.1524" layer="91"/>
+<wire x1="-142.24" y1="78.74" x2="-142.24" y2="81.28" width="0.1524" layer="91"/>
 </segment>
 </net>
@@
 <pinref part="D6" gate="G$1" pin="A"/>
 <pinref part="R59" gate="G$1" pin="1"/>
-<wire x1="121.92" y1="-60.96" x2="121.92" y2="-63.5" width="0.1524" layer="91"/>
+<wire x1="134.62" y1="-119.38" x2="134.62" y2="-121.92" width="0.1524" layer="91"/>
 </segment>
 </net>
@@
 <pinref part="D7" gate="G$1" pin="A"/>
 <pinref part="R79" gate="G$1" pin="1"/>
-<wire x1="132.08" y1="-60.96" x2="132.08" y2="-63.5" width="0.1524" layer="91"/>
+<wire x1="144.78" y1="-119.38" x2="144.78" y2="-121.92" width="0.1524" layer="91"/>
 </segment>
 </net>
@@
 <pinref part="D5" gate="G$1" pin="A"/>
 <pinref part="R80" gate="G$1" pin="1"/>
-<wire x1="142.24" y1="-60.96" x2="142.24" y2="-63.5" width="0.1524" layer="91"/>
+<wire x1="-142.24" y1="93.98" x2="-142.24" y2="91.44" width="0.1524" layer="91"/>
 </segment>
 </net>
 <net name="FPGA_LED_0" class="0">
 <segment>
-<label x="144.78" y="-48.26" size="1.778" layer="95"/>
-<wire x1="165.1" y1="-48.26" x2="142.24" y2="-48.26" width="0.1524" layer="91"/>
+<label x="-139.7" y="106.68" size="1.778" layer="95"/>
+<wire x1="-119.38" y1="106.68" x2="-142.24" y2="106.68" width="0.1524" layer="91"/>
 <pinref part="R80" gate="G$1" pin="2"/>
-<wire x1="142.24" y1="-48.26" x2="142.24" y2="-50.8" width="0.1524" layer="91"/>
-</segment>
-</net>
-<net name="FPGA_LED_1" class="0">
-<segment>
-<label x="144.78" y="-45.72" size="1.778" layer="95"/>
-<wire x1="132.08" y1="-45.72" x2="165.1" y2="-45.72" width="0.1524" layer="91"/>
-<pinref part="R79" gate="G$1" pin="2"/>
-<wire x1="132.08" y1="-45.72" x2="132.08" y2="-50.8" width="0.1524" layer="91"/>
-</segment>
-</net>
-<net name="FPGA_LED_2" class="0">
-<segment>
-<label x="144.78" y="-43.18" size="1.778" layer="95"/>
-<wire x1="121.92" y1="-43.18" x2="165.1" y2="-43.18" width="0.1524" layer="91"/>
-<pinref part="R59" gate="G$1" pin="2"/>
-<wire x1="121.92" y1="-43.18" x2="121.92" y2="-50.8" width="0.1524" layer="91"/>
+<wire x1="-142.24" y1="106.68" x2="-142.24" y2="104.14" width="0.1524" layer="91"/>
+</segment>
+<segment>
+<pinref part="U1" gate="G$1" pin="GPIOR_119_CTRL12"/>
+<wire x1="-30.48" y1="-22.86" x2="-76.2" y2="-22.86" width="0.1524" layer="91"/>
+<label x="-73.66" y="-22.86" size="1.778" layer="95"/>
 </segment>
 </net>
@@
 </segment>
 </net>
+<net name="ESP_LED_0" class="0">
+<segment>
+<pinref part="U15" gate="G$1" pin="IO22"/>
+<wire x1="157.48" y1="-210.82" x2="106.68" y2="-210.82" width="0.1524" layer="91"/>
+<label x="127" y="-210.82" size="1.778" layer="95"/>
+</segment>
+<segment>
+<label x="157.48" y="-104.14" size="1.778" layer="95"/>
+<wire x1="144.78" y1="-104.14" x2="177.8" y2="-104.14" width="0.1524" layer="91"/>
+<pinref part="R79" gate="G$1" pin="2"/>
+<wire x1="144.78" y1="-104.14" x2="144.78" y2="-109.22" width="0.1524" layer="91"/>
+</segment>
+</net>
+<net name="ESP_LED_1" class="0">
+<segment>
+<pinref part="U15" gate="G$1" pin="IO23"/>
+<wire x1="157.48" y1="-213.36" x2="106.68" y2="-213.36" width="0.1524" layer="91"/>
+<label x="127" y="-213.36" size="1.778" layer="95"/>
+</segment>
+<segment>
+<label x="157.48" y="-101.6" size="1.778" layer="95"/>
+<wire x1="134.62" y1="-101.6" x2="177.8" y2="-101.6" width="0.1524" layer="91"/>
+<pinref part="R59" gate="G$1" pin="2"/>
+<wire x1="134.62" y1="-101.6" x2="134.62" y2="-109.22" width="0.1524" layer="91"/>
+</segment>
+</net>

Commit message: Updated release dates
Connections:
- removed net FT_CONT_RX: U1.GPIOB_RXN06
- removed net FT_CONT_TX: U1.GPIOB_RXN04
Other:
- note added: "2024.04.16 - GSWDH LTD. FILM SCANNER MAIN REVISION 3.0.0 DESIGN BY GEORGE WALLER AT GSWDH LTD. GEORGEWALLER@GSWDH.CO.UK CONFIDENTIAL. FOR THE INTENDED READER ONLY."
- note removed: "2024.03.19 - GSWDH LTD. FILM SCANNER MAIN REVISION 3.0.0 DESIGN BY GEORGE WALLER AT GSWDH LTD. GEORGEWALLER@GSWDH.CO.UK CONFIDENTIAL. FOR THE INTENDED READER ONLY."
Changed lines of the file:
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@@
 <description>COVER</description>
 <plain>
-<text x="0" y="0" size="7.62" layer="97" font="vector" align="center">2024.03.19 - GSWDH LTD.
+<text x="0" y="0" size="7.62" layer="97" font="vector" align="center">2024.04.16 - GSWDH LTD.
 FILM SCANNER MAIN
 REVISION 3.0.0
@@
 </segment>
 </net>
-<net name="FT_CONT_TX" class="0">
-<segment>
-<wire x1="-76.2" y1="-71.12" x2="-30.48" y2="-71.12" width="0.1524" layer="91"/>
-<pinref part="U1" gate="G$1" pin="GPIOB_RXN04"/>
-<label x="-73.66" y="-71.12" size="1.778" layer="95"/>
-</segment>
-</net>
 <net name="FT_D7" class="0">
 <segment>
@@
 </segment>
 </net>
-<net name="FT_CONT_RX" class="0">
-<segment>
-<wire x1="-30.48" y1="-76.2" x2="-76.2" y2="-76.2" width="0.1524" layer="91"/>
-<pinref part="U1" gate="G$1" pin="GPIOB_RXN06"/>
-<label x="-73.66" y="-76.2" size="1.778" layer="95"/>
-</segment>
-</net>
