File: sensor.brd (EAGLE design)
At the start: 50 x 151 mm, 64 parts, among them CN3 15PIN 0.5MM, U1 TCD2565BFG, U10 LT1806, U11 SN74LVC2G17, U12 SN74LVC2G17, U13 SN74LVC2G17, U14 SN74LVC2G17, U15 SN74LVC2G17, U19 AD5258BRMZ1-R7, U20 SN74LVC2G17, U21 AD5258BRMZ1-R7, U22 AD5258BRMZ1-R7, U3 ADS7056, U6 LT1806, U7 ADS7056, U8 LT1806, U9 ADS7056

Commit message: Controller nearly done
Parts:
- added C10, C9: 0.1uF 50V, c_0603:0603
- added C11: 100pF 50V, c_0603:0603
- added C8: 100uF 50V, CAPACITORS:8MM_RADIAL_3.5MM_PITCH
- added FB2: 600R, INDUCTORS:0603
- added Q2: KSC2690A, TRANSISTORs:TO126V
- added R11: 20k, r_0603:0603
- added R3: 10k, r_0603:0603
Connections:
- new net N$3: C11.2, C9.2, FB2.2, Q2.2, R3.2
- new net N$4: C8.P, Q2.3, R11.2, R3.1
- new net PWR_SENS_UNREG: C10.2, Q2.1
- net GND: now also C10.1, C11.1, C8.N, C9.1, R11.1
Changed lines of the file:
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@@
 <element name="MECH7" library="MISC" package="MOUNTHOLE_6X3" value="6mm x 3mm" x="22" y="54" smashed="yes" rot="R180"/>
 <element name="MECH8" library="MISC" package="MOUNTHOLE_6X3" value="6mm x 3mm" x="-22" y="54" smashed="yes" rot="R180"/>
+<element name="Q2" library="TRANSISTORs" package="TO126V" value="KSC2690A" x="-129.5" y="-111.125" smashed="yes">
+<attribute name="FARNELL" value="2453953" x="-129.5" y="-102.625" size="0.5" layer="27" display="off"/>
+<attribute name="NAME" x="-126.505" y="-112.685" size="1" layer="25" rot="R180"/>
+<attribute name="PRICE_PER" value="0.536" x="-129.5" y="-102.625" size="0.5" layer="27" display="off"/>
+</element>
+<element name="R3" library="r_0603" package="0603" value="10k" x="-130.875" y="-119.625" smashed="yes">
+<attribute name="DIGIKEY" value="541-2980-1-ND" x="-130.875" y="-107.875" size="0.5" layer="27" display="off"/>
+<attribute name="HEIGHT" value="1" x="-130.875" y="-107.875" size="0.5" layer="27" display="off"/>
+<attribute name="MANUFACTURER" value="Vishay Dale" x="-130.875" y="-107.875" size="0.5" layer="27" display="off"/>
+<attribute name="NAME" x="-132.375" y="-118.875" size="1.016" layer="25"/>
+<attribute name="POWER" value="0.1W, 1/10W" x="-130.875" y="-107.875" size="0.5" layer="27" display="off"/>
+<attribute name="PRICE_PER" value="0.12000" x="-130.875" y="-107.875" size="0.5" layer="27" display="off"/>
+<attribute name="STOCK" value="50797" x="-130.875" y="-107.875" size="0.5" layer="27" display="off"/>
+<attribute name="TOLERANCE" value="±1%" x="-130.875" y="-107.875" size="0.5" layer="27" display="off"/>
+</element>
+<element name="R11" library="r_0603" package="0603" value="20k" x="-127.375" y="-119.625" smashed="yes">
+<attribute name="DIGIKEY" value="541-20.0KHCT-ND" x="-130.875" y="-111.125" size="0.5" layer="27" display="off"/>
+<attribute name="HEIGHT" value="1" x="-130.875" y="-111.125" size="0.5" layer="27" display="off"/>
+<attribute name="MANUFACTURER" value="Vishay Dale" x="-130.875" y="-111.125" size="0.5" layer="27" display="off"/>
+<attribute name="NAME" x="-128.875" y="-118.875" size="1.016" layer="25"/>
+<attribute name="POWER" value="0.1W, 1/10W" x="-130.875" y="-111.125" size="0.5" layer="27" display="off"/>
+<attribute name="PRICE_PER" value="0.07000" x="-130.875" y="-111.125" size="0.5" layer="27" display="off"/>
+<attribute name="STOCK" value="25018" x="-130.875" y="-111.125" size="0.5" layer="27" display="off"/>
+<attribute name="TOLERANCE" value="±1%" x="-130.875" y="-111.125" size="0.5" layer="27" display="off"/>
+</element>
+<element name="C8" library="CAPACITORS" package="8MM_RADIAL_3.5MM_PITCH" value="100uF 50V" x="-128.75" y="-105.5" smashed="yes">
+<attribute name="DIGIKEY" value="1572-1044-ND" x="-128.75" y="-116.625" size="0.5" layer="27" display="off"/>
+<attribute name="HEIGHT" value="14" x="-128.75" y="-116.625" size="0.5" layer="27" display="off"/>
+<attribute name="NAME" x="-125.75" y="-102.5" size="1" layer="25"/>
+<attribute name="PRICE_PER" value="0.223" x="-128.75" y="-116.625" size="0.5" layer="27" display="off"/>
+</element>
+<element name="C9" library="c_0603" package="0603" value="0.1uF 50V" x="-123.875" y="-111.875" smashed="yes">
+<attribute name="DIGIKEY" value="478-5778-1-ND" x="-130.875" y="-123" size="0.5" layer="27" display="off"/>
+<attribute name="HEIGHT" value="-" x="-130.875" y="-123" size="0.5" layer="27" display="off"/>
+<attribute name="MANUFACTURER" value="AVX Corporation" x="-130.875" y="-123" size="0.5" layer="27" display="off"/>
+<attribute name="NAME" x="-125.375" y="-111.125" size="1.016" layer="25"/>
+<attribute name="PRICE_PER" value="0.07000" x="-130.875" y="-123" size="0.5" layer="27" display="off"/>
+<attribute name="STOCK" value="883194" x="-130.875" y="-123" size="0.5" layer="27" display="off"/>
+<attribute name="TEMP_CO" value="X7R" x="-130.875" y="-123" size="0.5" layer="27" display="off"/>
+<attribute name="TOLERANCE" value="±5%" x="-130.875" y="-123" size="0.5" layer="27" display="off"/>
+<attribute name="VOLTAGE" value="50V" x="-130.875" y="-123" size="0.5" layer="27" display="off"/>
+</element>
+<element name="C10" library="c_0603" package="0603" value="0.1uF 50V" x="-130.875" y="-116.375" smashed="yes">
+<attribute name="DIGIKEY" value="478-5778-1-ND" x="-130.875" y="-126.25" size="0.5" layer="27" display="off"/>
+<attribute name="HEIGHT" value="-" x="-130.875" y="-126.25" size="0.5" layer="27" display="off"/>
+<attribute name="MANUFACTURER" value="AVX Corporation" x="-130.875" y="-126.25" size="0.5" layer="27" display="off"/>
+<attribute name="NAME" x="-132.375" y="-115.625" size="1.016" layer="25"/>
+<attribute name="PRICE_PER" value="0.07000" x="-130.875" y="-126.25" size="0.5" layer="27" display="off"/>
+<attribute name="STOCK" value="883194" x="-130.875" y="-126.25" size="0.5" layer="27" display="off"/>
+<attribute name="TEMP_CO" value="X7R" x="-130.875" y="-126.25" size="0.5" layer="27" display="off"/>
+<attribute name="TOLERANCE" value="±5%" x="-130.875" y="-126.25" size="0.5" layer="27" display="off"/>
+<attribute name="VOLTAGE" value="50V" x="-130.875" y="-126.25" size="0.5" layer="27" display="off"/>
+</element>
+<element name="C11" library="c_0603" package="0603" value="100pF 50V" x="-127.375" y="-116.375" smashed="yes">
+<attribute name="DIGIKEY" value="478-06035A101J4T4ACT-ND" x="-130.875" y="-129.5" size="0.5" layer="27" display="off"/>
+<attribute name="HEIGHT" value="-" x="-130.875" y="-129.5" size="0.5" layer="27" display="off"/>
+<attribute name="MANUFACTURER" value="AVX Corporation" x="-130.875" y="-129.5" size="0.5" layer="27" display="off"/>
+<attribute name="NAME" x="-128.875" y="-115.625" size="1.016" layer="25"/>
+<attribute name="PRICE_PER" value="0.13000" x="-130.875" y="-129.5" size="0.5" layer="27" display="off"/>
+<attribute name="STOCK" value="29039" x="-130.875" y="-129.5" size="0.5" layer="27" display="off"/>
+<attribute name="TEMP_CO" value="C0G, NP0" x="-130.875" y="-129.5" size="0.5" layer="27" display="off"/>
+<attribute name="TOLERANCE" value="±5%" x="-130.875" y="-129.5" size="0.5" layer="27" display="off"/>
+<attribute name="VOLTAGE" value="50V" x="-130.875" y="-129.5" size="0.5" layer="27" display="off"/>
+</element>
+<element name="FB2" library="INDUCTORS" package="0603" value="600R" x="-123.875" y="-116.375" smashed="yes">
+<attribute name="DIGIKEY" value="732-1593-1-ND" x="-130.875" y="-132.75" size="0.5" layer="27" display="off"/>
+<attribute name="HEIGHT" value="1" x="-130.875" y="-132.75" size="0.5" layer="27" display="off"/>
+<attribute name="NAME" x="-125.375" y="-115.625" size="1.016" layer="25"/>
+<attribute name="PRICE_PER" value="0.13" x="-130.875" y="-132.75" size="0.5" layer="27" display="off"/>
+</element>
 </elements>
 <signals>
@@
 <contactref element="C62" pad="1"/>
 <contactref element="C63" pad="1"/>
+<contactref element="R11" pad="1"/>
+<contactref element="C8" pad="N"/>
+<contactref element="C9" pad="1"/>
+<contactref element="C11" pad="1"/>
+<contactref element="C10" pad="1"/>
+<wire x1="-128.125" y1="-116.375" x2="-128.125" y2="-119.625" width="0" layer="19" extent="1-1"/>
+<wire x1="-131.625" y1="-116.375" x2="-128.125" y2="-116.375" width="0" layer="19" extent="1-1"/>
+<wire x1="-124.625" y1="-111.875" x2="-128.125" y2="-116.375" width="0" layer="19" extent="1-1"/>
+<wire x1="-127" y1="-105.5" x2="-124.625" y2="-111.875" width="0" layer="19" extent="1-1"/>
+<wire x1="-77.5" y1="-100" x2="-124.625" y2="-111.875" width="0" layer="19" extent="1-1"/>
 <wire x1="-77.5" y1="-96.75" x2="-77.5" y2="-100" width="0" layer="19" extent="1-1"/>
 <wire x1="-77.5" y1="-93.5" x2="-77.5" y2="-96.75" width="0" layer="19" extent="1-1"/>
@@
 <contactref element="U20" pad="3"/>
 </signal>
+<signal name="N$3">
+<contactref element="Q2" pad="2"/>
+<contactref element="R3" pad="2"/>
+<contactref element="C9" pad="2"/>
+<contactref element="C11" pad="2"/>
+<contactref element="FB2" pad="2"/>
+<wire x1="-126.625" y1="-116.375" x2="-130.125" y2="-119.625" width="0" layer="19" extent="1-1"/>
+<wire x1="-123.125" y1="-116.375" x2="-126.625" y2="-116.375" width="0" layer="19" extent="1-1"/>
+<wire x1="-123.125" y1="-111.875" x2="-123.125" y2="-116.375" width="0" layer="19" extent="1-1"/>
+<wire x1="-129.5" y1="-111.125" x2="-126.625" y2="-116.375" width="0" layer="19" extent="1-1"/>
+</signal>
+<signal name="N$4">
+<contactref element="R3" pad="1"/>
+<contactref element="R11" pad="2"/>
+<contactref element="Q2" pad="3"/>
+<contactref element="C8" pad="P"/>
+<wire x1="-126.625" y1="-119.625" x2="-131.625" y2="-119.625" width="0" layer="19" extent="1-1"/>
+<wire x1="-127.25" y1="-111.125" x2="-126.625" y2="-119.625" width="0" layer="19" extent="1-1"/>
+<wire x1="-130.5" y1="-105.5" x2="-127.25" y2="-111.125" width="0" layer="19" extent="1-1"/>
+</signal>
+<signal name="PWR_SENS_UNREG">
+<contactref element="Q2" pad="1"/>
+<contactref element="C10" pad="2"/>
+<wire x1="-131.75" y1="-111.125" x2="-130.125" y2="-116.375" width="0" layer="19" extent="1-1"/>
+</signal>
 </signals>
