File: control.brd (EAGLE design)
At the start: 50 x 120 mm, 116 parts, among them CN1 632723300011, CN2 JST GH 10 Pin, CN3 15PIN 0.5MM, CN4 8 PIN FFC, CN5 NEB-21-R, CN6 S4B-XH-SM4-TB, Q1 GSFP0449, Q2 KSC2690A, SW1 DPDT, U18 T8Q144C4, U2 USBLC6-2SC6, U23 TMC2208-LA-T, U3 93LC56B-I/SN, U4 W25Q128JV, U5 TPS62065, U6 FT2232H

Commit message: Controller nearly done
Parts:
- removed FB1: 600R, INDUCTORS:0603
- removed Q2: KSC2690A, TRANSISTORs:TO126V
- added C1, C43: 100nF 16V, CAPACITORS:0603
- added C18, C19, C20, C40, C41, C42, C44, C45, C46: 10uF 50V, CAPACITORS:0805
- added C47: 0.1uF 50V, c_0603:0603
- added C48: NO FIT, c_0603:0603
- added L1: 15uH 6.5A, INDUCTORS:SRP1035A
- added L2: 2.2uH 3.5A, INDUCTORS:SRN5040
- added R15: 5.23k, r_0603:0603
- added R18: 34k, r_0603:0603
- added R19: 10k, r_0603:0603
- added U1: TPS54302, ICs:SOT23-6
- added U7: TPS563201, ICs:SOT23-6
- C3: value 100uF 50V -> 100pF 50V; device CAPACITORS:8MM_RADIAL_3.5MM_PITCH -> c_0603:0603
- C4: value 0.1uF 50V -> 10uF 50V; device c_0603:0603 -> CAPACITORS:1210
- C6: value 100pF 50V -> 100uF 50V; device c_0603:0603 -> CAPACITORS:8MM_RADIAL_3.5MM_PITCH
- CN1: value 632723300011 -> USB C 2.0; device CONNECTORs:CONN_632723X0001_WRE -> CONNECTORs:MC-107D
- R11, R12, R13, R14, R59: device r_0402:0402 -> r_0603:0603
- R2: value 10k -> 51k; device r_0603:0603 -> RESISTORS:0603
- R4: value 20k -> 100k
- moved R12 247.8 mm to (-23.1, 0.12), turned to 180 degrees
- moved D6 246.2 mm to (-20.4, 0.12), turned to 180 degrees
- moved R11 243.7 mm to (-23.1, 1.38), turned to 180 degrees
- moved D5 242.1 mm to (-20.4, 1.38), turned to 180 degrees
- moved R59 239.6 mm to (-23.1, 2.62), turned to 180 degrees
- moved D10 238.0 mm to (-20.4, 2.62), turned to 180 degrees
- moved R14 215.6 mm to (-23.1, -44.2), turned to 180 degrees
- moved C6 215.3 mm to (20.5, -22.0), turned to 90 degrees
- moved D8 214.1 mm to (-20.4, -44.2), turned to 180 degrees
- moved R13 209.1 mm to (-23.1, -45.5), turned to 180 degrees
- moved D7 207.6 mm to (-20.4, -45.5), turned to 180 degrees
- moved C5 204.3 mm to (12.4, -26.9), turned to 90 degrees
- moved C3 203.5 mm to (15.6, -18.8), turned to 180 degrees
- moved C4 201.7 mm to (14.5, -27.8), turned to 90 degrees
- moved R4 200.8 mm to (15.6, -17.5), turned to 180 degrees
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Connections:
- removed net PWR_SENS_UNREG: C5.2, Q2.1
- new net N$2: C1.1, U1.6
- new net N$20: C43.2, L2.1, U7.2
- new net N$25: C48.1, R18.1, R19.2, U7.4
- new net N$6: C1.2, L1.1, U1.2
- new net N$7: C3.2, R2.1, R4.2
- new net PWR_SYS_12V: C18.2, C19.2, C20.2, C40.2, C41.2, C42.2, C47.2, C65.2, C66.2, C67.1, L1.2, R2.2, U23.22, U23.28, U7.3, U7.5
- net GND: now also C18.1, C19.1, C20.1, C40.1, C41.1, C42.1, C44.1, C45.1, C46.1, C47.1, C6.N, CN1.A12B1, CN1.B12A1, CN1.P$1, CN1.P$10, CN1.P$11, CN1.P$12, CN1.P$13, CN1.P$14, CN1.P$15, CN1.P$16, CN1.P$17, CN1.P$18, CN1.P$19, CN1.P$2, CN1.P$20, CN1.P$21, CN1.P$22, CN1.P$23, CN1.P$24, CN1.P$3, CN1.P$4, CN1.P$5, CN1.P$6, CN1.P$7, CN1.P$8, CN1.P$9, R15.1, R19.1, U1.1, U7.1; no longer C3.N, C6.1, CN1.1, CN1.2, CN1.3, CN1.4, CN1.A1, CN1.A12, CN1.B1, CN1.B12, R4.1
- net N$10: now also C43.1, U7.6; no longer C3.P, Q2.3, R2.1, R4.2
- net N$41: now also CN1.A9B4, CN1.B9A4; no longer CN1.A4, CN1.A9, CN1.B4, CN1.B9
- net N$9: now also C3.1, R15.2, R4.1, U1.4; no longer C4.2, C6.2, FB1.2, Q2.2, R2.2
- net PWR_LED_24V: now also C4.2, C5.2, C6.P, U1.3; no longer FB1.1
- net PWR_STP_12V: no longer C65.2, C66.2, C67.1, U23.22, U23.28
- net PWR_SYS_3V3: now also C44.2, C45.2, C46.2, C48.2, L2.2, R18.2
Routing:
- net PWR_SYS_12V: track 0.00 -> 64.1 mm, vias 0 -> 1
- net GND: track 94.4 -> 134.0 mm, vias 87 -> 122
- net N$51: track 7.26 -> 33.9 mm
- net FLS_SPI_MOSI: track 0.00 -> 24.8 mm
- net FLS_SPI_CLK: track 1.76 -> 25.1 mm
- net PWR_SYS_3V3: track 70.3 -> 93.2 mm, vias 36 -> 42
- net FLS_SPI_MISO: track 0.00 -> 20.6 mm
- net FLS_SPI_NCS: track 1.75 -> 21.4 mm, vias 0 -> 2
- net FT_CONT_NTXLED: track 0.00 -> 18.7 mm, vias 0 -> 2
- net FPGA_CONF_NCRST: track 0.00 -> 17.0 mm, vias 0 -> 2
- net STP_DIR: track 0.00 -> 16.8 mm, vias 0 -> 1
- net FT_CONT_NRXLED: track 0.00 -> 16.3 mm, vias 0 -> 2
- net STP_NEN: track 0.00 -> 15.5 mm, vias 0 -> 1
- net N$41: track 0.00 -> 15.0 mm
- net FPGA_CONF_CSI: track 0.00 -> 15.0 mm, vias 0 -> 2
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
Commit message: Controller nearly complete
Parts:
- added CN7: 8 PIN FFC, CONNECTORs:SFV8R-1STBE1HLF
- added R20, R21: 10k, r_0603:0603
- moved C70 33.5 mm to (-20.8, 15.9)
- moved C64 32.6 mm to (-10.8, 14.6)
- moved C65 32.6 mm to (-18.0, 20.8)
- moved C66 32.6 mm to (-12.8, 20.8)
- moved C67 32.6 mm to (-21.8, 20.0)
- moved C68 32.6 mm to (-18.0, 11.5)
- moved C69 32.6 mm to (-20.0, 13.5)
- moved R16 32.6 mm to (-14.0, 20.8)
- moved R17 32.6 mm to (-16.8, 20.8)
- moved U23 32.6 mm to (-15.4, 16.1)
- moved CN3 30.6 mm to (9.00, 31.5)
- moved CN6 29.7 mm to (-9.38, 29.4)
- moved MECH3 25.0 mm to (-22.0, 32.0)
- moved MECH4 25.0 mm to (22.0, 32.0)
- moved D10 1.38 mm to (-20.4, 4.00)
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Connections:
- removed net FPGA_SPI_CLK: U18.112
- removed net FPGA_SPI_DATA: U18.111
- removed net FPGA_SPI_NCS: U18.110
- removed net GPIOB_CN0: U18.72
- removed net GPIOB_CP0: U18.71
- removed net GPIOB_N10: U18.68
- removed net GPIOB_N12: U18.69
- removed net GPIOB_P10: U18.67
- removed net GPIOB_P12: U18.70
- removed net GPIOL_68: U18.139
- removed net GPIOL_69: U18.138
- removed net GPIOL_70: U18.137
- removed net GPIOL_71: U18.136
- removed net GPIOL_72: U18.135
- removed net GPIOL_73: U18.134
- removed net GPIOL_74: U18.132
- removed net GPIOL_75: U18.131
- removed net GPIOR_104: U18.103
- removed net GPIOR_105: U18.102
- removed net GPIOR_112: U18.101
- removed net GPIOR_113: U18.100
- removed net GPIOR_116: U18.99
- removed net GPIOR_117: U18.98
- removed net GPIOR_122: U18.97
- removed net GPIOR_123: U18.93
- removed net GPIOR_125: U18.92
- removed net GPIOR_135: U18.84
- removed net GPIOR_136: U18.83
- removed net GPIOR_138: U18.82
- removed net GPIOR_139: U18.81
- removed net GPIOR_154: U18.77
- removed net GPIOR_155: U18.76
- removed net GPIOR_76: U18.124
- removed net GPIOR_77: U18.123
- removed net GPIOR_78: U18.119
- removed net GPIOR_79: U18.118
- removed net GPIOR_80: U18.117
- removed net GPIOR_81: U18.116
- removed net GPIOR_82: U18.115
- removed net GPIOR_83: U18.114
- removed net GPIOR_84: U18.113
- removed net GPIOR_88: U18.109
- removed net GPIOR_94: U18.106
- removed net GPIOR_95: U18.105
- removed net N$21: D6.K
- removed net N$22: D5.K
- removed net N$23: D10.K
- removed net PWR_STP_12V: C69.2
- new net FPGA_STATUS: D6.K, U18.83
- new net PROC_JTAG_TCK: CN7.3, R20.1, U18.97
- new net PROC_JTAG_TDI: CN7.2, U18.98
- new net PROC_JTAG_TDO: CN7.5, R21.1, U18.92
- new net PROC_JTAG_TMS: CN7.4, U18.93
- new net PROC_SCANNING: D10.K, U18.81
- new net PROC_STATUS: D5.K, U18.82
- net FT_CLKOUT: now also U18.123
- net FT_CONT_NCTS: now also U18.109
- net FT_CONT_NDCD: now also U18.103
- net FT_CONT_NDSR: now also U18.105
- net FT_CONT_NDTR: now also U18.106
- net FT_CONT_NRI: now also U18.102
- net FT_CONT_NRTS: now also U18.110
- net FT_CONT_PWRSAV: now also U18.99
- net FT_CONT_RX: now also U18.111
- net FT_CONT_TX: now also U18.112
- net FT_CONT_TXDEN: now also U18.101
- net FT_D0: now also U18.139
- net FT_D1: now also U18.138
- net FT_D2: now also U18.137
- net FT_D3: now also U18.136
- net FT_D4: now also U18.135
- net FT_D5: now also U18.134
- net FT_D6: now also U18.132
- net FT_D7: now also U18.131
- net FT_NOE: now also U18.115
- net FT_NPWREN: now also U18.100
- net FT_NRD: now also U18.119
- net FT_NRST: now also U18.124
- net FT_NRXF: now also U18.117
- net FT_NSIWU: now also U18.114
- net FT_NSUSPEND: now also U18.113
- net FT_NTXE: now also U18.116
- net FT_NWR: now also U18.118
- net GND: now also CN7.8
- net PWR_SYS_12V: now also C69.2
- net PWR_SYS_3V3: now also CN7.1, R20.2, R21.2
- net STP_CLK: now also U18.71
- net STP_DIA: now also U18.84
- net STP_DIR: now also U18.68
- net STP_IDX: now also U18.72
- net STP_MS1: now also U18.76
- net STP_MS2: now also U18.77
- net STP_NEN: now also U18.67
- net STP_STP: now also U18.69
- net STP_UART_IO: now also U18.70
Routing:
- net PWR_SYS_12V: track 64.1 -> 128.7 mm, vias 1 -> 2
- net PWR_LED_24V: track 3.41 -> 58.3 mm
- net FT_D0: track 0.00 -> 37.4 mm, vias 0 -> 2
- net FT_D1: track 0.00 -> 35.7 mm, vias 0 -> 2
- net FT_D3: track 0.00 -> 35.6 mm, vias 0 -> 2
- net FT_D2: track 0.00 -> 34.2 mm, vias 0 -> 2
- net FT_D4: track 0.00 -> 33.1 mm, vias 0 -> 2
- net FT_NRST: track 0.00 -> 32.7 mm, vias 0 -> 2
- net FT_D5: track 0.00 -> 31.9 mm, vias 0 -> 2
- net FT_CONT_PWRSAV: track 4.18 -> 35.6 mm, vias 1 -> 2
- net FT_D6: track 0.00 -> 31.4 mm, vias 0 -> 2
- net FT_D7: track 0.00 -> 30.0 mm, vias 0 -> 2
- net FT_NPWREN: track 6.71 -> 36.7 mm, vias 1 -> 2
- net FT_CONT_TXDEN: track 0.00 -> 28.3 mm, vias 0 -> 2
- net FT_CONT_NDCD: track 0.00 -> 26.7 mm, vias 0 -> 2
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Other:
- board size 50 x 120 mm -> 50 x 95 mm
- board text added: "JTAG (FPGA)"
- board text added: "JTAG (PROC)"
