File: control.sch (EAGLE design)
At the start: 116 parts, among them CN1 632723300011, CN2 JST GH 10 Pin, CN3 15PIN 0.5MM, CN4 8 PIN FFC, CN5 NEB-21-R, CN6 S4B-XH-SM4-TB, Q1 GSFP0449, Q2 KSC2690A, SW1 DPDT, U18 T8Q144C4, U2 USBLC6-2SC6, U23 TMC2208-LA-T, U3 93LC56B-I/SN, U4 W25Q128JV, U5 TPS62065, U6 FT2232H

Commit message: Controller nearly done
Parts:
- removed FB1: 600R, INDUCTORS:742792651
- removed Q2: KSC2690A, TRANSISTORs:KSC2690AV
- added C1, C43: 100nF 16V, CAPACITORS:CL10B104KO8WPNC
- added C18, C19, C20, C40, C41, C42, C44, C45, C46: 10uF 50V, CAPACITORS:CL21A106KAYNNNE
- added C47: 0.1uF 50V, c_0603:06035C104JAT2A
- added C48: NO FIT, c_0603:06035A101J4T4A
- added L1: 15uH 6.5A, INDUCTORS:MWSA1004S-150MT
- added L2: 2.2uH 3.5A, INDUCTORS:SRN5040-2R2Y
- added R15: 5.23k, r_0603:CRCW06035K23FKEA
- added R18: 34k, r_0603:CRCW060334K0FKEA
- added R19: 10k, r_0603:CRCW060310K0FKTA
- added U1: TPS54302, ICs:TPS54302
- added U7: TPS563201, ICs:TPS563201DDCR
- C3: value 100uF 50V -> 100pF 50V; device CAPACITORS:107CKR050M -> c_0603:06035A101J4T4A
- C4: value 0.1uF 50V -> 10uF 50V; device c_0603:06035C104JAT2A -> CAPACITORS:C3225X7S1H106M250AB
- C6: value 100pF 50V -> 100uF 50V; device c_0603:06035A101J4T4A -> CAPACITORS:107CKR050M
- CN1: value 632723300011 -> USB C 2.0; device CONNECTORs:632723300011 -> CONNECTORs:MC-107D
- R11, R12, R13, R14, R59: device r_0402:RC0402FR-072K2L -> r_0603:CRCW06032K20FKEA
- R2: value 10k -> 51k; device r_0603:CRCW060310K0FKTA -> RESISTORS:CRCW060351K0FKEA
- R4: value 20k -> 100k; device r_0603:CRCW060320K0FKEA -> r_0603:CRCW0603100KFKEB
Connections:
- removed net PWR_SENS_UNREG: C5.2, Q2.E
- new net N$2: C1.1, U1.BOOT
- new net N$20: C43.2, L2.1, U7.SW
- new net N$25: C48.1, R18.1, R19.2, U7.FB
- new net N$6: C1.2, L1.1, U1.SW
- new net N$7: C3.2, R2.1, R4.2
- new net PWR_SYS_12V: C18.2, C19.2, C20.2, C40.2, C41.2, C42.2, C47.2, C65.2, C66.2, C67.A, L1.2, R2.2, U23.VS, U7.EN, U7.VIN
- net GND: now also C18.1, C19.1, C20.1, C40.1, C41.1, C42.1, C44.1, C45.1, C46.1, C47.1, C6.K, R15.1, R19.1, U1.GND, U7.GND; no longer C3.K, C6.1, CN1.SHELL, R4.1
- net N$10: now also C43.1, U7.BOOT; no longer C3.A, Q2.B, R2.1, R4.2
- net N$9: now also C3.1, R15.2, R4.1, U1.FB; no longer C4.2, C6.2, FB1.2, Q2.C, R2.2
- net PWR_LED_24V: now also C4.2, C5.2, C6.A, U1.VIN; no longer FB1.1
- net PWR_STP_12V: no longer C65.2, C66.2, C67.A, U23.VS
- net PWR_SYS_3V3: now also C44.2, C45.2, C46.2, C48.2, L2.2, R18.2
Other:
- moved on the sheet: C4, C5, R2, R4

Commit message: Controller nearly complete
Parts:
- added CN7: 8 PIN FFC, CONNECTORs:SFV8R-1STBE1HLF
- added R20, R21: 10k, r_0603:ERJ3EKF1002V
Connections:
- removed net FPGA_SPI_CLK: U18.GPIOR_86
- removed net FPGA_SPI_DATA: U18.GPIOR_85
- removed net FPGA_SPI_NCS: U18.GPIOR_87_CDI29
- removed net GPIOB_CN0: U18.GPIOB_CLKN0
- removed net GPIOB_CP0: U18.GPIOB_CLKP0
- removed net GPIOB_N10: U18.GPIOB_RXN10
- removed net GPIOB_N12: U18.GPIOB_RXN12_EXTFB0
- removed net GPIOB_P10: U18.GPIOB_RXP10
- removed net GPIOB_P12: U18.GPIOB_RXP12_EXTFB0
- removed net GPIOL_68: U18.GPIOL_68
- removed net GPIOL_69: U18.GPIOL_69_CBSEL1
- removed net GPIOL_70: U18.GPIOL_70_CBSEL0
- removed net GPIOL_71: U18.GPIOL_71_NSTATUS
- removed net GPIOL_72: U18.GPIOL_72_EXTFB0_CDI14
- removed net GPIOL_73: U18.GPIOL_73_EXTFB1_CDI15
- removed net GPIOL_74: U18.GPIOL_74_PLLIN0
- removed net GPIOL_75: U18.GPIOL_75_PLLIN1
- removed net GPIOR_104: U18.GPIOR_104_CDI25
- removed net GPIOR_105: U18.GPIOR_105_CDI24
- removed net GPIOR_112: U18.GPIOR_112_CDI23
- removed net GPIOR_113: U18.GPIOR_113_CDI22
- removed net GPIOR_116: U18.GPIOR_116_CTRL15
- removed net GPIOR_117: U18.GPIOR_117_CTRL14
- removed net GPIOR_122: U18.GPIOR_122_CLK13_CDI21
- removed net GPIOR_123: U18.GPIOR_123_CLK12_CDI20
- removed net GPIOR_125: U18.GPIOR_125_CLK10
- removed net GPIOR_135: U18.GPIOR_135_CDI17
- removed net GPIOR_136: U18.GPIOR_136_CDI16
- removed net GPIOR_138: U18.GPIOR_138
- removed net GPIOR_139: U18.GPIOR_139
- removed net GPIOR_154: U18.GPIOR_154
- removed net GPIOR_155: U18.GPIOR_155
- removed net GPIOR_76: U18.GPIOR_76_PLLIN0
- removed net GPIOR_77: U18.GPIOR_77_PLLIN1
- removed net GPIOR_78: U18.GPIOR_78_EXTFB0_CDI31
- removed net GPIOR_79: U18.GPIOR_79_EXTFB1_CDI30
- removed net GPIOR_80: U18.GPIOR_80
- removed net GPIOR_81: U18.GPIOR_81_MREFCLK
- removed net GPIOR_82: U18.GPIOR_82
- removed net GPIOR_83: U18.GPIOR_83
- removed net GPIOR_84: U18.GPIOR_84
- removed net GPIOR_88: U18.GPIOR_88_CDI28
- removed net GPIOR_94: U18.GPIOR_94_CDI27
- removed net GPIOR_95: U18.GPIOR_95_CDI26
- removed net N$21: D6.K
- removed net N$22: D5.K
- removed net N$23: D10.K
- removed net PWR_STP_12V: C69.2
- new net FPGA_STATUS: D6.K, U18.GPIOR_136_CDI16
- new net PROC_JTAG_TCK: CN7.3, R20.1, U18.GPIOR_122_CLK13_CDI21
- new net PROC_JTAG_TDI: CN7.2, U18.GPIOR_117_CTRL14
- new net PROC_JTAG_TDO: CN7.5, R21.1, U18.GPIOR_125_CLK10
- new net PROC_JTAG_TMS: CN7.4, U18.GPIOR_123_CLK12_CDI20
- new net PROC_SCANNING: D10.K, U18.GPIOR_139
- new net PROC_STATUS: D5.K, U18.GPIOR_138
- net FT_CLKOUT: now also U18.GPIOR_77_PLLIN1
- net FT_CONT_NCTS: now also U18.GPIOR_88_CDI28
- net FT_CONT_NDCD: now also U18.GPIOR_104_CDI25
- net FT_CONT_NDSR: now also U18.GPIOR_95_CDI26
- net FT_CONT_NDTR: now also U18.GPIOR_94_CDI27
- net FT_CONT_NRI: now also U18.GPIOR_105_CDI24
- net FT_CONT_NRTS: now also U18.GPIOR_87_CDI29
- net FT_CONT_PWRSAV: now also U18.GPIOR_116_CTRL15
- net FT_CONT_RX: now also U18.GPIOR_85
- net FT_CONT_TX: now also U18.GPIOR_86
- net FT_CONT_TXDEN: now also U18.GPIOR_112_CDI23
- net FT_D0: now also U18.GPIOL_68
- net FT_D1: now also U18.GPIOL_69_CBSEL1
- net FT_D2: now also U18.GPIOL_70_CBSEL0
- net FT_D3: now also U18.GPIOL_71_NSTATUS
- net FT_D4: now also U18.GPIOL_72_EXTFB0_CDI14
- net FT_D5: now also U18.GPIOL_73_EXTFB1_CDI15
- net FT_D6: now also U18.GPIOL_74_PLLIN0
- net FT_D7: now also U18.GPIOL_75_PLLIN1
- net FT_NOE: now also U18.GPIOR_82
- net FT_NPWREN: now also U18.GPIOR_113_CDI22
- net FT_NRD: now also U18.GPIOR_78_EXTFB0_CDI31
- net FT_NRST: now also U18.GPIOR_76_PLLIN0
- net FT_NRXF: now also U18.GPIOR_80
- net FT_NSIWU: now also U18.GPIOR_83
- net FT_NSUSPEND: now also U18.GPIOR_84
- net FT_NTXE: now also U18.GPIOR_81_MREFCLK
- net FT_NWR: now also U18.GPIOR_79_EXTFB1_CDI30
- net GND: now also CN7.8
- net PWR_SYS_12V: now also C69.2
- net PWR_SYS_3V3: now also CN7.1, R20.2, R21.2
- net STP_CLK: now also U18.GPIOB_CLKP0
- net STP_DIA: now also U18.GPIOR_135_CDI17
- net STP_DIR: now also U18.GPIOB_RXN10
- net STP_IDX: now also U18.GPIOB_CLKN0
- net STP_MS1: now also U18.GPIOR_155
- net STP_MS2: now also U18.GPIOR_154
- net STP_NEN: now also U18.GPIOB_RXP10
- net STP_STP: now also U18.GPIOB_RXN12_EXTFB0
- net STP_UART_IO: now also U18.GPIOB_RXP12_EXTFB0
