File: main.brd (EAGLE design)
At the start: 130 x 34 mm, 104 parts, among them CN1 DC-012A-D010, CN2 JST GH 6P V-TH, CN3 5.8ZSPT, CN5 MC-118LS-H100, CN6 JST GH 6P V-TH, Q1 GSFP0449, Q6 IRLML6244, U1 T20F169, U11 TPS70918, U12 AP7335, U2 USBLC6-2SC6, U24 SCHMITT, U25 SCHMITT, U37 W25Q128JV, U5 TPS62065, U7 TPS563201, U8 AR0822, U9 TPS62065

Commit message: Initial layout done
Parts:
- removed U37: W25Q128JV, ICs:SO8-208MIL
- added C22, C28, C34, C38, C52, C53, C54, C55, C56, C57, C59, C61, C64, C65, C66, C67, C72, C73, C74, C75, C76, C78, C79, C82: 0.1uF 16V, c_0402:0402
- added C23, C24: 10pF 10V, c_0402:0402
- added C58, C62, C63, C71, C77, C80: 10uF 6.3V, c_0402:0402
- added CN4, CN8: FFC 8P 0.5mm, CONNECTORs:HC-FPC-05-09-8RLTAG
- added R10: 2.2k, r_0402:0402
- added R11, R12, R13, R137, R138, R14, R140, R141, R142, R143, R144, R146, R147, R16, R26, R7, R76, R77, R8, R9: 10k, r_0402:0402
- added R17: 20k, r_0402:0402
- added R20: 16k, r_0402:0402
- added R21: 51k, r_0402:0402
- added R25: 24k, r_0402:0402
- added R6: 12k, r_0402:0402
- added U10: AP7335, ICs:DFN2020-6
- added U13: W958D8NBYA5I, ICs:VBGA24
- added U3: 93LC56B-I/SN, ICs:SO8
- added U4: W25Q128JV, ICs:SO8-208MIL
- added U6: FT2232H, ICs:QFN64
- added XTAL2: 12MHz, CRYSTALS:3.2X3.5SMD
- C25: value 0.1uF 10V -> 0.1uF 16V
- C27: value 0.1uF 10V -> 1uF 10V
- C43: value 100nF 16V -> 0.1uF 16V; device CAPACITORS:0603 -> c_0402:0402
- C48: device c_0603:0603 -> c_0402:0402
- C49: value 2.2uF 6.3V -> 1uF 10V
- C7: value 100pF 50V -> 100pF 25V; device c_0603:0603 -> c_0402:0402
- R1, R18, R19, R5, R68, R72, R73: device r_0603:0603 -> r_0402:0402
- R58, R66: value 20k -> 10k
- U11: value TPS70918 -> AP7335; device ICs:SOT23-5 -> ICs:DFN2020-6
- moved CN5 77.5 mm to (-57.5, 0.00)
- moved R3 66.7 mm to (-24.1, -7.25), turned to 0 degrees
- moved OSC1 66.1 mm to (-24.0, -9.38), turned to 90 degrees
- moved C25 57.5 mm to (-24.0, -11.4), turned to 180 degrees
- moved U2 56.2 mm to (-42.5, -14.0), turned to 90 degrees
- moved U11 42.1 mm to (-11.5, 2.75), turned to 0 degrees
- moved C49 41.9 mm to (-9.12, 2.12), turned to 0 degrees
- moved C41 37.6 mm to (-15.2, 8.50), flipped to the top, turned to 90 degrees
- moved C27 33.1 mm to (-15.2, 13.2), turned to 270 degrees
- moved C69 18.2 mm to (40.6, -6.75)
- moved C70 18.2 mm to (36.0, -6.75)
- moved U24 18.2 mm to (38.6, -7.50)
- moved U25 18.2 mm to (34.0, -7.50)
- moved R72 18.1 mm to (38.1, -10.2)
- moved R73 18.1 mm to (33.5, -10.2)
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Connections:
- removed net PSS_CLK_33M: R3.2
- removed net PSS_FLASH_D0: U37.5
- removed net PSS_FLASH_D1: U37.2
- removed net PSS_FLASH_D2: U37.3
- removed net PSS_FLASH_D3: U37.7
- removed net PSS_FLASH_NCS: U37.1
- removed net PSS_FLASH_SCLK: U37.6
- removed net PWR_FPGA_0V95: C37.2, C39.2, L3.2, R148.2
- new net FLS_NHOLD: R138.1, U4.7
- new net FLS_SPI_CLK: R144.1, U1.K1, U4.6
- new net FLS_SPI_MISO: R12.1, U1.J2, U4.2
- new net FLS_SPI_MOSI: R11.1, U1.J1, U4.5
- new net FLS_SPI_NCS: R142.1, U1.L1, U4.1
- new net FPGA_CLK33M: R3.2, U1.J12
- new net FPGA_CONF_CBUS_0: R141.1, U1.J11
- new net FPGA_CONF_CBUS_1: R140.1, U1.G13
- new net FPGA_CONF_CDONE: R147.1, U1.L2
- new net FPGA_CONF_NCRST: C66.2, CN8.7, R146.1, U1.K3
- new net FPGA_CONF_NTEST: R143.1, U1.H12
- new net FPGA_JTAG_TCK: CN8.4, R76.1, U1.H1
- new net FPGA_JTAG_TDI: CN8.5, U1.J3
- new net FPGA_JTAG_TDO: CN8.2, R77.1, U1.G1
- new net FPGA_JTAG_TMS: CN8.3, U1.H2
- new net FT_CLKOUT: U1.M13, U6.32
- new net FT_CONT_RX: U1.L10, U6.39
- new net FT_CONT_TX: U1.L9, U6.38
- new net FT_D0: U1.M12, U6.16
- new net FT_D1: U1.N12, U6.17
- new net FT_D2: U1.M11, U6.18
- new net FT_D3: U1.N11, U6.19
- new net FT_D4: U1.M10, U6.21
- new net FT_D5: U1.N10, U6.22
- new net FT_D6: U1.M9, U6.23
- new net FT_D7: U1.N9, U6.24
- new net FT_NOE: U1.L7, U6.33
- new net FT_NRD: U1.N8, U6.28
- new net FT_NRST: U1.L11, U6.14
- new net FT_NRXF: U1.L8, U6.26
- new net FT_NSIWU: U1.N7, U6.30
- new net FT_NTXE: U1.M8, U6.27
- new net FT_NWR: U1.M7, U6.29
- new net LED_FT_CONT_NRXLED: U6.54
- new net LED_FT_CONT_NTXLED: U6.55
- new net N$17: R21.1, R25.2, U11.6
- new net N$23: R26.1, U1.N4
- new net N$38: R137.1, U4.3
- new net N$42: R6.2, U6.6
- new net N$43: R7.1, U3.1, U6.63
- new net N$44: R8.1, U3.2, U6.62
- new net N$45: R10.2, U3.3, U6.61
- new net N$46: R10.1, R9.1, U3.4
- new net N$49: C23.2, U6.3, XTAL2.3
- new net N$50: C24.2, U6.2, XTAL2.1
- new net N$51: C55.2, C56.2, C57.2, C58.2, U6.12, U6.37, U6.49, U6.64
- new net N$8: R17.1, R20.2, U10.6
- new net PROC_JTAG_TCK: CN4.4, R13.1, U1.N3
- new net PROC_JTAG_TDI: CN4.5, U1.M5
- new net PROC_JTAG_TDO: CN4.2, R14.1, U1.N2
- new net PROC_JTAG_TMS: CN4.3, U1.F2
- new net PROC_NRST: CN4.7, R16.1, U1.G3
- new net PWR_FPGA_1V2: C37.2, C39.2, C71.2, C72.2, C73.2, C74.2, C75.2, C76.2, L3.2, R148.2, U1.C3, U1.E10, U1.E4, U1.E6, U1.E8, U1.F7, U1.F9, U1.G10, U1.G4, U1.G5, U1.G8, U1.G9, U1.H6, U1.J10, U1.J6
- new net PWR_FPGA_2V5: C62.2, C82.2, R21.2, U1.E7, U1.E9, U11.4
- new net RAM_CLK_N: U1.M1, U13.B1
- new net RAM_CLK_P: U1.M2, U13.B2
- new net RAM_D0: U1.N6, U13.D3
- new net RAM_D1: U1.K5, U13.D2
- new net RAM_D2: U1.M6, U13.C4
- new net RAM_D3: U1.L6, U13.D4
- new net RAM_D4: U1.K6, U13.D5
- new net RAM_D5: U1.N5, U13.E3
- new net RAM_D6: U1.M3, U13.E2
- new net RAM_D7: U1.L4, U13.E1
- new net RAM_NCS: U1.L3, U13.A3
- new net RAM_NRST: U1.K4, U13.A4
- new net RAM_RWDS: U1.L5, U13.C3
- net AR_CLK: now also U1.F3
- net AR_GPIO0: now also U1.C1
- net AR_GPIO1: now also U1.C2
- net AR_GPIO2: now also U1.D1
- net AR_GPIO3: now also U1.D2
- net AR_I2C_SCL: now also U1.E1
- net AR_I2C_SDA: now also U1.F1
- net AR_MIPI_CLK_N: now also U1.B12
- net AR_MIPI_CLK_P: now also U1.A12
- net AR_MIPI_D0_N: now also U1.C10
- net AR_MIPI_D0_P: now also U1.D10
- net AR_MIPI_D1_N: now also U1.A11
- net AR_MIPI_D1_P: now also U1.B11
- net AR_MIPI_D2_N: now also U1.C13
- net AR_MIPI_D2_P: now also U1.B13
- net AR_MIPI_D3_N: now also U1.D12
- net AR_MIPI_D3_P: now also U1.C12
- net AR_NRESET: now also U1.E3
- net AR_XSHUTDOWN: now also U1.B1
- net GND: now also C22.1, C23.1, C24.1, C28.1, C34.1, C38.1, C52.1, C53.1, C54.1, C55.1, C56.1, C57.1, C58.1, C59.1, C61.1, C62.1, C63.1, C64.1, C65.1, C66.1, C67.1, C71.1, C72.1, C73.1, C74.1, C75.1, C76.1, C77.1, C78.1, C79.1, C80.1, C82.1, CN4.1, CN8.1, R20.1, R25.1, R26.2, R6.1, U1.A1, U1.A13, U1.C11, U1.D11, U1.D3, U1.E12, U1.E2, U1.E5, U1.F5, U1.F6, U1.F8, U1.G6, U1.G7, U1.J7, U1.J8, U1.K12, U1.K2, U1.L12, U1.M4, U1.N1, U1.N13, U10.2, U10.7, U11.7, U13.B3, U13.C1, U13.E5, U3.5, U4.4, U6.1, U6.10, U6.11, U6.13, U6.15, U6.25, U6.35, U6.41, U6.44, U6.45, U6.47, U6.5, U6.51, U6.PAD, XTAL2.2, XTAL2.4; no longer U37.4
- net LED_PWM_CONT: now also U1.F12
- net MTR_SENSE_A: now also U1.E13
- net MTR_SENSE_B: now also U1.F13
- net PWR_SYS_1V8: now also C41.2, C63.2, C64.2, C65.2, C67.2, R17.2, U1.F4, U1.H4, U1.H5, U1.J5, U10.4, U13.B4, U13.D1, U13.E4; no longer C25.2, C49.2, OSC1.1, OSC1.4, U11.5
- net PWR_SYS_3V3: now also C22.2, C25.2, C28.2, C34.2, C38.2, C49.2, C52.2, C53.2, C54.2, C59.2, C61.2, C77.2, C78.2, C79.2, C80.2, CN4.8, CN8.8, OSC1.1, OSC1.4, R11.2, R12.2, R13.2, R137.2, R138.2, R14.2, R140.2, R141.2, R142.2, R143.2, R144.2, R146.2, R147.2, R16.2, R7.2, R76.2, R77.2, R8.2, R9.2, U1.F10, U1.H10, U1.H7, U1.H8, U1.H9, U1.J4, U1.J9, U10.1, U10.3, U3.8, U4.8, U6.20, U6.31, U6.4, U6.42, U6.46, U6.50, U6.56, U6.59, U6.9; no longer C41.2, U37.8
- net USB_D_N: now also U6.7
- net USB_D_P: now also U6.8
Routing:
- net GND: track 100.7 -> 168.9 mm, vias 97 -> 177
- net MTR_SENSE_A: track 0.00 -> 65.8 mm, vias 0 -> 1
- net PWR_SYS_1V8: track 27.1 -> 89.0 mm, vias 4 -> 12
- net MTR_SENSE_B: track 0.00 -> 61.5 mm, vias 0 -> 1
- net LED_PWM_CONT: track 0.00 -> 58.6 mm, vias 0 -> 1
- net PWR_SYS_3V3: track 43.9 -> 90.0 mm, vias 10 -> 47
- net USB_VBUS: track 0.00 -> 42.7 mm, vias 0 -> 1
- net N$51: track 0.00 -> 33.3 mm, vias 0 -> 4
- net PROC_NRST: track 0.00 -> 32.4 mm, vias 0 -> 1
- net PROC_JTAG_TMS: track 0.00 -> 29.2 mm, vias 0 -> 3
- net N$12: track 0.00 -> 27.3 mm, vias 0 -> 2
- net N$13: track 0.00 -> 26.2 mm, vias 0 -> 1
- net FLS_SPI_MOSI: track 0.00 -> 25.9 mm
- net PWR_FPGA_1V2: track 0.00 -> 25.1 mm, vias 0 -> 16
- net PROC_JTAG_TDI: track 0.00 -> 23.9 mm, vias 0 -> 1
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- added copper zone on layer 1, net GND
- added copper zone on layer 16, net GND
- added copper zone on layer 3, net PWR_FPGA_1V2
- removed copper zone on layer 3, net PWR_DDR3_1V35
