File: main.brd (EAGLE design)
At the start: 130 x 34 mm, 196 parts, among them CN1 DC-012A-D010, CN2 JST GH 6P V-TH, CN3 5.8ZSPT, CN5 MC-118LS-H100, CN6 JST GH 6P V-TH, CN8 FFC 8P 0.5mm, Q1 GSFP0449, Q2 MMBT3904, Q3 MMBT3904, U1 T20F169, U10 AP7335, U11 AP7335, U12 AP7335, U13 W958D8NBYA5I, U14 AS4950, U15 ESP32, U16 PI4ULS3V204ZBEX, U2 USBLC6-2SC6, U24 SCHMITT, U3 93LC56B-I/SN, U4 SCHMITT, U5 TPS62065, U6 FT2232H, U7 TPS563201, U8 AR0822, U9 TPS62065

Commit message: DRC compelte. Top and bottom copper fill.  Pushed to Fusion
Routing:
- net GND: track 193.6 -> 194.1 mm
- added copper zone on layer 1, net GND
- added copper zone on layer 16, net GND
Changed lines of the file:
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@@
 </layers>
 <board>
-<fusionsync huburn="a.YnVzaW5lc3M6bXl1Y2wxNDk2" projecturn="a.YnVzaW5lc3M6bXl1Y2wxNDk2IzIwMjIwMzI1NTEwNjk2MjUx" f3durn="urn:adsk.wipprod:dm.lineage:P9SLlJ01T8W2nK3aE3uNkQ" pcbguid="" lastpulledtime="" lastsyncedchangeguid="" latestrevisionid="1badfdd0-5c60-406b-8db1-5a285c325208" lastsyncedrevisionid="1badfdd0-5c60-406b-8db1-5a285c325208" lastboardhashguid="6285d1a9-6f23-04d9-8519-e9656412f81e" lastpushedtime="2024-04-14T18:23:25Z" linktopcb3d="true"/>
+<fusionsync huburn="a.YnVzaW5lc3M6bXl1Y2wxNDk2" projecturn="a.YnVzaW5lc3M6bXl1Y2wxNDk2IzIwMjIwMzI1NTEwNjk2MjUx" f3durn="urn:adsk.wipprod:dm.lineage:P9SLlJ01T8W2nK3aE3uNkQ" pcbguid="" lastpulledtime="" lastsyncedchangeguid="" latestrevisionid="b00044a3-fe5d-49ae-9846-cf26a2e424a0" lastsyncedrevisionid="b00044a3-fe5d-49ae-9846-cf26a2e424a0" lastboardhashguid="a5ae111e-9ae0-ac62-7b0b-17c3a497e20e" lastpushedtime="2024-04-14T19:21:15Z" linktopcb3d="true"/>
 <plain>
 <wire x1="-65" y1="14" x2="-65" y2="-14" width="0" layer="20" locked="yes"/>
@@
 <wire x1="37.625" y1="-4.625" x2="36.875" y2="-4.625" width="0.1016" layer="16"/>
 <via x="36.875" y="-4.625" extent="1-16" drill="0.3"/>
-<wire x1="37.625" y1="-6" x2="37.625" y2="-6.875" width="0.1016" layer="16"/>
-<via x="37.625" y="-6.875" extent="1-16" drill="0.3"/>
+<wire x1="37.625" y1="-6" x2="37.5" y2="-6.125" width="0.1016" layer="16"/>
+<wire x1="37.5" y1="-6.125" x2="37" y2="-6.125" width="0.1016" layer="16"/>
+<wire x1="37" y1="-6.125" x2="36.5" y2="-5.625" width="0.1016" layer="16"/>
+<via x="36.5" y="-5.625" extent="1-16" drill="0.3"/>
 <wire x1="19.25" y1="-3.625" x2="19.25" y2="-2.75" width="0.1016" layer="16"/>
 <via x="19.25" y="-2.75" extent="1-16" drill="0.3"/>
@@
 <wire x1="48.25" y1="5.5" x2="48.25" y2="4.5" width="0.1016" layer="16"/>
 <via x="48.25" y="4.5" extent="1-16" drill="0.25"/>
-<wire x1="48.25" y1="-7" x2="49" y2="-8" width="0" layer="19" extent="1-1"/>
+<polygon width="0.15" layer="1" isolate="1" rank="6">
+<vertex x="-65" y="-17"/>
+<vertex x="65" y="-17"/>
+<vertex x="65" y="17"/>
+<vertex x="34" y="17"/>
+<vertex x="34" y="9.875"/>
+<vertex x="14" y="9.875"/>
+<vertex x="14" y="17"/>
+<vertex x="-65" y="17"/>
+</polygon>
+<polygon width="0.15" layer="16" isolate="1" rank="6">
+<vertex x="-65" y="-17"/>
+<vertex x="65" y="-17"/>
+<vertex x="65" y="17"/>
+<vertex x="34" y="17"/>
+<vertex x="34" y="9.875"/>
+<vertex x="14" y="9.875"/>
+<vertex x="14" y="17"/>
+<vertex x="-65" y="17"/>
+</polygon>
 </signal>
 <signal name="PWR_SYS_3V3">
@@
 <contactref element="D15" pad="2A"/>
 <contactref element="U15" pad="27"/>
-<wire x1="32.47" y1="-4.75" x2="32.5" y2="-4.72" width="0.1016" layer="1"/>
 <wire x1="32.5" y1="-4.72" x2="30.28" y2="-4.72" width="0.1016" layer="1"/>
 <wire x1="30.28" y1="-4.72" x2="30.25" y2="-4.75" width="0.1016" layer="1"/>

Commit message: Updated release dates
Connections:
- removed net FT_CONT_RX: U1.L10
- removed net FT_CONT_TX: U1.L9
Other:
- board text added: "Soke Eng. - knokke 3.0.0 2024.04.16"
Changed lines of the file:
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@@
 <text x="-30" y="8" size="2" layer="16" rot="MR0">Soke Eng. - knokke
 3.0.0
-2024.04.01</text>
+2024.04.16</text>
 <text x="-30" y="8" size="2" layer="30" rot="MR0">Soke Eng. - knokke
 3.0.0
@@
 <wire x1="-29.3536" y1="0.6036" x2="-33.75" y2="5" width="0.1016" layer="16"/>
 </signal>
-<signal name="FT_CONT_TX">
-<contactref element="U1" pad="L9"/>
-</signal>
-<signal name="FT_CONT_RX">
-<contactref element="U1" pad="L10"/>
-</signal>
 <signal name="LED_FT_CONT_NRXLED">
