File: led.sch (EAGLE design)
At the start: 7 parts

Commit message: Progress
Parts:
- removed TP1, TP2: TEST_POINT_SQUARE, MISC:TEST_POINT_SQUARE
- added C1, C2: 0.1uF 50V, c_0603:C0603C104K5RAC7081
- added C3: 1uF 50V, c_1206:C1206C105K5RACAUTO
- added C4: 2.2uF 10V, c_0603:CL10B225KP8NFNC
- added CN1: JST GH 10 Pin, CONNECTORs:1.25-10PWT
- added D10, D11, D12, D6, D7, D8, D9: 5000K, OPTO:SPHWH1L5N605YER3A4
- added MECH1, MECH2, MECH3, MECH4: 6mm x 3mm, MISC:MOUNTHOLE
- added Q1: FDD5612, TRANSISTORs:FDD5612
- added R1, R2, R7, R8: 1R, RESISTORS:CRCW12061R00FKEA
- added R3: 0.33R, RESISTORS:CRL0603-FW-R330ELF
- added R4: 100R, r_0603:CRCW0603100RFKEC
- added R5: 20k, r_0603:CRCW060320K0FKEA
- added R6: 10k, r_0603:CRCW060310K0FKTA
- added TH1: 10k 4037k, RESISTORS:NTCG164BF103HT1
- added U1: NCS20071, ICs:NCS20071SN2T1G
- added U2: TPS70950, ICs:TPS70950DBVT
Connections:
- removed net A: D1.A, TP1.P$1
- removed net K: D5.K, TP2.P$1
- new net GND: C1.1, C2.1, C3.1, C4.1, CN1.4, CN1.5, CN1.6, CN1.7, R3.1, R6.1, U1.V-, U2.GND
- new net LED_PWM_CONT: CN1.8, R5.1
- new net N$10: D11.K, D12.A
- new net N$11: D10.K, D11.A
- new net N$13: D1.A, R1.1
- new net N$16: D12.K, D3.K, D6.K, D9.K, Q1.D
- new net N$17: C1.2, R5.2, R6.2, U1.+
- new net N$18: Q1.G, R4.2
- new net N$19: R4.1, U1.OUT
- new net N$20: Q1.S, R3.2, U1.-
- new net N$22: C2.2, C4.2, U1.V+, U2.VOUT
- new net N$5: D5.K, D6.A
- new net N$6: D4.A, R2.1
- new net N$7: D8.K, D9.A
- new net N$8: D10.A, R7.1
- new net N$9: D7.A, R8.1
- new net PWR_LED_24V: C3.2, CN1.1, CN1.2, CN1.3, R1.2, R2.2, R7.2, R8.2, U2.EN, U2.VIN
- new net TEMP_SEN_A: CN1.9, TH1.2
- new net TEMP_SEN_B: CN1.10, TH1.1
- net N$3: now also D7.K, D8.A; no longer D3.K, D4.A
Other:
- moved on the sheet: D1, D2, D3, D4, D5

Commit message: Progression
Parts:
- removed C1, C2: 0.1uF 50V, c_0603:C0603C104K5RAC7081
- removed C3: 1uF 50V, c_1206:C1206C105K5RACAUTO
- removed C4: 2.2uF 10V, c_0603:CL10B225KP8NFNC
- removed CN1: JST GH 10 Pin, CONNECTORs:1.25-10PWT
- removed Q1: FDD5612, TRANSISTORs:FDD5612
- removed R1, R2, R7, R8: 1R, RESISTORS:CRCW12061R00FKEA
- removed R3: 0.33R, RESISTORS:CRL0603-FW-R330ELF
- removed R4: 100R, r_0603:CRCW0603100RFKEC
- removed R5: 20k, r_0603:CRCW060320K0FKEA
- removed R6: 10k, r_0603:CRCW060310K0FKTA
- removed TH1: 10k 4037k, RESISTORS:NTCG164BF103HT1
- removed U1: NCS20071, ICs:NCS20071SN2T1G
- removed U2: TPS70950, ICs:TPS70950DBVT
- added TP1, TP2: 2MM_TEST_POINT, MISC:2MM_TEST_POINT
Connections:
- removed net GND: C1.1, C2.1, C3.1, C4.1, CN1.4, CN1.5, CN1.6, CN1.7, R3.1, R6.1, U1.V-, U2.GND
- removed net LED_PWM_CONT: CN1.8, R5.1
- removed net N$10: D11.K, D12.A
- removed net N$11: D10.K, D11.A
- removed net N$13: D1.A, R1.1
- removed net N$16: D12.K, D3.K, D6.K, D9.K, Q1.D
- removed net N$17: C1.2, R5.2, R6.2, U1.+
- removed net N$18: Q1.G, R4.2
- removed net N$19: R4.1, U1.OUT
- removed net N$20: Q1.S, R3.2, U1.-
- removed net N$22: C2.2, C4.2, U1.V+, U2.VOUT
- removed net N$7: D8.K, D9.A
- removed net N$8: D10.A, R7.1
- removed net N$9: D7.A, R8.1
- removed net PWR_LED_24V: C3.2, CN1.1, CN1.2, CN1.3, R1.2, R2.2, R7.2, R8.2, U2.EN, U2.VIN
- removed net TEMP_SEN_A: CN1.9, TH1.2
- removed net TEMP_SEN_B: CN1.10, TH1.1
- new net ANODE: D1.A, D2.A, D3.A, D4.A, D5.A, D6.A, TP1.P$1
- new net CATHODE: D10.K, D11.K, D12.K, D7.K, D8.K, D9.K, TP2.P$1
- net N$1: now also D7.A; no longer D2.A
- net N$2: now also D8.A; no longer D3.A
- net N$3: now also D3.K, D9.A; no longer D7.K, D8.A
- net N$4: now also D10.A; no longer D5.A
- net N$5: now also D11.A; no longer D6.A
- net N$6: now also D12.A, D6.K; no longer D4.A, R2.1
Other:
- moved on the sheet: D1, D10, D11, D12, D2, D3, D4, D5, D6, D7, D8, D9
