File: led_drv.sch (EAGLE design)
At the start: 33 parts, among them CN1 JST GH 10 Pin, Q1 FDD5612, U1 NCS20071, U2 TPS70950

Commit message: New LED driver PCB
Parts:
- removed CN1: JST GH 10 Pin, CONNECTORs:1.25-10PWT
- removed D1, D10, D11, D12, D2, D3, D4, D5, D6, D7, D8, D9: 5000K, OPTO:SPHWH1L5N605YER3A4
- removed MECH3, MECH4: 6mm x 3mm, MISC:MOUNTHOLE
- removed R2, R7, R8: 1R, RESISTORS:CRCW12061R00FKEA
- removed TH1: 10k 4037k, RESISTORS:NTCG164BF103HT1
- added TP1, TP2, TP3, TP4, TP5, TP6: TEST_POINT_SQUARE, MISC:TEST_POINT_SQUARE
- C3: value 1uF 50V -> 1uF 25V; device c_1206:C1206C105K5RACAUTO -> c_0603:C0603C105K3RAC7411
- R1: value 1R -> 100R; device RESISTORS:CRCW12061R00FKEA -> r_0603:CRCW0603100RFKEC
Connections:
- removed net N$10: D11.K, D12.A
- removed net N$11: D10.K, D11.A
- removed net N$13: D1.A, R1.1
- removed net N$2: D2.K, D3.A
- removed net N$3: D7.K, D8.A
- removed net N$4: D4.K, D5.A
- removed net N$5: D5.K, D6.A
- removed net N$6: D4.A, R2.1
- removed net N$7: D8.K, D9.A
- removed net N$8: D10.A, R7.1
- removed net N$9: D7.A, R8.1
- removed net PWR_LED_24V: C3.2, CN1.1, CN1.2, CN1.3, R1.2, R2.2, R7.2, R8.2, U2.EN, U2.VIN
- removed net TEMP_SEN_A: CN1.9, TH1.2
- removed net TEMP_SEN_B: CN1.10, TH1.1
- new net GND_SIG: C1.1, R6.1, TP4.P$1
- new net PWR_LED_18V: C3.2, TP2.P$1, TP5.P$1, U2.EN, U2.VIN
- net GND: now also TP3.P$1; no longer C1.1, CN1.4, CN1.5, CN1.6, CN1.7, R6.1
- net LED_PWM_CONT: now also TP1.P$1; no longer CN1.8
- net N$1: now also Q1.S, R1.2, R3.2; no longer D1.K, D2.A
- net N$16: now also TP6.P$1; no longer D12.K, D3.K, D6.K, D9.K
- net N$20: now also R1.1; no longer Q1.S, R3.2
Other:
- moved on the sheet: R1
