File: led.brd (EAGLE design)
At the start: 14 x 26 mm, 7 parts

Commit message: New LED layout
Parts:
- added D6: 5000K, OPTO:LH502C
- moved D1 5.00 mm to (7.00, 28.2)
- moved D2 5.00 mm to (7.00, 23.1)
- moved D3 5.00 mm to (7.00, 18.0)
- moved D4 5.00 mm to (7.00, 12.9)
- moved D5 5.00 mm to (7.00, 7.75)
Connections:
- removed net N$2: D2.K, D3.A
- removed net N$4: D4.K, D5.A
- new net N$5: D5.K, D6.A
- net A: now also D3.A, D5.A
- net K: now also D2.K, D4.K, D6.K; no longer D5.K
Routing:
- net K: track 6.03 -> 1.41 mm
- net N$5: track 0.00 -> 2.62 mm
- net N$4: track 2.62 -> 0.00 mm
- net N$2: track 2.62 -> 0.00 mm
- added copper zone on layer 1, net K
Other:
- board size 14 x 26 mm -> 14 x 31 mm
