File: led.brd (EAGLE design)
At the start: 14 x 26 mm, 7 parts

Commit message: Progress
Parts:
- removed TP1, TP2: TEST_POINT_SQUARE, MISC:OSPREY_HSS_PAD
- added C1, C2: 0.1uF 50V, c_0603:0603
- added C3: 1uF 50V, c_1206:1206
- added C4: 2.2uF 10V, c_0603:0603
- added CN1: JST GH 10 Pin, CONNECTORs:1.25-10PWT
- added D10, D11, D12, D6, D7, D8, D9: 5000K, OPTO:LH502C
- added MECH1, MECH2, MECH3, MECH4: 6mm x 3mm, MISC:MOUNTHOLE_6X3
- added Q1: FDD5612, TRANSISTORs:TO252
- added R1, R2, R7, R8: 1R, RESISTORS:1206
- added R3: 0.33R, RESISTORS:0603
- added R4: 100R, r_0603:0603
- added R5: 20k, r_0603:0603
- added R6: 10k, r_0603:0603
- added TH1: 10k 4037k, RESISTORS:0603
- added U1: NCS20071, ICs:SOT23-5
- added U2: TPS70950, ICs:SOT23-5
- moved D4 22.8 mm to (-2.56, -12.8), turned to 270 degrees
- moved D1 14.2 mm to (-2.56, 12.8)
- moved D2 14.2 mm to (-2.56, 7.69)
- moved D3 14.2 mm to (-2.56, 2.56)
- moved D5 14.2 mm to (-2.56, -7.69), turned to 270 degrees
Connections:
- removed net A: D1.A, TP1.1
- removed net K: D5.K, TP2.1
- new net GND: C1.1, C2.1, C3.1, C4.1, CN1.4, CN1.5, CN1.6, CN1.7, R3.1, R6.1, U1.2, U2.2
- new net LED_PWM_CONT: CN1.8, R5.1
- new net N$10: D11.K, D12.A
- new net N$11: D10.K, D11.A
- new net N$13: D1.A, R1.1
- new net N$16: D12.K, D3.K, D6.K, D9.K, Q1.2
- new net N$17: C1.2, R5.2, R6.2, U1.3
- new net N$18: Q1.1, R4.2
- new net N$19: R4.1, U1.1
- new net N$20: Q1.3, R3.2, U1.4
- new net N$22: C2.2, C4.2, U1.5, U2.5
- new net N$5: D5.K, D6.A
- new net N$6: D4.A, R2.1
- new net N$7: D8.K, D9.A
- new net N$8: D10.A, R7.1
- new net N$9: D7.A, R8.1
- new net PWR_LED_24V: C3.2, CN1.1, CN1.2, CN1.3, R1.2, R2.2, R7.2, R8.2, U2.1, U2.3
- new net TEMP_SEN_A: CN1.9, TH1.2
- new net TEMP_SEN_B: CN1.10, TH1.1
- net N$3: now also D7.K, D8.A; no longer D3.K, D4.A
Routing:
- net GND: track 0.00 -> 131.6 mm
- net PWR_LED_24V: track 0.00 -> 96.2 mm
- net LED_PWM_CONT: track 0.00 -> 48.1 mm
- net N$16: track 0.00 -> 22.3 mm
- net N$20: track 0.00 -> 20.6 mm
- net N$22: track 0.00 -> 10.5 mm
- net K: track 6.03 -> 0.00 mm
- net N$17: track 0.00 -> 5.13 mm
- net TEMP_SEN_A: track 0.00 -> 4.68 mm
- net N$19: track 0.00 -> 3.58 mm
- net TEMP_SEN_B: track 0.00 -> 3.54 mm
- net N$7: track 0.00 -> 2.62 mm
- net N$5: track 0.00 -> 2.62 mm
- net N$11: track 0.00 -> 2.62 mm
- net N$10: track 0.00 -> 2.62 mm
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- added copper zone on layer 1, net PLANE
- removed copper zone on layer 1, net A
Other:
- board size 14 x 26 mm -> 50 x 50 mm

Commit message: FTDI and CCD routed
Parts:
- moved MECH1 1.41 mm to (-10.0, -10.0)
- moved MECH2 1.41 mm to (-10.0, 10.0)
- moved MECH3 1.41 mm to (10.0, 10.0)
- moved MECH4 1.41 mm to (10.0, -10.0)
Routing:
- removed copper zone on layer 1, net PLANE
Changed lines of the file:
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@@
 <setting verticaltext="up"/>
 </settings>
-<grid distance="0.125" unitdist="mm" unit="mm" style="lines" multiple="1" display="yes" altdistance="0.0625" altunitdist="mm" altunit="mm"/>
+<grid distance="0.1" unitdist="mm" unit="mm" style="lines" multiple="1" display="yes" altdistance="0.0625" altunitdist="mm" altunit="mm"/>
 <layers>
 <layer number="1" name="Top" color="4" fill="1" visible="yes" active="yes"/>
@@
 </layers>
 <board>
-<fusionsync huburn="a.YnVzaW5lc3M6bXl1Y2wxNDk2" projecturn="a.YnVzaW5lc3M6bXl1Y2wxNDk2IzIwMjIwMzI1NTEwNjk2MjUx" f3durn="urn:adsk.wipprod:dm.lineage:EBDbe4bRQn2SoMot8VX7aQ" pcbguid="" lastpulledtime="" lastsyncedchangeguid="" latestrevisionid="b7922e21-8bae-4f5b-a0f9-7ee542d19b22" lastsyncedrevisionid="b7922e21-8bae-4f5b-a0f9-7ee542d19b22" lastboardhashguid="e4326e94-9937-d6ec-a489-b1db77b3a7e5" lastpushedtime="2024-01-21T22:24:46Z" linktopcb3d="true"/>
+<fusionsync huburn="a.YnVzaW5lc3M6bXl1Y2wxNDk2" projecturn="a.YnVzaW5lc3M6bXl1Y2wxNDk2IzIwMjIwMzI1NTEwNjk2MjUx" f3durn="urn:adsk.wipprod:dm.lineage:EBDbe4bRQn2SoMot8VX7aQ" pcbguid="" lastpulledtime="" lastsyncedchangeguid="" latestrevisionid="3b36d295-92bd-4a33-93f4-9afc759f84f0" lastsyncedrevisionid="3b36d295-92bd-4a33-93f4-9afc759f84f0" lastboardhashguid="82e2d37c-5323-3068-0343-bf393cc3bb86" lastpushedtime="2024-02-17T15:42:22Z" linktopcb3d="true"/>
 <plain>
-<wire x1="-22" y1="-25" x2="22" y2="-25" width="0" layer="20" locked="yes"/>
-<wire x1="22" y1="-25" x2="25" y2="-22" width="0" layer="20" curve="90" locked="yes"/>
-<wire x1="25" y1="-22" x2="25" y2="22" width="0" layer="20" locked="yes"/>
-<wire x1="25" y1="22" x2="22" y2="25" width="0" layer="20" curve="90" locked="yes"/>
-<wire x1="22" y1="25" x2="-22" y2="25" width="0" layer="20" locked="yes"/>
-<wire x1="-22" y1="25" x2="-25" y2="22" width="0" layer="20" curve="90" locked="yes"/>
-<wire x1="-25" y1="22" x2="-25" y2="-22" width="0" layer="20" locked="yes"/>
-<wire x1="-25" y1="-22" x2="-22" y2="-25" width="0" layer="20" curve="90" locked="yes"/>
+<wire x1="-22" y1="-25" x2="22" y2="-25" width="0" layer="20"/>
+<wire x1="22" y1="-25" x2="25" y2="-22" width="0" layer="20" curve="90"/>
+<wire x1="25" y1="-22" x2="25" y2="22" width="0" layer="20"/>
+<wire x1="25" y1="22" x2="22" y2="25" width="0" layer="20" curve="90"/>
+<wire x1="22" y1="25" x2="-22" y2="25" width="0" layer="20"/>
+<wire x1="-22" y1="25" x2="-25" y2="22" width="0" layer="20" curve="90"/>
+<wire x1="-25" y1="22" x2="-25" y2="-22" width="0" layer="20"/>
+<wire x1="-25" y1="-22" x2="-22" y2="-25" width="0" layer="20" curve="90"/>
 </plain>
 <attributes>
@@
 <attribute name="VOLTAGE" value="10V" x="17.4375" y="-14.6875" size="1.778" layer="27" rot="R90" display="off"/>
 </element>
-<element name="MECH1" library="MISC" package="MOUNTHOLE_6X3" value="6mm x 3mm" x="-9" y="-9" locked="yes" smashed="yes"/>
-<element name="MECH2" library="MISC" package="MOUNTHOLE_6X3" value="6mm x 3mm" x="-9" y="9" locked="yes" smashed="yes"/>
-<element name="MECH3" library="MISC" package="MOUNTHOLE_6X3" value="6mm x 3mm" x="9" y="9" locked="yes" smashed="yes"/>
-<element name="MECH4" library="MISC" package="MOUNTHOLE_6X3" value="6mm x 3mm" x="9" y="-9" locked="yes" smashed="yes"/>
-<element name="CN1" library="CONNECTORs" package="1.25-10PWT" value="JST GH 10 Pin" x="-15" y="4" locked="yes" smashed="yes" rot="R315">
-<attribute name="HEIGHT" value="3.6" x="-15" y="4" locked="yes" size="0.5" layer="27" rot="R315" display="off"/>
-<attribute name="LCSC" value="C5340797" x="-15" y="4" locked="yes" size="0.5" layer="27" rot="R315" display="off"/>
-<attribute name="NAME" x="-19.331028125" y="12.927221875" locked="yes" size="0.5" layer="25" rot="R315"/>
-<attribute name="PRICE_PER" value="0.035" x="-15" y="4" locked="yes" size="0.5" layer="27" rot="R315" display="off"/>
+<element name="MECH1" library="MISC" package="MOUNTHOLE_6X3" value="6mm x 3mm" x="-10" y="-10" smashed="yes"/>
+<element name="MECH2" library="MISC" package="MOUNTHOLE_6X3" value="6mm x 3mm" x="-10" y="10" smashed="yes"/>
+<element name="MECH3" library="MISC" package="MOUNTHOLE_6X3" value="6mm x 3mm" x="10" y="10" smashed="yes"/>
+<element name="MECH4" library="MISC" package="MOUNTHOLE_6X3" value="6mm x 3mm" x="10" y="-10" smashed="yes"/>
+<element name="CN1" library="CONNECTORs" package="1.25-10PWT" value="JST GH 10 Pin" x="-15" y="4" smashed="yes" rot="R315">
+<attribute name="HEIGHT" value="3.6" x="-15" y="4" size="0.5" layer="27" rot="R315" display="off"/>
+<attribute name="LCSC" value="C5340797" x="-15" y="4" size="0.5" layer="27" rot="R315" display="off"/>
+<attribute name="NAME" x="-19.331028125" y="12.927221875" size="0.5" layer="25" rot="R315"/>
+<attribute name="PRICE_PER" value="0.035" x="-15" y="4" size="0.5" layer="27" rot="R315" display="off"/>
 </element>
 <element name="TH1" library="RESISTORS" package="0603" value="10k 4037k" x="-6.75" y="4.125" smashed="yes" rot="R90">
@@
 <wire x1="-7.670046875" y1="3.375" x2="-6.75" y2="3.375" width="0.15" layer="1"/>
 </signal>
-<signal name="PLANE">
-<polygon width="0.15" layer="1">
-<vertex x="0" y="-25"/>
-<vertex x="25" y="-25"/>
-<vertex x="25" y="0"/>
-<vertex x="25" y="25"/>
-<vertex x="0" y="25"/>
-<vertex x="-25" y="25"/>
-<vertex x="-25" y="0"/>
-<vertex x="-25" y="-25"/>
-</polygon>
-</signal>
 </signals>
 <mfgpreviewcolors>
@@
 the document will break the link to the Fusion PCB feature.
 </note>
-<note version="8.5" severity="warning">
-Since Version 8.5, EAGLE supports locking for holes, vias, wires and polygons.
-The locking property on all objects of these types will not be understood in this version.
-</note>
 </compatibility>

Commit message: New LED PCB formfactor. UART debug added to FPGA for softcore.
Parts:
- moved C1 71.1 mm to (13.8, -81.8)
- moved C2 71.1 mm to (19.3, -78.4)
- moved C3 71.1 mm to (18.8, -89.7)
- moved C4 71.1 mm to (15.9, -85.8)
- moved Q1 71.1 mm to (11.9, -70.4)
- moved R1 71.1 mm to (-4.06, -53.3)
- moved R2 71.1 mm to (-4.06, -88.9)
- moved R3 71.1 mm to (16.4, -66.3)
- moved R4 71.1 mm to (17.2, -75.3)
- moved R5 71.1 mm to (12.6, -81.8)
- moved R6 71.1 mm to (15.1, -81.8)
- moved R7 71.1 mm to (1.06, -88.9)
- moved R8 71.1 mm to (1.06, -53.3)
- moved TH1 71.1 mm to (-8.25, -67.0)
- moved U1 71.1 mm to (18.6, -80.6)
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Routing:
- net GND: track 131.6 -> 0.00 mm
- net PWR_LED_24V: track 96.2 -> 0.00 mm
- net LED_PWM_CONT: track 48.1 -> 0.00 mm
- net N$16: track 22.3 -> 0.00 mm
- net N$20: track 20.6 -> 0.00 mm
- net N$22: track 10.5 -> 0.00 mm
- net N$17: track 5.13 -> 0.00 mm
- net TEMP_SEN_A: track 4.68 -> 0.00 mm
- net N$19: track 3.58 -> 0.00 mm
- net TEMP_SEN_B: track 3.54 -> 0.00 mm
- net N$4: track 2.73 -> 0.00 mm
- net N$7: track 2.62 -> 0.00 mm
- net N$5: track 2.62 -> 0.00 mm
- net N$3: track 2.62 -> 0.00 mm
- net N$2: track 2.62 -> 0.00 mm
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Other:
- board size 50 x 50 mm -> 28 x 67 mm

Commit message: Progression
Parts:
- removed C1, C2: 0.1uF 50V, c_0603:0603
- removed C3: 1uF 50V, c_1206:1206
- removed C4: 2.2uF 10V, c_0603:0603
- removed CN1: JST GH 10 Pin, CONNECTORs:1.25-10PWT
- removed Q1: FDD5612, TRANSISTORs:TO252
- removed R1, R2, R7, R8: 1R, RESISTORS:1206
- removed R3: 0.33R, RESISTORS:0603
- removed R4: 100R, r_0603:0603
- removed R5: 20k, r_0603:0603
- removed R6: 10k, r_0603:0603
- removed TH1: 10k 4037k, RESISTORS:0603
- removed U1: NCS20071, ICs:SOT23-5
- removed U2: TPS70950, ICs:SOT23-5
- added TP1, TP2: 2MM_TEST_POINT, MISC:2MM_TEST_PAD
- turned D1 to 180 degrees
- turned D10 to 180 degrees
- turned D11 to 180 degrees
- turned D12 to 180 degrees
- turned D2 to 180 degrees
- turned D3 to 180 degrees
- turned D4 to 180 degrees
- turned D5 to 180 degrees
- turned D6 to 180 degrees
- turned D7 to 180 degrees
- turned D8 to 180 degrees
- turned D9 to 180 degrees
Connections:
- removed net GND: C1.1, C2.1, C3.1, C4.1, CN1.4, CN1.5, CN1.6, CN1.7, R3.1, R6.1, U1.2, U2.2
- removed net LED_PWM_CONT: CN1.8, R5.1
- removed net N$10: D11.K, D12.A
- removed net N$11: D10.K, D11.A
- removed net N$13: D1.A, R1.1
- removed net N$16: D12.K, D3.K, D6.K, D9.K, Q1.2
- removed net N$17: C1.2, R5.2, R6.2, U1.3
- removed net N$18: Q1.1, R4.2
- removed net N$19: R4.1, U1.1
- removed net N$20: Q1.3, R3.2, U1.4
- removed net N$22: C2.2, C4.2, U1.5, U2.5
- removed net N$7: D8.K, D9.A
- removed net N$8: D10.A, R7.1
- removed net N$9: D7.A, R8.1
- removed net PWR_LED_24V: C3.2, CN1.1, CN1.2, CN1.3, R1.2, R2.2, R7.2, R8.2, U2.1, U2.3
- removed net TEMP_SEN_A: CN1.9, TH1.2
- removed net TEMP_SEN_B: CN1.10, TH1.1
- new net ANODE: D1.A, D2.A, D3.A, D4.A, D5.A, D6.A, TP1.1
- new net CATHODE: D10.K, D11.K, D12.K, D7.K, D8.K, D9.K, TP2.1
- net N$1: now also D7.A; no longer D2.A
- net N$2: now also D8.A; no longer D3.A
- net N$3: now also D3.K, D9.A; no longer D7.K, D8.A
- net N$4: now also D10.A; no longer D5.A
- net N$5: now also D11.A; no longer D6.A
- net N$6: now also D12.A, D6.K; no longer D4.A, R2.1
Routing:
- net N$6: track 0.00 -> 2.62 mm
- net N$5: track 0.00 -> 2.62 mm
- net N$4: track 0.00 -> 2.62 mm
- net N$3: track 0.00 -> 2.62 mm
- net N$2: track 0.00 -> 2.62 mm
- net N$1: track 0.00 -> 2.62 mm
- added copper zone on layer 1, net ANODE
- added copper zone on layer 1, net CATHODE
Other:
- board size 28 x 67 mm -> 28 x 34 mm

Commit message: ESP32 added with architecture implemented. First attempt.
Changed lines of the file:
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@@
 <setting verticaltext="up"/>
 </settings>
-<grid distance="1" unitdist="mm" unit="mm" style="lines" multiple="1" display="yes" altdistance="0.0625" altunitdist="mm" altunit="mm"/>
+<grid distance="0.125" unitdist="mm" unit="mm" style="lines" multiple="1" display="yes" altdistance="0.0625" altunitdist="mm" altunit="mm"/>
 <layers>
 <layer number="1" name="Top" color="4" fill="1" visible="yes" active="yes"/>
@@
 <wire x1="14" y1="16" x2="14" y2="-16" width="0" layer="20"/>
 <wire x1="14" y1="-16" x2="13" y2="-17" width="0" layer="20" curve="-90"/>
+<rectangle x1="-10" y1="-17" x2="-6" y2="-13" layer="21"/>
 </plain>
 <attributes>
